Commit message: add Rizon 4s support

File: flexiv_description/urdf/rizon.ros2_control.xacro (robot description, xacro)
@@ -1,5 +1,5 @@
 <?xml version="1.0"?>
 <robot xmlns:xacro="http://www.ros.org/wiki/xacro">
-  <xacro:macro name="rizon4_ros2_control" params="prefix robot_ip local_ip use_fake_hardware:=^|false fake_sensor_commands:=^|false initial_positions_file">
+  <xacro:macro name="rizon_ros2_control" params="prefix robot_ip local_ip use_fake_hardware:=^|false fake_sensor_commands:=^|false initial_positions_file">
     <xacro:property name="initial_positions" value="${load_yaml(initial_positions_file)['initial_positions']}"/>
     <ros2_control name="FlexivHardwareInterface" type="system">

File: flexiv_description/urdf/rizon.urdf.xacro (robot description, xacro)
@@ -4,14 +4,15 @@
   <xacro:arg name="robot_ip" default="" />
   <xacro:arg name="local_ip" default="" />
+  <xacro:arg name="rizon_type" default="rizon4"/>
   <xacro:arg name="use_fake_hardware" default="false" />
   <xacro:arg name="fake_sensor_commands" default="false" />
   <xacro:arg name="initial_positions_file" default="$(find flexiv_description)/config/initial_positions.yaml"/>
   <xacro:arg name="prefix" default="" />
-  <xacro:include filename="$(find flexiv_description)/urdf/rizon4_joints_links.xacro" />
-  <xacro:rizon4_joints_links product_id="A02L-M" prefix="$(arg prefix)" mesh_prefix_path="package://flexiv_description/" />
+  <xacro:include filename="$(find flexiv_description)/urdf/rizon_joints_links.xacro" />
+  <xacro:rizon_joints_links rizon_type="$(arg rizon_type)" prefix="$(arg prefix)" mesh_prefix_path="package://flexiv_description/" />
   <xacro:include filename="$(find flexiv_description)/urdf/flexiv_arm_materials.xacro" />
   <xacro:flexiv_arm_materials />
-  <xacro:include filename="$(find flexiv_description)/urdf/rizon4.ros2_control.xacro"/>
-  <xacro:rizon4_ros2_control prefix="$(arg prefix)" robot_ip="$(arg robot_ip)" local_ip="$(arg local_ip)" use_fake_hardware="$(arg use_fake_hardware)" fake_sensor_commands="$(arg fake_sensor_commands)" initial_positions_file="$(arg initial_positions_file)"/>
+  <xacro:include filename="$(find flexiv_description)/urdf/rizon.ros2_control.xacro"/>
+  <xacro:rizon_ros2_control prefix="$(arg prefix)" robot_ip="$(arg robot_ip)" local_ip="$(arg local_ip)" use_fake_hardware="$(arg use_fake_hardware)" fake_sensor_commands="$(arg fake_sensor_commands)" initial_positions_file="$(arg initial_positions_file)"/>
   <!-- Used for fixing robot -->
 </robot>

File: flexiv_description/urdf/rizon_joints_links.xacro (robot description, xacro)
@@ -2,10 +2,10 @@
 <robot xmlns:xacro="http://www.ros.org/wiki/xacro">
   <!--
-    product_id = "A02L-M"
+    rizon_type = "rizon4", "rizon4s"
     prefix = "", "left_"
     mesh_prefix_path = "", "package://flexiv_description/"
     NOTE: accurate kinematic but approximated dynamics parameters
   -->
-  <xacro:macro name="rizon4_joints_links" params="product_id prefix mesh_prefix_path">
+  <xacro:macro name="rizon_joints_links" params="rizon_type prefix mesh_prefix_path">
     <!-- JOINTS-->
     <joint name="${prefix}base_joint" type="fixed">
@@ -66,6 +66,9 @@
       <parent link="${prefix}link7"/>
       <child link="${prefix}flange"/>
-      <xacro:if value="${product_id=='A02L-M'}">
+      <xacro:if value="${rizon_type=='rizon4'}">
         <origin xyz="0.0 0.0 0.081" rpy="0 0 ${-pi}"/>
+      </xacro:if>
+      <xacro:if value="${rizon_type=='rizon4s'}">
+        <origin xyz="0.0 0.0 0.124" rpy="0 0 ${-pi}"/>
       </xacro:if>
     </joint>
@@ -82,11 +85,11 @@
         <origin xyz="0 0 0" rpy="0 0 0"/>
         <geometry>
-          <mesh filename="${mesh_prefix_path}meshes/rizon4/visual/link0.obj" />
-        </geometry>
-      </visual>
-      <collision>
-        <origin xyz="0 0 0" rpy="0 0 0"/>
-        <geometry>
-          <mesh filename="${mesh_prefix_path}meshes/rizon4/collision/link0.obj" />
+          <mesh filename="${mesh_prefix_path}meshes/${rizon_type}/visual/link0.obj" />
+        </geometry>
+      </visual>
+      <collision>
+        <origin xyz="0 0 0" rpy="0 0 0"/>
+        <geometry>
+          <mesh filename="${mesh_prefix_path}meshes/${rizon_type}/collision/link0.obj" />
         </geometry>
       </collision>
@@ -101,11 +104,11 @@
         <origin xyz="0 0 0" rpy="0 0 0" />
         <geometry>
-          <mesh filename="${mesh_prefix_path}meshes/rizon4/visual/link1.obj" />
-        </geometry>
-      </visual>
-      <collision>
-        <origin xyz="0 0 0" rpy="0 0 0" />
-        <geometry>
-          <mesh filename="${mesh_prefix_path}meshes/rizon4/collision/link1.obj" />
+          <mesh filename="${mesh_prefix_path}meshes/${rizon_type}/visual/link1.obj" />
+        </geometry>
+      </visual>
+      <collision>
+        <origin xyz="0 0 0" rpy="0 0 0" />
+        <geometry>
+          <mesh filename="${mesh_prefix_path}meshes/${rizon_type}/collision/link1.obj" />
         </geometry>
       </collision>
@@ -120,11 +123,11 @@
         <origin xyz="0 0 0" rpy="0 0 0"/>
         <geometry>
-          <mesh filename="${mesh_prefix_path}meshes/rizon4/visual/link2.obj" />
-        </geometry>
-      </visual>
-      <collision>
-        <origin xyz="0 0 0" rpy="0 0 0"/>
-        <geometry>
-          <mesh filename="${mesh_prefix_path}meshes/rizon4/collision/link2.obj" />
+          <mesh filename="${mesh_prefix_path}meshes/${rizon_type}/visual/link2.obj" />
+        </geometry>
+      </visual>
+      <collision>
+        <origin xyz="0 0 0" rpy="0 0 0"/>
+        <geometry>
+          <mesh filename="${mesh_prefix_path}meshes/${rizon_type}/collision/link2.obj" />
         </geometry>
       </collision>
@@ -139,11 +142,11 @@
         <origin xyz="0 0 0" rpy="0 0 0" />
         <geometry>
-          <mesh filename="${mesh_prefix_path}meshes/rizon4/visual/link3.obj" />
-        </geometry>
-      </visual>
-      <collision>
-        <origin xyz="0 0 0" rpy="0 0 0" />
-        <geometry>
-          <mesh filename="${mesh_prefix_path}meshes/rizon4/collision/link3.obj" />
+          <mesh filename="${mesh_prefix_path}meshes/${rizon_type}/visual/link3.obj" />
+        </geometry>
+      </visual>
+      <collision>
+        <origin xyz="0 0 0" rpy="0 0 0" />
+        <geometry>
+          <mesh filename="${mesh_prefix_path}meshes/${rizon_type}/collision/link3.obj" />
         </geometry>
       </collision>
@@ -158,11 +161,11 @@
         <origin xyz="0 0 0" rpy="0 0 0"/>
         <geometry>
-          <mesh filename="${mesh_prefix_path}meshes/rizon4/visual/link4.obj" />
-        </geometry>
-      </visual>
-      <collision>
-        <origin xyz="0 0 0" rpy="0 0 0"/>
-        <geometry>
-          <mesh filename="${mesh_prefix_path}meshes/rizon4/collision/link4.obj" />
+          <mesh filename="${mesh_prefix_path}meshes/${rizon_type}/visual/link4.obj" />
+        </geometry>
+      </visual>
+      <collision>
+        <origin xyz="0 0 0" rpy="0 0 0"/>
+        <geometry>
+          <mesh filename="${mesh_prefix_path}meshes/${rizon_type}/collision/link4.obj" />
         </geometry>
       </collision>
@@ -177,11 +180,11 @@
         <origin xyz="0 0 0" rpy="0 0 0"/>
         <geometry>
-          <mesh filename="${mesh_prefix_path}meshes/rizon4/visual/link5.obj" />
-        </geometry>
-      </visual>
-      <collision>
-        <origin xyz="0 0 0" rpy="0 0 0"/>
-        <geometry>
-          <mesh filename="${mesh_prefix_path}meshes/rizon4/collision/link5.obj" />
+          <mesh filename="${mesh_prefix_path}meshes/${rizon_type}/visual/link5.obj" />
+        </geometry>
+      </visual>
+      <collision>
+        <origin xyz="0 0 0" rpy="0 0 0"/>
+        <geometry>
+          <mesh filename="${mesh_prefix_path}meshes/${rizon_type}/collision/link5.obj" />
         </geometry>
       </collision>
@@ -196,16 +199,16 @@
         <origin xyz="0 0 0" rpy="0 0 0"/>
         <geometry>
-          <mesh filename="${mesh_prefix_path}meshes/rizon4/visual/link6.obj" />
-        </geometry>
-      </visual>
-      <collision>
-        <origin xyz="0 0 0" rpy="0 0 0"/>
-        <geometry>
-          <mesh filename="${mesh_prefix_path}meshes/rizon4/collision/link6.obj" />
+          <mesh filename="${mesh_prefix_path}meshes/${rizon_type}/visual/link6.obj" />
+        </geometry>
+      </visual>
+      <collision>
+        <origin xyz="0 0 0" rpy="0 0 0"/>
+        <geometry>
+          <mesh filename="${mesh_prefix_path}meshes/${rizon_type}/collision/link6.obj" />
         </geometry>
       </collision>
     </link>
     <link name="${prefix}link7">
-      <xacro:if value="${product_id=='A02L-M'}">
+      <xacro:if value="${rizon_type=='rizon4'}">
         <inertial>
           <mass value="0.8" />
@@ -216,5 +219,5 @@
           <origin xyz="0 0 0" rpy="0 0 0"/>
           <geometry>
-            <mesh filename="${mesh_prefix_path}meshes/rizon4/visual/link7.obj" />
+            <mesh filename="${mesh_prefix_path}meshes/${rizon_type}/visual/link7.obj" />
           </geometry>
         </visual>
@@ -222,5 +225,24 @@
           <origin xyz="0 0 0" rpy="0 0 0"/>
           <geometry>
-            <mesh filename="${mesh_prefix_path}meshes/rizon4/collision/link7.obj" />
+            <mesh filename="${mesh_prefix_path}meshes/${rizon_type}/collision/link7.obj" />
+          </geometry>
+        </collision>
+      </xacro:if>
+      <xacro:if value="${rizon_type=='rizon4s'}">
+        <inertial>
+          <mass value="1.4" />
+          <origin xyz="0.0 0.0 0.05" rpy="0 0 0"/>
+          <inertia ixx="0.003" iyy="0.003" izz="0.002" ixy="0.0" ixz="0.0" iyz="0.0"/>
+        </inertial>
+        <visual>
+          <origin xyz="0 0 0" rpy="0 0 0"/>
+          <geometry>
+            <mesh filename="${mesh_prefix_path}meshes/${rizon_type}/visual/link7.obj" />
+          </geometry>
+        </visual>
+        <collision>
+          <origin xyz="0 0 0" rpy="0 0 0"/>
+          <geometry>
+            <mesh filename="${mesh_prefix_path}meshes/${rizon_type}/collision/link7.obj" />
           </geometry>
         </collision>

File: flexiv_moveit_config/srdf/rizon.srdf.xacro (robot description, xacro)
@@ -2,8 +2,8 @@
 <robot xmlns:xacro="http://wiki.ros.org/xacro" name="$(arg name)">
     <!-- robot name parameter -->
-    <xacro:arg name="name" default="rizon4"/>
+    <xacro:arg name="name" default="rizon"/>
     <!-- parameters -->
     <xacro:arg name="prefix" default="" />
-    <xacro:include filename="$(find flexiv_moveit_config)/srdf/rizon4_macro.srdf.xacro"/>
-    <xacro:rizon4_srdf name="$(arg name)" prefix="$(arg prefix)"/>
+    <xacro:include filename="$(find flexiv_moveit_config)/srdf/rizon_macro.srdf.xacro"/>
+    <xacro:rizon_srdf name="$(arg name)" prefix="$(arg prefix)"/>
 </robot>

File: flexiv_moveit_config/srdf/rizon_macro.srdf.xacro (robot description, xacro)
@@ -1,5 +1,5 @@
 <?xml version="1.0" encoding="UTF-8"?>
 <robot xmlns:xacro="http://www.ros.org/wiki/xacro">
-    <xacro:macro name="rizon4_srdf" params="name prefix">
+    <xacro:macro name="rizon_srdf" params="name prefix">
         <group name="${prefix}${name}_arm">
             <chain base_link="${prefix}base_link" tip_link="${prefix}flange" />
