Commit message: Add .stl collision mesh files for Rizon 4 and 4s

File: flexiv_description/urdf/rizon_joints_links.xacro (robot description, xacro)
@@ -91,5 +91,5 @@
         <origin xyz="0 0 0" rpy="0 0 0"/>
         <geometry>
-          <mesh filename="${mesh_prefix_path}meshes/${rizon_type}/collision/link0.obj" />
+          <mesh filename="${mesh_prefix_path}meshes/${rizon_type}/collision/link0.stl" />
         </geometry>
       </collision>
@@ -110,5 +110,5 @@
         <origin xyz="0 0 0" rpy="0 0 0" />
         <geometry>
-          <mesh filename="${mesh_prefix_path}meshes/${rizon_type}/collision/link1.obj" />
+          <mesh filename="${mesh_prefix_path}meshes/${rizon_type}/collision/link1.stl" />
         </geometry>
       </collision>
@@ -129,5 +129,5 @@
         <origin xyz="0 0 0" rpy="0 0 0"/>
         <geometry>
-          <mesh filename="${mesh_prefix_path}meshes/${rizon_type}/collision/link2.obj" />
+          <mesh filename="${mesh_prefix_path}meshes/${rizon_type}/collision/link2.stl" />
         </geometry>
       </collision>
@@ -148,5 +148,5 @@
         <origin xyz="0 0 0" rpy="0 0 0" />
         <geometry>
-          <mesh filename="${mesh_prefix_path}meshes/${rizon_type}/collision/link3.obj" />
+          <mesh filename="${mesh_prefix_path}meshes/${rizon_type}/collision/link3.stl" />
         </geometry>
       </collision>
@@ -167,5 +167,5 @@
         <origin xyz="0 0 0" rpy="0 0 0"/>
         <geometry>
-          <mesh filename="${mesh_prefix_path}meshes/${rizon_type}/collision/link4.obj" />
+          <mesh filename="${mesh_prefix_path}meshes/${rizon_type}/collision/link4.stl" />
         </geometry>
       </collision>
@@ -186,5 +186,5 @@
         <origin xyz="0 0 0" rpy="0 0 0"/>
         <geometry>
-          <mesh filename="${mesh_prefix_path}meshes/${rizon_type}/collision/link5.obj" />
+          <mesh filename="${mesh_prefix_path}meshes/${rizon_type}/collision/link5.stl" />
         </geometry>
       </collision>
@@ -205,5 +205,5 @@
         <origin xyz="0 0 0" rpy="0 0 0"/>
         <geometry>
-          <mesh filename="${mesh_prefix_path}meshes/${rizon_type}/collision/link6.obj" />
+          <mesh filename="${mesh_prefix_path}meshes/${rizon_type}/collision/link6.stl" />
         </geometry>
       </collision>
@@ -225,5 +225,5 @@
           <origin xyz="0 0 0" rpy="0 0 0"/>
           <geometry>
-            <mesh filename="${mesh_prefix_path}meshes/${rizon_type}/collision/link7.obj" />
+            <mesh filename="${mesh_prefix_path}meshes/${rizon_type}/collision/link7.stl" />
           </geometry>
         </collision>
@@ -244,5 +244,5 @@
           <origin xyz="0 0 0" rpy="0 0 0"/>
           <geometry>
-            <mesh filename="${mesh_prefix_path}meshes/${rizon_type}/collision/link7.obj" />
+            <mesh filename="${mesh_prefix_path}meshes/${rizon_type}/collision/link7.stl" />
           </geometry>
         </collision>
