Commit message: Update URDF xacro files for Rizon 10

File: flexiv_description/urdf/flexiv_arm_materials.xacro (robot description, xacro)
@@ -3,14 +3,14 @@
   <xacro:macro name="flexiv_arm_materials">
     <material name="rizon_blue">
-      <color rgba="0. 0. 1. 0.5"/>
+      <color rgba="0.0 0.0 1.0 0.5"/>
     </material>
     <material name="rizon_light_grey">
-      <color rgba="0.9 0.9 0.9 1"/>
+      <color rgba="0.7 0.7 0.7 1.0"/>
     </material>
     <material name="rizon_dark_grey">
-      <color rgba="0.2 0.2 0.2 1"/>
+      <color rgba="0.4 0.4 0.4 1.0"/>
     </material>
     <material name="rizon_white">
-      <color rgba="1 1 1 1"/>
+      <color rgba="1.0 1.0 1.0 1.0"/>
     </material>
   </xacro:macro>

File: flexiv_description/urdf/rizon.urdf.xacro (robot description, xacro)
@@ -1,18 +1,25 @@
 <?xml version="1.0" encoding="utf-8"?>
-<robot xmlns:xacro="http://www.ros.org/wiki/xacro" name="rizon4">
+<robot xmlns:xacro="http://www.ros.org/wiki/xacro" name="$(arg name)">
   <!-- Enable setting arguments from the launch file -->
+  <xacro:arg name="name" default="rizon"/>
+  <!-- 'rizon_type' values: rizon4, rizon4s, rizon10 -->
+  <xacro:arg name="rizon_type" default="rizon4"/>
+  <!-- import main macro -->
+  <xacro:include filename="$(find flexiv_description)/urdf/rizon_macro.xacro"/>
+  <!-- parameters -->
+  <xacro:arg name="prefix" default="" />
   <xacro:arg name="robot_ip" default="" />
   <xacro:arg name="local_ip" default="" />
-  <xacro:arg name="rizon_type" default="rizon4"/>
   <xacro:arg name="use_fake_hardware" default="false" />
   <xacro:arg name="fake_sensor_commands" default="false" />
   <xacro:arg name="initial_positions_file" default="$(find flexiv_description)/config/initial_positions.yaml"/>
-  <xacro:arg name="prefix" default="" />
-  <xacro:include filename="$(find flexiv_description)/urdf/rizon_joints_links.xacro" />
-  <xacro:rizon_joints_links rizon_type="$(arg rizon_type)" prefix="$(arg prefix)" mesh_prefix_path="package://flexiv_description/" />
-  <xacro:include filename="$(find flexiv_description)/urdf/flexiv_arm_materials.xacro" />
-  <xacro:flexiv_arm_materials />
-  <xacro:include filename="$(find flexiv_description)/urdf/rizon.ros2_control.xacro"/>
-  <xacro:rizon_ros2_control prefix="$(arg prefix)" robot_ip="$(arg robot_ip)" local_ip="$(arg local_ip)" use_fake_hardware="$(arg use_fake_hardware)" fake_sensor_commands="$(arg fake_sensor_commands)" initial_positions_file="$(arg initial_positions_file)"/>
-  <!-- Used for fixing robot -->
+  <xacro:rizon_robot
+    rizon_type="$(arg rizon_type)"
+    prefix="$(arg prefix)"
+    robot_ip="$(arg robot_ip)"
+    local_ip="$(arg local_ip)"
+    use_fake_hardware="$(arg use_fake_hardware)"
+    fake_sensor_commands="$(arg fake_sensor_commands)"
+    initial_positions_file="$(arg initial_positions_file)">
+  </xacro:rizon_robot>
 </robot>

File: flexiv_description/urdf/rizon10_joints_links.xacro (robot description, xacro)
@@ -2,10 +2,10 @@
 <robot xmlns:xacro="http://www.ros.org/wiki/xacro">
   <!--
-    rizon_type = "rizon4", "rizon4s"
+    rizon_type = "rizon10"
     prefix = "", "left_"
     mesh_prefix_path = "", "package://flexiv_description/"
     NOTE: accurate kinematic but approximated dynamics parameters
   -->
-  <xacro:macro name="rizon_joints_links" params="rizon_type prefix mesh_prefix_path">
+  <xacro:macro name="rizon10_joints_links" params="rizon_type prefix mesh_prefix_path">
     <!-- JOINTS-->
     <joint name="${prefix}base_joint" type="fixed">
@@ -17,59 +17,54 @@
       <parent link="${prefix}base_link"/>
       <child link="${prefix}link1"/>
-      <origin xyz="0.0 0.0 0.155" rpy="0 0 ${pi}"/>
-      <axis xyz="0 0 1"/>
-      <limit effort="123" lower="-2.7925" upper="2.7925" velocity="2.0944"/>
+      <origin xyz="0.0 0.0 0.21" rpy="0 0 ${-pi}"/>
+      <axis xyz="0 0 1"/>
+      <limit effort="261" lower="-2.7925" upper="2.7925" velocity="1.7453" />
     </joint>
     <joint name="${prefix}joint2" type="revolute">
       <parent link="${prefix}link1"/>
       <child link="${prefix}link2"/>
-      <origin xyz="0.0 0.03 0.210" rpy="0 0 0"/>
+      <origin xyz="0.0 0.0675 0.24" rpy="0.0 0.0 0.0"/>
       <axis xyz="0 1 0"/>
-      <limit effort="123" lower="-2.2689" upper="2.2689" velocity="2.0944"/>
+      <limit effort="261" lower="-2.6704" upper="2.6704" velocity="1.7453" />
     </joint>
     <joint name="${prefix}joint3" type="revolute">
       <parent link="${prefix}link2"/>
       <child link="${prefix}link3"/>
-      <origin xyz="0.0 0.035 0.205" rpy="0 0 0"/>
-      <axis xyz="0 0 1"/>
-      <limit effort="64" lower="-2.9671" upper="2.9671" velocity="2.4435"/>
+      <origin xyz="0.0 0.0625 0.2275" rpy="0.0 0.0 0.0"/>
+      <axis xyz="0 0 1"/>
+      <limit effort="123" lower="-2.7925" upper="2.7925" velocity="2.0944" />
     </joint>
     <joint name="${prefix}joint4" type="revolute">
       <parent link="${prefix}link3"/>
       <child link="${prefix}link4"/>
-      <origin xyz="-0.02 -0.03 0.19" rpy="0 0 ${-pi}"/>
+      <origin xyz="0.0 -0.0625 0.2225" rpy="0 0 ${-pi}"/>
       <axis xyz="0 1 0"/>
-      <limit effort="64" lower="-1.8675" upper="2.6878" velocity="2.4435" />
+      <limit effort="123" lower="-2.7053" upper="2.7053" velocity="2.0944" />
     </joint>
     <joint name="${prefix}joint5" type="revolute">
       <parent link="${prefix}link4"/>
       <child link="${prefix}link5"/>
-      <origin xyz="-0.02 0.025 0.195" rpy="0 0 ${-pi}"/>
-      <axis xyz="0 0 1"/>
-      <limit effort="39" lower="-2.9671" upper="2.9671" velocity="4.8869" />
+      <origin xyz="0.0 0.0575 0.205" rpy="0 0 ${-pi}"/>
+      <axis xyz="0 0 1"/>
+      <limit effort="57" lower="-2.9671" upper="2.9671" velocity="3.8397" />
     </joint>
     <joint name="${prefix}joint6" type="revolute">
       <parent link="${prefix}link5"/>
       <child link="${prefix}link6"/>
-      <origin xyz="0.0 0.03 0.19" rpy="0 0 0"/>
+      <origin xyz="0.0 0.03 0.19" rpy="0.0 0.0 0.0"/>
       <axis xyz="0 1 0"/>
-      <limit effort="39" lower="-1.3963" upper="4.5379" velocity="4.8869" />
+      <limit effort="57" lower="-1.3963" upper="4.5379" velocity="3.8397" />
     </joint>
     <joint name="${prefix}joint7" type="revolute">
       <parent link="${prefix}link6"/>
       <child link="${prefix}link7"/>
-      <origin xyz="-0.055 0.070 0.11" rpy="0 ${-pi/2} 0"/>
-      <axis xyz="0 0 1"/>
-      <limit effort="39" lower="-2.9671" upper="2.9671" velocity="4.8869" />
+      <origin xyz="-0.015 0.073 0.11" rpy="0 ${-pi/2} 0"/>
+      <axis xyz="0 0 1"/>
+      <limit effort="57" lower="-2.9671" upper="2.9671" velocity="3.8397" />
     </joint>
     <joint name="${prefix}link7_to_flange" type="fixed">
       <parent link="${prefix}link7"/>
       <child link="${prefix}flange"/>
-      <xacro:if value="${rizon_type=='rizon4'}">
-        <origin xyz="0.0 0.0 0.081" rpy="0 0 ${-pi}"/>
-      </xacro:if>
-      <xacro:if value="${rizon_type=='rizon4s'}">
-        <origin xyz="0.0 0.0 0.124" rpy="0 0 ${-pi}"/>
-      </xacro:if>
+      <origin xyz="0.0 0.0 0.081" rpy="0 0 ${-pi}"/>
     </joint>
     <!-- LINKS -->
@@ -78,7 +73,7 @@
     <link name="${prefix}base_link">
       <inertial>
-        <mass value="3.7" />
-        <origin rpy="0 0 0" xyz="0.0 -0.0 0.09" />
-        <inertia ixx="0.019" ixy="0.0" ixz="0.0" iyy="0.02" iyz="0.0" izz="0.009" />
+        <mass value="9.2" />
+        <origin rpy="0 0 0" xyz="0.0 -0.0 0.13" />
+        <inertia ixx="0.08" ixy="0.0" ixz="-0.0" iyy="0.08" iyz="0.0" izz="0.04" />
       </inertial>
       <visual>
@@ -87,4 +82,5 @@
           <mesh filename="${mesh_prefix_path}meshes/${rizon_type}/visual/link0.obj" />
         </geometry>
+        <material name="rizon_light_grey" />
       </visual>
       <collision>
@@ -97,7 +93,7 @@
     <link name="${prefix}link1">
       <inertial>
-        <mass value="3.7" />
-        <origin rpy="0 0 0" xyz="0.0 0.01 0.15" />
-        <inertia ixx="0.028" ixy="0.0" ixz="0.0" iyy="0.027" iyz="0.002" izz="0.008" />
+        <mass value="9.7" />
+        <origin rpy="0 0 0" xyz="0.0 0.03 0.16" />
+        <inertia ixx="0.18" ixy="0.0" ixz="0.0" iyy="0.17" iyz="0.02" izz="0.04" />
       </inertial>
       <visual>
@@ -106,4 +102,5 @@
           <mesh filename="${mesh_prefix_path}meshes/${rizon_type}/visual/link1.obj" />
         </geometry>
+        <material name="rizon_light_grey" />
       </visual>
       <collision>
@@ -116,7 +113,7 @@
     <link name="${prefix}link2">
       <inertial>
-        <mass value="2.7" />
-        <origin rpy="0 0 0" xyz="0.0 0.04 0.1" />
-        <inertia ixx="0.023" ixy="0.0" ixz="0.0" iyy="0.024" iyz="-0.0" izz="0.004" />
+        <mass value="6.2" />
+        <origin rpy="0 0 0" xyz="0.0 0.03 0.11" />
+        <inertia ixx="0.1" ixy="0.0" ixz="0.0" iyy="0.08" iyz="0.02" izz="0.03" />
       </inertial>
       <visual>
@@ -125,4 +122,5 @@
           <mesh filename="${mesh_prefix_path}meshes/${rizon_type}/visual/link2.obj" />
         </geometry>
+        <material name="rizon_dark_grey" />
       </visual>
       <collision>
@@ -135,7 +133,7 @@
     <link name="${prefix}link3">
       <inertial>
-        <mass value="2.4" />
-        <origin rpy="0 0 0" xyz="-0.01 -0.0 0.13" />
-        <inertia ixx="0.014" ixy="0.0" ixz="-0.001" iyy="0.014" iyz="-0.001" izz="0.004" />
+        <mass value="4.6" />
+        <origin rpy="0 0 0" xyz="0.0 -0.03 0.17" />
+        <inertia ixx="0.04" ixy="-0.0" ixz="-0.0" iyy="0.03" iyz="-0.01" izz="0.01" />
       </inertial>
       <visual>
@@ -144,4 +142,5 @@
           <mesh filename="${mesh_prefix_path}meshes/${rizon_type}/visual/link3.obj" />
         </geometry>
+        <material name="rizon_dark_grey" />
       </visual>
       <collision>
@@ -156,5 +155,5 @@
         <mass value="2.4" />
         <origin rpy="0 0 0" xyz="-0.01 0.03 0.1" />
-        <inertia ixx="0.018" ixy="0.0" ixz="-0.002" iyy="0.019" iyz="-0.001" izz="0.003" />
+        <inertia ixx="0.02" ixy="0.0" ixz="-0.0" iyy="0.02" iyz="-0.0" izz="0.0" />
       </inertial>
       <visual>
@@ -163,4 +162,5 @@
           <mesh filename="${mesh_prefix_path}meshes/${rizon_type}/visual/link4.obj" />
         </geometry>
+        <material name="rizon_dark_grey" />
       </visual>
       <collision>
@@ -175,5 +175,5 @@
         <mass value="2.4" />
         <origin rpy="0 0 0" xyz="0.0 0.0 0.13" />
-        <inertia ixx="0.014" ixy="0.0" ixz="0.0" iyy="0.013" iyz="0.001" izz="0.004" />
+        <inertia ixx="0.01" ixy="0.0" ixz="0.0" iyy="0.01" iyz="0.0" izz="0.0" />
       </inertial>
       <visual>
@@ -182,4 +182,5 @@
           <mesh filename="${mesh_prefix_path}meshes/${rizon_type}/visual/link5.obj" />
         </geometry>
+        <material name="rizon_dark_grey" />
       </visual>
       <collision>
@@ -192,7 +193,7 @@
     <link name="${prefix}link6">
       <inertial>
-        <mass value="2.1" />
-        <origin rpy="0 0 0" xyz="-0.01 0.06 0.07" />
-        <inertia ixx="0.008" ixy="-0.0" ixz="-0.001" iyy="0.009" iyz="0.002" izz="0.004" />
+        <mass value="2.3" />
+        <origin rpy="0 0 0" xyz="0.02 0.06 0.07" />
+        <inertia ixx="0.01" ixy="0.0" ixz="0.0" iyy="0.01" iyz="0.0" izz="0.0" />
       </inertial>
       <visual>
@@ -201,4 +202,5 @@
           <mesh filename="${mesh_prefix_path}meshes/${rizon_type}/visual/link6.obj" />
         </geometry>
+        <material name="rizon_dark_grey" />
       </visual>
       <collision>
@@ -210,42 +212,22 @@
     </link>
     <link name="${prefix}link7">
-      <xacro:if value="${rizon_type=='rizon4'}">
-        <inertial>
-          <mass value="0.8" />
-          <origin rpy="0 0 0" xyz="0.0 0.0 0.03" />
-          <inertia ixx="0.001" ixy="0.0" ixz="0.0" iyy="0.001" iyz="0.0" izz="0.001" />
-        </inertial>
-        <visual>
-          <origin xyz="0 0 0" rpy="0 0 0"/>
-          <geometry>
-            <mesh filename="${mesh_prefix_path}meshes/${rizon_type}/visual/link7.obj" />
-          </geometry>
-        </visual>
-        <collision>
-          <origin xyz="0 0 0" rpy="0 0 0"/>
-          <geometry>
-            <mesh filename="${mesh_prefix_path}meshes/${rizon_type}/collision/link7.stl" />
-          </geometry>
-        </collision>
-      </xacro:if>
-      <xacro:if value="${rizon_type=='rizon4s'}">
-        <inertial>
-          <mass value="1.4" />
-          <origin xyz="0.0 0.0 0.05" rpy="0 0 0"/>
-          <inertia ixx="0.003" iyy="0.003" izz="0.002" ixy="0.0" ixz="0.0" iyz="0.0"/>
-        </inertial>
-        <visual>
-          <origin xyz="0 0 0" rpy="0 0 0"/>
-          <geometry>
-            <mesh filename="${mesh_prefix_path}meshes/${rizon_type}/visual/link7.obj" />
-          </geometry>
-        </visual>
-        <collision>
-          <origin xyz="0 0 0" rpy="0 0 0"/>
-          <geometry>
-            <mesh filename="${mesh_prefix_path}meshes/${rizon_type}/collision/link7.stl" />
-          </geometry>
-        </collision>
-      </xacro:if>
+      <inertial>
+        <mass value="0.9" />
+        <origin rpy="0 0 0" xyz="0.0 -0.0 0.03" />
+        <inertia ixx="0.0" ixy="0.0" ixz="0.0" iyy="0.0" iyz="0.0" izz="0.0" />
+      </inertial>
+      <visual>
+        <origin xyz="0 0 0" rpy="0 0 0"/>
+        <geometry>
+          <mesh filename="${mesh_prefix_path}meshes/${rizon_type}/visual/link7.obj" />
+        </geometry>
+        <material name="rizon_dark_grey" />
+      </visual>
+      <collision>
+        <origin xyz="0 0 0" rpy="0 0 0"/>
+        <geometry>
+          <mesh filename="${mesh_prefix_path}meshes/${rizon_type}/collision/link7.stl" />
+        </geometry>
+      </collision>
     </link>
     <link name="${prefix}flange"/>

File: flexiv_description/urdf/rizon4.ros2_control.xacro (robot description, xacro)
@@ -1,5 +1,5 @@
 <?xml version="1.0"?>
 <robot xmlns:xacro="http://www.ros.org/wiki/xacro">
-  <xacro:macro name="rizon_ros2_control" params="prefix robot_ip local_ip use_fake_hardware:=^|false fake_sensor_commands:=^|false initial_positions_file">
+  <xacro:macro name="rizon4_ros2_control" params="prefix robot_ip local_ip use_fake_hardware:=^|false fake_sensor_commands:=^|false initial_positions_file">
     <xacro:property name="initial_positions" value="${load_yaml(initial_positions_file)['initial_positions']}"/>
     <ros2_control name="FlexivHardwareInterface" type="system">
