Commit message: Update urdf and ros2_control xacro files

File: flexiv_description/urdf/flexiv_arm.materials.xacro (robot description, xacro)
@@ -1,5 +1,4 @@
 <?xml version="1.0" ?>
 <robot xmlns:xacro="http://www.ros.org/wiki/xacro">
-  <xacro:macro name="flexiv_arm_materials">
     <material name="rizon_blue">
       <color rgba="0.0 0.0 1.0 0.5"/>
@@ -14,4 +13,3 @@
       <color rgba="1.0 1.0 1.0 1.0"/>
     </material>
-  </xacro:macro>
 </robot>

File: flexiv_description/urdf/rizon.urdf.xacro (robot description, xacro)
@@ -14,4 +14,6 @@
   <xacro:arg name="fake_sensor_commands" default="false" />
   <xacro:arg name="initial_positions_file" default="$(find flexiv_description)/config/initial_positions.yaml"/>
+  <!-- convert to property to use substitution in function -->
+  <xacro:property name="initial_positions_file" default="$(arg initial_positions_file)"/>
   <xacro:rizon_robot
     rizon_type="$(arg rizon_type)"
@@ -21,5 +23,5 @@
     use_fake_hardware="$(arg use_fake_hardware)"
     fake_sensor_commands="$(arg fake_sensor_commands)"
-    initial_positions_file="$(arg initial_positions_file)">
+    initial_positions="${xacro.load_yaml(initial_positions_file)}">
   </xacro:rizon_robot>
 </robot>

File: flexiv_description/urdf/rizon10.ros2_control.xacro (robot description, xacro)
@@ -1,11 +1,17 @@
 <?xml version="1.0"?>
 <robot xmlns:xacro="http://www.ros.org/wiki/xacro">
-  <xacro:macro name="rizon10_ros2_control" params="prefix robot_ip local_ip use_fake_hardware:=^|false fake_sensor_commands:=^|false initial_positions_file">
-    <xacro:property name="initial_positions" value="${load_yaml(initial_positions_file)['initial_positions']}"/>
+  <xacro:macro name="rizon10_ros2_control" params="
+    prefix
+    robot_ip
+    local_ip
+    use_fake_hardware:=false
+    fake_sensor_commands:=false
+    initial_positions:=${dict(joint1=0.0,joint2=-0.69813,joint3=0.0,joint4=1.570796,joint5=0.0,joint6=0.69813,joint7=0.0)}
+    ">
     <ros2_control name="FlexivHardwareInterface" type="system">
       <hardware>
         <xacro:if value="${use_fake_hardware}">
-          <plugin>fake_components/GenericSystem</plugin>
-          <param name="fake_sensor_commands">${fake_sensor_commands}</param>
+          <plugin>mock_components/GenericSystem</plugin>
+          <param name="mock_sensor_commands">${fake_sensor_commands}</param>
           <param name="state_following_offset">0.0</param>
         </xacro:if>
@@ -26,8 +32,10 @@
         </command_interface>
         <command_interface name="effort"/>
-        <state_interface name="position"/>
+        <state_interface name="position">
+          <!-- initial position for the FakeSystem -->
+          <param name="initial_value">${initial_positions['joint1']}</param>
+        </state_interface>
         <state_interface name="velocity"/>
         <state_interface name="effort"/>
-        <param name="initial_position">${initial_positions['joint1']}</param>        <!-- initial position for the FakeSystem -->
       </joint>
       <joint name="${prefix}joint2">
@@ -41,8 +49,10 @@
         </command_interface>
         <command_interface name="effort"/>
-        <state_interface name="position"/>
+        <state_interface name="position">
+          <!-- initial position for the FakeSystem -->
+          <param name="initial_value">${initial_positions['joint2']}</param>
+        </state_interface>
         <state_interface name="velocity"/>
         <state_interface name="effort"/>
-        <param name="initial_position">${initial_positions['joint2']}</param>        <!-- initial position for the FakeSystem -->
       </joint>
       <joint name="${prefix}joint3">
@@ -56,8 +66,10 @@
         </command_interface>
         <command_interface name="effort"/>
-        <state_interface name="position"/>
+        <state_interface name="position">
+          <!-- initial position for the FakeSystem -->
+          <param name="initial_value">${initial_positions['joint3']}</param>
+        </state_interface>
         <state_interface name="velocity"/>
         <state_interface name="effort"/>
-        <param name="initial_position">${initial_positions['joint3']}</param>        <!-- initial position for the FakeSystem -->
       </joint>
       <joint name="${prefix}joint4">
@@ -71,8 +83,10 @@
         </command_interface>
         <command_interface name="effort"/>
-        <state_interface name="position"/>
+        <state_interface name="position">
+          <!-- initial position for the FakeSystem -->
+          <param name="initial_value">${initial_positions['joint4']}</param>
+        </state_interface>
         <state_interface name="velocity"/>
         <state_interface name="effort"/>
-        <param name="initial_position">${initial_positions['joint4']}</param>        <!-- initial position for the FakeSystem -->
       </joint>
       <joint name="${prefix}joint5">
@@ -86,8 +100,10 @@
         </command_interface>
         <command_interface name="effort"/>
-        <state_interface name="position"/>
+        <state_interface name="position">
+          <!-- initial position for the FakeSystem -->
+          <param name="initial_value">${initial_positions['joint5']}</param>
+        </state_interface>
         <state_interface name="velocity"/>
         <state_interface name="effort"/>
-        <param name="initial_position">${initial_positions['joint5']}</param>        <!-- initial position for the FakeSystem -->
       </joint>
       <joint name="${prefix}joint6">
@@ -101,8 +117,10 @@
         </command_interface>
         <command_interface name="effort"/>
-        <state_interface name="position"/>
+        <state_interface name="position">
+          <!-- initial position for the FakeSystem -->
+          <param name="initial_value">${initial_positions['joint6']}</param>
+        </state_interface>
         <state_interface name="velocity"/>
         <state_interface name="effort"/>
-        <param name="initial_position">${initial_positions['joint6']}</param>        <!-- initial position for the FakeSystem -->
       </joint>
       <joint name="${prefix}joint7">
@@ -116,8 +134,10 @@
         </command_interface>
         <command_interface name="effort"/>
-        <state_interface name="position"/>
+        <state_interface name="position">
+          <!-- initial position for the FakeSystem -->
+          <param name="initial_value">${initial_positions['joint7']}</param>
+        </state_interface>
         <state_interface name="velocity"/>
         <state_interface name="effort"/>
-        <param name="initial_position">${initial_positions['joint7']}</param>        <!-- initial position for the FakeSystem -->
       </joint>
       <sensor name="${prefix}force_torque_sensor">

File: flexiv_description/urdf/rizon4.ros2_control.xacro (robot description, xacro)
@@ -1,11 +1,17 @@
 <?xml version="1.0"?>
 <robot xmlns:xacro="http://www.ros.org/wiki/xacro">
-  <xacro:macro name="rizon4_ros2_control" params="prefix robot_ip local_ip use_fake_hardware:=^|false fake_sensor_commands:=^|false initial_positions_file">
-    <xacro:property name="initial_positions" value="${load_yaml(initial_positions_file)['initial_positions']}"/>
+  <xacro:macro name="rizon4_ros2_control" params="
+    prefix
+    robot_ip
+    local_ip
+    use_fake_hardware:=false
+    fake_sensor_commands:=false
+    initial_positions:=${dict(joint1=0.0,joint2=-0.69813,joint3=0.0,joint4=1.570796,joint5=0.0,joint6=0.69813,joint7=0.0)}
+    ">
     <ros2_control name="FlexivHardwareInterface" type="system">
       <hardware>
         <xacro:if value="${use_fake_hardware}">
-          <plugin>fake_components/GenericSystem</plugin>
-          <param name="fake_sensor_commands">${fake_sensor_commands}</param>
+          <plugin>mock_components/GenericSystem</plugin>
+          <param name="mock_sensor_commands">${fake_sensor_commands}</param>
           <param name="state_following_offset">0.0</param>
         </xacro:if>
@@ -26,8 +32,10 @@
         </command_interface>
         <command_interface name="effort"/>
-        <state_interface name="position"/>
+        <state_interface name="position">
+          <!-- initial position for the FakeSystem -->
+          <param name="initial_value">${initial_positions['joint1']}</param>
+        </state_interface>
         <state_interface name="velocity"/>
         <state_interface name="effort"/>
-        <param name="initial_position">${initial_positions['joint1']}</param>        <!-- initial position for the FakeSystem -->
       </joint>
       <joint name="${prefix}joint2">
@@ -41,8 +49,10 @@
         </command_interface>
         <command_interface name="effort"/>
-        <state_interface name="position"/>
+        <state_interface name="position">
+          <!-- initial position for the FakeSystem -->
+          <param name="initial_value">${initial_positions['joint2']}</param>
+        </state_interface>
         <state_interface name="velocity"/>
         <state_interface name="effort"/>
-        <param name="initial_position">${initial_positions['joint2']}</param>        <!-- initial position for the FakeSystem -->
       </joint>
       <joint name="${prefix}joint3">
@@ -56,8 +66,10 @@
         </command_interface>
         <command_interface name="effort"/>
-        <state_interface name="position"/>
+        <state_interface name="position">
+          <!-- initial position for the FakeSystem -->
+          <param name="initial_value">${initial_positions['joint3']}</param>
+        </state_interface>
         <state_interface name="velocity"/>
         <state_interface name="effort"/>
-        <param name="initial_position">${initial_positions['joint3']}</param>        <!-- initial position for the FakeSystem -->
       </joint>
       <joint name="${prefix}joint4">
@@ -71,8 +83,10 @@
         </command_interface>
         <command_interface name="effort"/>
-        <state_interface name="position"/>
+        <state_interface name="position">
+          <!-- initial position for the FakeSystem -->
+          <param name="initial_value">${initial_positions['joint4']}</param>
+        </state_interface>
         <state_interface name="velocity"/>
         <state_interface name="effort"/>
-        <param name="initial_position">${initial_positions['joint4']}</param>        <!-- initial position for the FakeSystem -->
       </joint>
       <joint name="${prefix}joint5">
@@ -86,8 +100,10 @@
         </command_interface>
         <command_interface name="effort"/>
-        <state_interface name="position"/>
+        <state_interface name="position">
+          <!-- initial position for the FakeSystem -->
+          <param name="initial_value">${initial_positions['joint5']}</param>
+        </state_interface>
         <state_interface name="velocity"/>
         <state_interface name="effort"/>
-        <param name="initial_position">${initial_positions['joint5']}</param>        <!-- initial position for the FakeSystem -->
       </joint>
       <joint name="${prefix}joint6">
@@ -101,8 +117,10 @@
         </command_interface>
         <command_interface name="effort"/>
-        <state_interface name="position"/>
+        <state_interface name="position">
+          <!-- initial position for the FakeSystem -->
+          <param name="initial_value">${initial_positions['joint6']}</param>
+        </state_interface>
         <state_interface name="velocity"/>
         <state_interface name="effort"/>
-        <param name="initial_position">${initial_positions['joint6']}</param>        <!-- initial position for the FakeSystem -->
       </joint>
       <joint name="${prefix}joint7">
@@ -116,8 +134,10 @@
         </command_interface>
         <command_interface name="effort"/>
-        <state_interface name="position"/>
+        <state_interface name="position">
+          <!-- initial position for the FakeSystem -->
+          <param name="initial_value">${initial_positions['joint7']}</param>
+        </state_interface>
         <state_interface name="velocity"/>
         <state_interface name="effort"/>
-        <param name="initial_position">${initial_positions['joint7']}</param>        <!-- initial position for the FakeSystem -->
       </joint>
       <sensor name="${prefix}force_torque_sensor">

File: flexiv_description/urdf/rizon_macro.xacro (robot description, xacro)
@@ -8,16 +8,18 @@
     use_fake_hardware:=false
     fake_sensor_commands:=false
-    initial_positions_file">
-    <xacro:include filename="$(find flexiv_description)/urdf/flexiv_arm_materials.xacro" />
+    initial_positions:=${dict(joint1=0.0,joint2=-0.69813,joint3=0.0,joint4=1.570796,joint5=0.0,joint6=0.69813,joint7=0.0)}
+    ">
+    <!-- Import Rviz colors -->
+    <xacro:include filename="$(find flexiv_description)/urdf/flexiv_arm.materials.xacro" />
     <!-- Rizon 4 or 4s-->
     <xacro:if value="${rizon_type=='rizon4' or rizon_type=='rizon4s'}">
       <xacro:include filename="$(find flexiv_description)/urdf/rizon4_joints_links.xacro" />
-      <xacro:rizon4_joints_links rizon_type="$(arg rizon_type)" prefix="$(arg prefix)" mesh_prefix_path="package://flexiv_description/" />
+      <xacro:rizon4_joints_links rizon_type="${rizon_type}" prefix="${prefix}" mesh_prefix_path="package://flexiv_description/" />
       <!-- ros2 control include -->
       <xacro:include filename="$(find flexiv_description)/urdf/rizon4.ros2_control.xacro"/>
-      <xacro:rizon4_ros2_control prefix="$(arg prefix)" robot_ip="$(arg robot_ip)"
-        local_ip="$(arg local_ip)" use_fake_hardware="$(arg use_fake_hardware)"
-        fake_sensor_commands="$(arg fake_sensor_commands)"
-        initial_positions_file="$(arg initial_positions_file)"
+      <xacro:rizon4_ros2_control prefix="${prefix}" robot_ip="${robot_ip}"
+        local_ip="${local_ip}" use_fake_hardware="${use_fake_hardware}"
+        fake_sensor_commands="${fake_sensor_commands}"
+        initial_positions="${initial_positions}"
         />
     </xacro:if>
@@ -25,11 +27,11 @@
     <xacro:if value="${rizon_type=='rizon10'}">
       <xacro:include filename="$(find flexiv_description)/urdf/rizon10_joints_links.xacro" />
-      <xacro:rizon10_joints_links rizon_type="$(arg rizon_type)" prefix="$(arg prefix)" mesh_prefix_path="package://flexiv_description/" />
+      <xacro:rizon10_joints_links rizon_type="${rizon_type}" prefix="${prefix}" mesh_prefix_path="package://flexiv_description/" />
       <!-- ros2 control include -->
       <xacro:include filename="$(find flexiv_description)/urdf/rizon10.ros2_control.xacro"/>
-      <xacro:rizon10_ros2_control prefix="$(arg prefix)" robot_ip="$(arg robot_ip)"
-        local_ip="$(arg local_ip)" use_fake_hardware="$(arg use_fake_hardware)"
-        fake_sensor_commands="$(arg fake_sensor_commands)"
-        initial_positions_file="$(arg initial_positions_file)"
+      <xacro:rizon10_ros2_control prefix="${prefix}" robot_ip="${robot_ip}"
+        local_ip="${local_ip}" use_fake_hardware="${use_fake_hardware}"
+        fake_sensor_commands="${fake_sensor_commands}"
+        initial_positions="${initial_positions}"
         />
     </xacro:if>
