Commit message: fix

File: flexiv_description/urdf/grav.urdf (robot description, URDF)
Before this commit: robot flexiv_GN01, 14 links, 13 joints
Links:
- link base_link: geometry collision mesh filename=package://flexiv_description/meshes/grav/collision/base.stl scale=0.001 0.001 0.001; visual mesh filename=package://flexiv_description/meshes/grav/visual/base.stl scale=0.001 0.001 0.001
- link left_finger_mount: geometry visual mesh filename=package://flexiv_description/meshes/grav/visual/finger_moun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 scale=0.001 0.001 0.001
- link left_finger_tip: geometry collision mesh filename=package://flexiv_description/meshes/grav/collision/finger_t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 scale=0.001 0.001 0.001; visual mesh filename=package://flexiv_description/meshes/grav/visual/finger_tip.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 scale=0.001 0.001 0.001
- link left_inner_bar: geometry visual mesh filename=package://flexiv_description/meshes/grav/visual/inner_bar.s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 scale=0.001 0.001 0.001
- link left_outer_bar: geometry visual mesh filename=package://flexiv_description/meshes/grav/visual/outer_bar.s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 scale=0.001 0.001 0.001
- link right_finger_mount: geometry visual mesh filename=package://flexiv_description/meshes/grav/visual/finger_moun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 scale=0.001 0.001 0.001
- link right_finger_tip: geometry collision mesh filename=package://flexiv_description/meshes/grav/collision/finger_t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 scale=0.001 0.001 0.001; visual mesh filename=package://flexiv_description/meshes/grav/visual/finger_tip.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 scale=0.001 0.001 0.001
- link right_inner_bar: geometry visual mesh filename=package://flexiv_description/meshes/grav/visual/inner_bar.s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 scale=0.001 0.001 0.001
- link right_outer_bar: geometry visual mesh filename=package://flexiv_description/meshes/grav/visual/outer_bar.s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 scale=0.001 0.001 0.001
