Commit message: Update links material color

File: flexiv_description/urdf/rizon10_joints_links.xacro (robot description, xacro)
@@ -82,5 +82,5 @@
           <mesh filename="${mesh_prefix_path}meshes/${rizon_type}/visual/link0.obj" />
         </geometry>
-        <material name="rizon_light_grey" />
+        <material name="rizon_dark_grey" />
       </visual>
       <collision>
@@ -102,5 +102,5 @@
           <mesh filename="${mesh_prefix_path}meshes/${rizon_type}/visual/link1.obj" />
         </geometry>
-        <material name="rizon_light_grey" />
+        <material name="rizon_dark_grey" />
       </visual>
       <collision>

Commit message: Fix static or unrealistic inertia value

File: flexiv_description/urdf/rizon10_joints_links.xacro (robot description, xacro)
@@ -75,5 +75,5 @@
         <mass value="9.2" />
         <origin rpy="0 0 0" xyz="0.0 -0.0 0.13" />
-        <inertia ixx="0.08" ixy="0.0" ixz="-0.0" iyy="0.08" iyz="0.0" izz="0.04" />
+        <inertia ixx="0.08" ixy="0.0" ixz="-0.0003" iyy="0.08" iyz="0.001" izz="0.04" />
       </inertial>
       <visual>
@@ -95,5 +95,5 @@
         <mass value="9.7" />
         <origin rpy="0 0 0" xyz="0.0 0.03 0.16" />
-        <inertia ixx="0.18" ixy="0.0" ixz="0.0" iyy="0.17" iyz="0.02" izz="0.04" />
+        <inertia ixx="0.18" ixy="0.0002" ixz="0.0001" iyy="0.17" iyz="0.02" izz="0.04" />
       </inertial>
       <visual>
@@ -115,5 +115,5 @@
         <mass value="6.2" />
         <origin rpy="0 0 0" xyz="0.0 0.03 0.11" />
-        <inertia ixx="0.1" ixy="0.0" ixz="0.0" iyy="0.08" iyz="0.02" izz="0.03" />
+        <inertia ixx="0.1" ixy="0.0" ixz="0.0001" iyy="0.08" iyz="0.02" izz="0.03" />
       </inertial>
       <visual>
@@ -135,5 +135,5 @@
         <mass value="4.6" />
         <origin rpy="0 0 0" xyz="0.0 -0.03 0.17" />
-        <inertia ixx="0.04" ixy="-0.0" ixz="-0.0" iyy="0.03" iyz="-0.01" izz="0.01" />
+        <inertia ixx="0.03" ixy="-0.0001" ixz="-0.0001" iyy="0.03" iyz="-0.006" izz="0.01" />
       </inertial>
       <visual>
@@ -155,5 +155,5 @@
         <mass value="2.4" />
         <origin rpy="0 0 0" xyz="-0.01 0.03 0.1" />
-        <inertia ixx="0.02" ixy="0.0" ixz="-0.0" iyy="0.02" iyz="-0.0" izz="0.0" />
+        <inertia ixx="0.03" ixy="0.0" ixz="-0.0001" iyy="0.03" iyz="0.0007" izz="0.005" />
       </inertial>
       <visual>
@@ -175,5 +175,5 @@
         <mass value="2.4" />
         <origin rpy="0 0 0" xyz="0.0 0.0 0.13" />
-        <inertia ixx="0.01" ixy="0.0" ixz="0.0" iyy="0.01" iyz="0.0" izz="0.0" />
+        <inertia ixx="0.01" ixy="0.0" ixz="0.0" iyy="0.01" iyz="0.001" izz="0.004" />
       </inertial>
       <visual>
@@ -195,5 +195,5 @@
         <mass value="2.3" />
         <origin rpy="0 0 0" xyz="0.02 0.06 0.07" />
-        <inertia ixx="0.01" ixy="0.0" ixz="0.0" iyy="0.01" iyz="0.0" izz="0.0" />
+        <inertia ixx="0.01" ixy="0.0003" ixz="0.001" iyy="0.01" iyz="0.002" izz="0.004" />
       </inertial>
       <visual>
@@ -215,5 +215,5 @@
         <mass value="0.9" />
         <origin rpy="0 0 0" xyz="0.0 -0.0 0.03" />
-        <inertia ixx="0.0" ixy="0.0" ixz="0.0" iyy="0.0" iyz="0.0" izz="0.0" />
+        <inertia ixx="0.001" ixy="0.0" ixz="0.0" iyy="0.001" iyz="0.0" izz="0.001" />
       </inertial>
       <visual>

File: flexiv_description/urdf/rizon4_joints_links.xacro (robot description, xacro)
@@ -80,5 +80,5 @@
         <mass value="3.7" />
         <origin rpy="0 0 0" xyz="0.0 -0.0 0.09" />
-        <inertia ixx="0.02" ixy="0.0" ixz="0.0" iyy="0.02" iyz="0.0" izz="0.01" />
+        <inertia ixx="0.02" ixy="0.0" ixz="0.0" iyy="0.02" iyz="0.0001" izz="0.009" />
       </inertial>
       <visual>
@@ -100,5 +100,5 @@
         <mass value="3.7" />
         <origin rpy="0 0 0" xyz="0.0 0.01 0.15" />
-        <inertia ixx="0.03" ixy="0.0" ixz="0.0" iyy="0.03" iyz="0.0" izz="0.01" />
+        <inertia ixx="0.03" ixy="0.0" ixz="0.0" iyy="0.03" iyz="0.002" izz="0.008" />
       </inertial>
       <visual>
@@ -120,5 +120,5 @@
         <mass value="2.7" />
         <origin rpy="0 0 0" xyz="0.0 0.04 0.1" />
-        <inertia ixx="0.02" ixy="0.0" ixz="0.0" iyy="0.02" iyz="-0.0" izz="0.0" />
+        <inertia ixx="0.02" ixy="0.0" ixz="0.0" iyy="0.02" iyz="-0.0003" izz="0.004" />
       </inertial>
       <visual>
@@ -140,5 +140,5 @@
         <mass value="2.4" />
         <origin rpy="0 0 0" xyz="-0.01 -0.0 0.13" />
-        <inertia ixx="0.01" ixy="0.0" ixz="-0.0" iyy="0.01" iyz="-0.0" izz="0.0" />
+        <inertia ixx="0.01" ixy="0.00" ixz="-0.001" iyy="0.01" iyz="-0.0007" izz="0.004" />
       </inertial>
       <visual>
@@ -160,5 +160,5 @@
         <mass value="2.4" />
         <origin rpy="0 0 0" xyz="-0.01 0.03 0.1" />
-        <inertia ixx="0.02" ixy="0.0" ixz="-0.0" iyy="0.02" iyz="-0.0" izz="0.0" />
+        <inertia ixx="0.02" ixy="0.00" ixz="-0.002" iyy="0.02" iyz="-0.001" izz="0.003" />
       </inertial>
       <visual>
@@ -180,5 +180,5 @@
         <mass value="2.4" />
         <origin rpy="0 0 0" xyz="0.0 0.0 0.13" />
-        <inertia ixx="0.01" ixy="0.0" ixz="0.0" iyy="0.01" iyz="0.0" izz="0.0" />
+        <inertia ixx="0.01" ixy="0.0" ixz="0.0" iyy="0.01" iyz="0.001" izz="0.004" />
       </inertial>
       <visual>
@@ -200,5 +200,5 @@
         <mass value="2.1" />
         <origin rpy="0 0 0" xyz="-0.01 0.06 0.07" />
-        <inertia ixx="0.01" ixy="-0.0" ixz="-0.001" iyy="0.01" iyz="0.0" izz="0.0" />
+        <inertia ixx="0.01" ixy="-0.000" ixz="-0.001" iyy="0.01" iyz="0.002" izz="0.004" />
       </inertial>
       <visual>
@@ -221,5 +221,5 @@
           <mass value="0.8" />
           <origin rpy="0 0 0" xyz="0.0 0.0 0.03" />
-          <inertia ixx="0.0" ixy="0.0" ixz="0.0" iyy="0.0" iyz="0.0" izz="0.0" />
+          <inertia ixx="0.001" ixy="0.0" ixz="0.0" iyy="0.001" iyz="0.0" izz="0.001" />
         </inertial>
         <visual>
@@ -241,5 +241,5 @@
           <mass value="1.4" />
           <origin xyz="0.0 0.0 0.05" rpy="0 0 0"/>
-          <inertia ixx="0.0" iyy="0.0" izz="0.0" ixy="0.0" ixz="0.0" iyz="0.0"/>
+          <inertia ixx="0.001" ixy="0.0" ixz="0.0" iyy="0.001" iyz="0.0" izz="0.001" />
         </inertial>
         <visual>

Commit message: Update Rizon10 and Rizon10s URDF xacro

File: flexiv_description/urdf/rizon10_joints_links.xacro (robot description, xacro)
@@ -1,7 +1,7 @@
-<?xml version="1.0" ?>
+<?xml version="1.0"?>
 <robot xmlns:xacro="http://www.ros.org/wiki/xacro">
   <!--
-    rizon_type = "rizon10", "rizon10s"
-    prefix = "", "left_"
+    rizon_type = "Rizon10", "Rizon10s"
+    prefix = "Rizon10-123456_"
     mesh_prefix_path = "", "package://flexiv_description/"
     NOTE: accurate kinematic but approximated dynamics parameters
@@ -10,65 +10,79 @@
     <!-- JOINTS-->
     <joint name="${prefix}base_joint" type="fixed">
-      <parent link="world"/>
+      <parent link="world" />
       <child link="${prefix}base_link" />
-      <origin xyz="0.0 0.0 0.0" rpy="0.0 0.0 0.0"/>
+      <origin xyz="0.0 0.0 0.0" rpy="0.0 0.0 0.0" />
     </joint>
     <joint name="${prefix}joint1" type="revolute">
-      <parent link="${prefix}base_link"/>
-      <child link="${prefix}link1"/>
-      <origin xyz="0.0 0.0 0.21" rpy="0 0 ${-pi}"/>
-      <axis xyz="0 0 1"/>
-      <limit effort="261" lower="-2.7925" upper="2.7925" velocity="1.7453" />
+      <parent link="${prefix}base_link" />
+      <child link="${prefix}link1" />
+      <origin xyz="0.0 0.0 0.21" rpy="0 0 ${-pi}" />
+      <axis xyz="0 0 1" />
+      <limit effort="261" lower="-2.8798" upper="2.8798" velocity="1.7453" />
+      <safety_controller k_position="100.0" k_velocity="40.0" soft_lower_limit="-2.7925"
+        soft_upper_limit="2.7925" />
     </joint>
     <joint name="${prefix}joint2" type="revolute">
-      <parent link="${prefix}link1"/>
-      <child link="${prefix}link2"/>
-      <origin xyz="0.0 0.0675 0.24" rpy="0.0 0.0 0.0"/>
-      <axis xyz="0 1 0"/>
-      <limit effort="261" lower="-2.6704" upper="2.6704" velocity="1.7453" />
+      <parent link="${prefix}link1" />
+      <child link="${prefix}link2" />
+      <origin xyz="0.0 0.0675 0.24" rpy="0.0 0.0 0.0" />
+      <axis xyz="0 1 0" />
+      <limit effort="261" lower="-2.7576" upper="2.7576" velocity="1.7453" />
+      <safety_controller k_position="100.0" k_velocity="40.0" soft_lower_limit="-2.6704"
+        soft_upper_limit="2.6704" />
     </joint>
     <joint name="${prefix}joint3" type="revolute">
-      <parent link="${prefix}link2"/>
-      <child link="${prefix}link3"/>
-      <origin xyz="0.0 0.0625 0.2275" rpy="0.0 0.0 0.0"/>
-      <axis xyz="0 0 1"/>
+      <parent link="${prefix}link2" />
+      <child link="${prefix}link3" />
+      <origin xyz="0.0 0.0625 0.2275" rpy="0.0 0.0 0.0" />
+      <axis xyz="0 0 1" />
+      <limit effort="123" lower="-2.8798" upper="2.8798" velocity="2.0944" />
+      <safety_controller k_position="100.0" k_velocity="40.0" soft_lower_limit="-2.7925"
+        soft_upper_limit="2.7925" />
+    </joint>
+    <joint name="${prefix}joint4" type="revolute">
+      <parent link="${prefix}link3" />
+      <child link="${prefix}link4" />
+      <origin xyz="0.0 -0.0625 0.2225" rpy="0 0 ${-pi}" />
+      <axis xyz="0 1 0" />
       <limit effort="123" lower="-2.7925" upper="2.7925" velocity="2.0944" />
-    </joint>
-    <joint name="${prefix}joint4" type="revolute">
-      <parent link="${prefix}link3"/>
-      <child link="${prefix}link4"/>
-      <origin xyz="0.0 -0.0625 0.2225" rpy="0 0 ${-pi}"/>
-      <axis xyz="0 1 0"/>
-      <limit effort="123" lower="-2.7053" upper="2.7053" velocity="2.0944" />
+      <safety_controller k_position="100.0" k_velocity="40.0" soft_lower_limit="-2.7053"
+        soft_upper_limit="2.7053" />
     </joint>
     <joint name="${prefix}joint5" type="revolute">
-      <parent link="${prefix}link4"/>
-      <child link="${prefix}link5"/>
-      <origin xyz="0.0 0.0575 0.205" rpy="0 0 ${-pi}"/>
-      <axis xyz="0 0 1"/>
-      <limit effort="57" lower="-2.9671" upper="2.9671" velocity="3.8397" />
+      <parent link="${prefix}link4" />
+      <child link="${prefix}link5" />
+      <origin xyz="0.0 0.0575 0.205" rpy="0 0 ${-pi}" />
+      <axis xyz="0 0 1" />
+      <limit effort="57" lower="-3.0543" upper="3.0543" velocity="3.8397" />
+      <safety_controller k_position="100.0" k_velocity="40.0" soft_lower_limit="-2.9671"
+        soft_upper_limit="2.9671" />
     </joint>
     <joint name="${prefix}joint6" type="revolute">
-      <parent link="${prefix}link5"/>
-      <child link="${prefix}link6"/>
-      <origin xyz="0.0 0.03 0.19" rpy="0.0 0.0 0.0"/>
-      <axis xyz="0 1 0"/>
-      <limit effort="57" lower="-1.3963" upper="4.5379" velocity="3.8397" />
+      <parent link="${prefix}link5" />
+      <child link="${prefix}link6" />
+      <origin xyz="0.0 0.03 0.19" rpy="0.0 0.0 0.0" />
+      <axis xyz="0 1 0" />
+      <limit effort="57" lower="-1.4835" upper="4.6251" velocity="3.8397" />
+      <safety_controller k_position="100.0" k_velocity="40.0" soft_lower_limit="-1.3963"
+        soft_upper_limit="4.5379" />
     </joint>
     <joint name="${prefix}joint7" type="revolute">
-      <parent link="${prefix}link6"/>
-      <child link="${prefix}link7"/>
-      <origin xyz="-0.015 0.073 0.11" rpy="0 ${-pi/2} 0"/>
-      <axis xyz="0 0 1"/>
-      <limit effort="57" lower="-2.9671" upper="2.9671" velocity="3.8397" />
+      <parent link="${prefix}link6" />
+      <child link="${prefix}link7" />
+      <origin xyz="-0.015 0.073 0.11" rpy="0 ${-pi/2} 0" />
+      <axis xyz="0 0 1" />
+      <limit effort="57" lower="-3.0543" upper="3.0543" velocity="3.8397" />
+      <safety_controller k_position="100.0" k_velocity="40.0" soft_lower_limit="-2.9671"
+        soft_upper_limit="2.9671" />
     </joint>
     <joint name="${prefix}link7_to_flange" type="fixed">
-      <parent link="${prefix}link7"/>
-      <child link="${prefix}flange"/>
-      <xacro:if value="${rizon_type=='rizon10'}">
-        <origin xyz="0.0 0.0 0.081" rpy="0 0 ${-pi}"/>
+      <parent link="${prefix}link7" />
+      <child link="${prefix}flange" />
+      <xacro:if value="${rizon_type=='Rizon10'}">
+        <origin xyz="0.0 0.0 0.081" rpy="0 0 ${-pi}" />
       </xacro:if>
-      <xacro:if value="${rizon_type=='rizon10s'}">
-        <origin xyz="0.0 0.0 0.124" rpy="0 0 ${-pi}"/>
+      <xacro:if value="${rizon_type=='Rizon10s'}">
+        <origin xyz="0.0 0.0 0.124" rpy="0 0 ${-pi}" />
       </xacro:if>
     </joint>
@@ -78,27 +92,32 @@
     <link name="${prefix}base_link">
       <inertial>
-        <mass value="9.2" />
-        <origin rpy="0 0 0" xyz="0.0 -0.0 0.13" />
-        <inertia ixx="0.08" ixy="0.0" ixz="-0.0003" iyy="0.08" iyz="0.001" izz="0.04" />
-      </inertial>
-      <visual name="shell">
-        <origin xyz="0 0 0" rpy="0 0 0"/>
+        <mass value="8.1" />
+        <origin rpy="0 0 0" xyz="0.0 -0.0 0.12" />
+        <inertia ixx="0.06" ixy="0.0" ixz="-0.0003" iyy="0.06" iyz="0.001" izz="0.03" />
+      </inertial>
+      <visual name="shell">
+        <origin xyz="0 0 0" rpy="0 0 0" />
         <geometry>
           <mesh filename="${mesh_prefix_path}meshes/${rizon_type}/visual/link0.obj" />
         </geometry>
-        <material name="rizon_dark_grey" />
-      </visual>
-      <collision name="hull">
-        <origin xyz="0 0 0" rpy="0 0 0"/>
+      </visual>
+      <collision name="convex_mesh">
+        <origin xyz="0 0 0" rpy="0 0 0" />
         <geometry>
           <mesh filename="${mesh_prefix_path}meshes/${rizon_type}/collision/link0.stl" />
         </geometry>
       </collision>
+      <workspace>
+        <origin rpy="0 0 0" xyz="0 0 0.450" />
+        <geometry>
+          <sphere radius="0.955" />
+        </geometry>
+      </workspace>
     </link>
     <link name="${prefix}link1">
       <inertial>
-        <mass value="9.7" />
-        <origin rpy="0 0 0" xyz="0.0 0.03 0.16" />
-        <inertia ixx="0.18" ixy="0.0002" ixz="0.0001" iyy="0.17" iyz="0.02" izz="0.04" />
+        <mass value="9.5" />
+        <origin rpy="0 0 0" xyz="0.0 0.02 0.16" />
+        <inertia ixx="0.12" ixy="0.0" ixz="-0.0" iyy="0.11" iyz="0.01" izz="0.04" />
       </inertial>
       <visual name="shell">
@@ -107,14 +126,13 @@
           <mesh filename="${mesh_prefix_path}meshes/${rizon_type}/visual/link1.obj" />
         </geometry>
-        <material name="rizon_dark_grey" />
       </visual>
       <visual name="ring">
         <origin rpy="0 0 0" xyz="0 0 -0.0025" />
         <geometry>
-          <mesh filename="${mesh_prefix_path}meshes/${rizon_type}/visual/ring.obj" scale="0.079 0.079 0.002" />
-        </geometry>
-        <material name="rizon_white" />
-      </visual>
-      <collision name="hull">
+          <mesh filename="${mesh_prefix_path}meshes/${rizon_type}/visual/ring.obj"
+            scale="0.079 0.079 0.002" />
+        </geometry>
+      </visual>
+      <collision name="convex_mesh">
         <origin xyz="0 0 0" rpy="0 0 0" />
         <geometry>
@@ -125,24 +143,23 @@
     <link name="${prefix}link2">
       <inertial>
-        <mass value="6.2" />
-        <origin rpy="0 0 0" xyz="0.0 0.03 0.11" />
-        <inertia ixx="0.1" ixy="0.0" ixz="0.0001" iyy="0.08" iyz="0.02" izz="0.03" />
-      </inertial>
-      <visual name="shell">
-        <origin xyz="0 0 0" rpy="0 0 0"/>
+        <mass value="6.6" />
+        <origin rpy="0 0 0" xyz="-0.0 0.06 0.09" />
+        <inertia ixx="0.08" ixy="0.0" ixz="0.0" iyy="0.08" iyz="0.0" izz="0.01" />
+      </inertial>
+      <visual name="shell">
+        <origin xyz="0 0 0" rpy="0 0 0" />
         <geometry>
           <mesh filename="${mesh_prefix_path}meshes/${rizon_type}/visual/link2.obj" />
         </geometry>
-        <material name="rizon_dark_grey" />
-      </visual>
-      <visual name="ring">
-        <origin rpy="1.5707963 0 0" xyz="0 -0.0025 0" />
-        <geometry>
-          <mesh filename="${mesh_prefix_path}meshes/${rizon_type}/visual/ring.obj" scale="0.079 0.079 0.002" />
-        </geometry>
-        <material name="rizon_white" />
-      </visual>
-      <collision name="hull">
-        <origin xyz="0 0 0" rpy="0 0 0"/>
+      </visual>
+      <visual name="ring">
+        <origin rpy="${pi/2} 0 0" xyz="0 -0.0025 0" />
+        <geometry>
+          <mesh filename="${mesh_prefix_path}meshes/${rizon_type}/visual/ring.obj"
+            scale="0.079 0.079 0.002" />
+        </geometry>
+      </visual>
+      <collision name="convex_mesh">
+        <origin xyz="0 0 0" rpy="0 0 0" />
         <geometry>
           <mesh filename="${mesh_prefix_path}meshes/${rizon_type}/collision/link2.stl" />
@@ -152,7 +169,7 @@
     <link name="${prefix}link3">
       <inertial>
-        <mass value="4.6" />
-        <origin rpy="0 0 0" xyz="0.0 -0.03 0.17" />
-        <inertia ixx="0.03" ixy="-0.0001" ixz="-0.0001" iyy="0.03" iyz="-0.006" izz="0.01" />
+        <mass value="4.5" />
+        <origin rpy="0 0 0" xyz="-0.0 -0.02 0.17" />
+        <inertia ixx="0.03" ixy="0.0" ixz="-0.0" iyy="0.03" iyz="-0.01" izz="0.01" />
       </inertial>
       <visual name="shell">
@@ -161,14 +178,13 @@
           <mesh filename="${mesh_prefix_path}meshes/${rizon_type}/visual/link3.obj" />
         </geometry>
-        <material name="rizon_dark_grey" />
       </visual>
       <visual name="ring">
         <origin rpy="0 0 0" xyz="0 0 -0.0025" />
         <geometry>
-          <mesh filename="${mesh_prefix_path}meshes/${rizon_type}/visual/ring.obj" scale="0.062 0.062 0.002" />
-        </geometry>
-        <material name="rizon_white" />
-      </visual>
-      <collision name="hull">
+          <mesh filename="${mesh_prefix_path}meshes/${rizon_type}/visual/ring.obj"
+            scale="0.062 0.062 0.002" />
+        </geometry>
+      </visual>
+      <collision name="convex_mesh">
         <origin xyz="0 0 0" rpy="0 0 0" />
         <geometry>
@@ -179,51 +195,49 @@
     <link name="${prefix}link4">
       <inertial>
+        <mass value="3.2" />
+        <origin rpy="0 0 0" xyz="0.0 0.05 0.09" />
+        <inertia ixx="0.03" ixy="0.0" ixz="0.0001" iyy="0.03" iyz="0.0007" izz="0.005" />
+      </inertial>
+      <visual name="shell">
+        <origin xyz="0 0 0" rpy="0 0 0" />
+        <geometry>
+          <mesh filename="${mesh_prefix_path}meshes/${rizon_type}/visual/link4.obj" />
+        </geometry>
+      </visual>
+      <visual name="ring">
+        <origin rpy="${pi/2} 0 0" xyz="0 -0.0025 0" />
+        <geometry>
+          <mesh filename="${mesh_prefix_path}meshes/${rizon_type}/visual/ring.obj"
+            scale="0.062 0.062 0.002" />
+        </geometry>
+      </visual>
+      <collision name="convex_mesh">
+        <origin xyz="0 0 0" rpy="0 0 0" />
+        <geometry>
+          <mesh filename="${mesh_prefix_path}meshes/${rizon_type}/collision/link4.stl" />
+        </geometry>
+      </collision>
+    </link>
+    <link name="${prefix}link5">
+      <inertial>
         <mass value="2.4" />
-        <origin rpy="0 0 0" xyz="-0.01 0.03 0.1" />
-        <inertia ixx="0.03" ixy="0.0" ixz="-0.0001" iyy="0.03" iyz="0.0007" izz="0.005" />
-      </inertial>
-      <visual name="shell">
-        <origin xyz="0 0 0" rpy="0 0 0"/>
-        <geometry>
-          <mesh filename="${mesh_prefix_path}meshes/${rizon_type}/visual/link4.obj" />
-        </geometry>
-        <material name="rizon_dark_grey" />
-      </visual>
-      <visual name="ring">
-        <origin rpy="1.5707963 0 0" xyz="0 -0.0025 0" />
-        <geometry>
-          <mesh filename="${mesh_prefix_path}meshes/${rizon_type}/visual/ring.obj" scale="0.062 0.062 0.002" />
-        </geometry>
-        <material name="rizon_white" />
-      </visual>
-      <collision name="hull">
-        <origin xyz="0 0 0" rpy="0 0 0"/>
-        <geometry>
-          <mesh filename="${mesh_prefix_path}meshes/${rizon_type}/collision/link4.stl" />
-        </geometry>
-      </collision>
-    </link>
-    <link name="${prefix}link5">
-      <inertial>
-        <mass value="2.4" />
-        <origin rpy="0 0 0" xyz="0.0 0.0 0.13" />
+        <origin rpy="0 0 0" xyz="0.0 0.0 0.14" />
         <inertia ixx="0.01" ixy="0.0" ixz="0.0" iyy="0.01" iyz="0.001" izz="0.004" />
       </inertial>
       <visual name="shell">
-        <origin xyz="0 0 0" rpy="0 0 0"/>
+        <origin xyz="0 0 0" rpy="0 0 0" />
         <geometry>
           <mesh filename="${mesh_prefix_path}meshes/${rizon_type}/visual/link5.obj" />
         </geometry>
-        <material name="rizon_dark_grey" />
       </visual>
       <visual name="ring">
         <origin rpy="0 0 0" xyz="0 0 -0.0025" />
         <geometry>
-          <mesh filename="${mesh_prefix_path}meshes/${rizon_type}/visual/ring.obj" scale="0.051 0.051 0.002" />
-        </geometry>
-        <material name="rizon_white" />
-      </visual>
-      <collision name="hull">
-        <origin xyz="0 0 0" rpy="0 0 0"/>
+          <mesh filename="${mesh_prefix_path}meshes/${rizon_type}/visual/ring.obj"
+            scale="0.051 0.051 0.002" />
+        </geometry>
+      </visual>
+      <collision name="convex_mesh">
+        <origin xyz="0 0 0" rpy="0 0 0" />
         <geometry>
           <mesh filename="${mesh_prefix_path}meshes/${rizon_type}/collision/link5.stl" />
@@ -238,19 +252,18 @@
       </inertial>
       <visual name="shell">
-        <origin xyz="0 0 0" rpy="0 0 0"/>
+        <origin xyz="0 0 0" rpy="0 0 0" />
         <geometry>
           <mesh filename="${mesh_prefix_path}meshes/${rizon_type}/visual/link6.obj" />
         </geometry>
-        <material name="rizon_dark_grey" />
-      </visual>
-      <visual name="ring">
-        <origin rpy="1.5707963 0 0" xyz="0 -0.0025 0" />
-        <geometry>
-          <mesh filename="${mesh_prefix_path}meshes/${rizon_type}/visual/ring.obj" scale="0.051 0.051 0.002" />
-        </geometry>
-        <material name="rizon_white" />
-      </visual>
-      <collision name="hull">
-        <origin xyz="0 0 0" rpy="0 0 0"/>
+      </visual>
+      <visual name="ring">
+        <origin rpy="${pi/2} 0 0" xyz="0 -0.0025 0" />
+        <geometry>
+          <mesh filename="${mesh_prefix_path}meshes/${rizon_type}/visual/ring.obj"
+            scale="0.051 0.051 0.002" />
+        </geometry>
+      </visual>
+      <collision name="convex_mesh">
+        <origin xyz="0 0 0" rpy="0 0 0" />
         <geometry>
           <mesh filename="${mesh_prefix_path}meshes/${rizon_type}/collision/link6.stl" />
@@ -259,26 +272,25 @@
     </link>
     <link name="${prefix}link7">
-      <xacro:if value="${rizon_type=='rizon10'}">
+      <xacro:if value="${rizon_type=='Rizon10'}">
         <inertial>
-          <mass value="0.9" />
-          <origin rpy="0 0 0" xyz="0.0 -0.0 0.03" />
+          <mass value="0.8" />
+          <origin rpy="0 0 0" xyz="0.0 0.0 0.03" />
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
File: flexiv_description/urdf/rizon4r_joints_links.xacro (robot description, xacro)
@@ -3,5 +3,5 @@
   <!--
     rizon_type = "Rizon4R"
-    prefix = "Rizon4-123456_"
+    prefix = "Rizon4R-123456_"
     mesh_prefix_path = "", "package://flexiv_description/"
     NOTE: accurate kinematic but approximated dynamics parameters
