Commit message: Add Grav gripper Moveit SRDF configuration files

File: flexiv_description/urdf/grav_macro.xacro (robot description, xacro)
@@ -38,4 +38,11 @@
         <material name="flexiv_black" />
       </visual>
+      <collision>
+        <origin rpy="0 0 1.5707963267948966" xyz="0 0 0" />
+        <geometry>
+          <mesh filename="${mesh_prefix_path}meshes/grav/collision/outer_bar.stl"
+            scale="0.001 0.001 0.001" />
+        </geometry>
+      </collision>
     </link>
     <link name="${prefix}left_inner_bar">
@@ -53,4 +60,11 @@
         <material name="flexiv_black" />
       </visual>
+      <collision>
+        <origin rpy="0 0 1.5707963267948966" xyz="0 0 0" />
+        <geometry>
+          <mesh filename="${mesh_prefix_path}meshes/grav/collision/inner_bar.stl"
+            scale="0.001 0.001 0.001" />
+        </geometry>
+      </collision>
     </link>
     <link name="${prefix}left_finger_mount">
@@ -105,4 +119,11 @@
         <material name="flexiv_black" />
       </visual>
+      <collision>
+        <origin rpy="0 0 1.5707963267948966" xyz="0 0 0" />
+        <geometry>
+          <mesh filename="${mesh_prefix_path}meshes/grav/collision/outer_bar.stl"
+            scale="0.001 0.001 0.001" />
+        </geometry>
+      </collision>
     </link>
     <link name="${prefix}right_inner_bar">
@@ -120,4 +141,11 @@
         <material name="flexiv_black" />
       </visual>
+      <collision>
+        <origin rpy="0 0 1.5707963267948966" xyz="0 0 0" />
+        <geometry>
+          <mesh filename="${mesh_prefix_path}meshes/grav/collision/inner_bar.stl"
+            scale="0.001 0.001 0.001" />
+        </geometry>
+      </collision>
     </link>
     <link name="${prefix}right_finger_mount">

File: flexiv_moveit_config/srdf/rizon.srdf.xacro (robot description, xacro)
@@ -1,9 +1,18 @@
 <?xml version="1.0" encoding="UTF-8"?>
-<robot xmlns:xacro="http://wiki.ros.org/xacro" name="$(arg name)">
+<robot xmlns:xacro="http://wiki.ros.org/xacro" name="(arg name)">
     <!-- robot name parameter -->
-    <xacro:arg name="name" default="rizon"/>
+    <xacro:arg name="name" default="rizon" />
     <!-- parameters -->
     <xacro:arg name="prefix" default="" />
-    <xacro:include filename="$(find flexiv_moveit_config)/srdf/rizon_macro.srdf.xacro"/>
-    <xacro:rizon_srdf name="$(arg name)" prefix="$(arg prefix)"/>
+    <xacro:arg name="load_gripper" default="false" />
+    <xacro:property name="name" value="$(arg name)"/>
+    <xacro:include filename="$(find flexiv_moveit_config)/srdf/rizon_macro.srdf.xacro" />
+    <xacro:rizon_srdf name="${name}" prefix="$(arg prefix)" />
+    <!-- Load gripper -->
+    <xacro:if value="$(arg load_gripper)">
+        <xacro:include filename="$(find flexiv_moveit_config)/srdf/grav.srdf.xacro" />
+        <xacro:grav_srdf prefix="$(arg prefix)" />
+        <xacro:include filename="$(find flexiv_moveit_config)/srdf/rizon_grav.srdf.xacro" />
+        <xacro:rizon_grav_srdf name="${name}" prefix="$(arg prefix)" />
+    </xacro:if>
 </robot>

Commit message: Update Gripper SRDF in MoveIt configuration

File: flexiv_description/urdf/grav_macro.xacro (robot description, xacro)
@@ -323,5 +323,5 @@
     </link>
     <!-- Connect the gripper to the robot flange link -->
-    <joint name="${prefix}gripper_joint" type="fixed">
+    <joint name="${prefix}gripper_base_joint" type="fixed">
       <origin rpy="0 0 0" xyz="0 0 0" />
       <parent link="${prefix}flange" />

File: flexiv_moveit_config/srdf/grav.srdf.xacro (robot description, xacro)
@@ -1,21 +1,34 @@
 <?xml version="1.0" encoding="UTF-8"?>
 <robot xmlns:xacro="http://www.ros.org/wiki/xacro">
-    <xacro:macro name="grav_srdf" params="prefix">
+    <xacro:macro name="grav_srdf" params="name prefix">
         <group name="${prefix}grav_gripper">
-            <link name="${prefix}grav_base_link" />
-            <link name="${prefix}grav_tcp" />
-            <link name="${prefix}closed_fingers_tcp" />
-            <link name="${prefix}right_finger_tcp" />
-            <link name="${prefix}left_finger_tcp" />
-            <link name="${prefix}left_outer_bar" />
-            <link name="${prefix}left_inner_bar" />
-            <link name="${prefix}left_finger_mount" />
-            <link name="${prefix}left_finger_tip" />
-            <link name="${prefix}right_outer_bar" />
-            <link name="${prefix}right_inner_bar" />
-            <link name="${prefix}right_finger_mount" />
-            <link name="${prefix}right_finger_tip" />
+            <joint name="${prefix}gripper_base_joint" />
+            <joint name="${prefix}open_fingers_tcp_joint" />
+            <joint name="${prefix}closed_fingers_tcp_joint" />
+            <joint name="${prefix}left_outer_knuckle_joint" />
+            <joint name="${prefix}left_inner_knuckle_joint" />
+            <joint name="${prefix}left_inner_finger_joint" />
+            <joint name="${prefix}left_inner_finger_pad_joint" />
+            <joint name="${prefix}left_finger_tcp_joint" />
+            <joint name="${prefix}right_outer_knuckle_joint" />
+            <joint name="${prefix}right_inner_knuckle_joint" />
+            <joint name="${prefix}right_inner_finger_joint" />
+            <joint name="${prefix}right_inner_finger_pad_joint" />
+            <joint name="${prefix}right_finger_tcp_joint" />
             <joint name="${prefix}finger_width_joint" />
         </group>
+        <passive_joint name="${prefix}left_outer_knuckle_joint" />
+        <passive_joint name="${prefix}left_inner_knuckle_joint" />
+        <passive_joint name="${prefix}left_inner_finger_joint" />
+        <passive_joint name="${prefix}right_outer_knuckle_joint" />
+        <passive_joint name="${prefix}right_inner_knuckle_joint" />
+        <passive_joint name="${prefix}right_inner_finger_joint" />
+        <group_state name="open" group="${prefix}grav_gripper">
+            <joint name="${prefix}finger_width_joint" value="0.1" />
+        </group_state>
+        <group_state name="closed" group="${prefix}grav_gripper">
+            <joint name="${prefix}finger_width_joint" value="0.0" />
+        </group_state>
+        <end_effector name="${prefix}grav_gripper" parent_link="${prefix}flange" group="${prefix}grav_gripper" parent_group="${prefix}${name}_arm"/>
         <disable_collisions link1="${prefix}grav_base_link" link2="${prefix}grav_tcp" reason="Never" />
         <disable_collisions link1="${prefix}grav_base_link" link2="${prefix}closed_fingers_tcp" reason="Never" />
@@ -42,4 +55,8 @@
         <disable_collisions link1="${prefix}left_finger_tip" link2="${prefix}closed_fingers_tcp" reason="Adjacent" />
         <disable_collisions link1="${prefix}right_finger_tip" link2="${prefix}closed_fingers_tcp" reason="Adjacent" />
+        <disable_collisions link1="${prefix}grav_base_link" link2="${prefix}link7" reason="Adjacent" />
+        <disable_collisions link1="${prefix}grav_base_link" link2="${prefix}flange" reason="Adjacent" />
+        <disable_collisions link1="${prefix}closed_fingers_tcp" link2="${prefix}link7" reason="Adjacent" />
+        <disable_collisions link1="${prefix}closed_fingers_tcp" link2="${prefix}flange" reason="Adjacent" />
     </xacro:macro>
 </robot>

File: flexiv_moveit_config/srdf/rizon.srdf.xacro (robot description, xacro)
@@ -12,7 +12,5 @@
     <xacro:if value="$(arg load_gripper)">
         <xacro:include filename="$(find flexiv_moveit_config)/srdf/grav.srdf.xacro" />
-        <xacro:grav_srdf prefix="$(arg prefix)" />
-        <xacro:include filename="$(find flexiv_moveit_config)/srdf/rizon_grav.srdf.xacro" />
-        <xacro:rizon_grav_srdf name="${name}" prefix="$(arg prefix)" />
+        <xacro:grav_srdf name="${name}" prefix="$(arg prefix)" />
     </xacro:if>
 </robot>

Commit message: Rename directory name to Grav

File: flexiv_description/urdf/grav_macro.xacro (robot description, xacro)
@@ -12,12 +12,12 @@
         <origin rpy="0 0 1.5707963267948966" xyz="0 0 0" />
         <geometry>
-          <mesh filename="${mesh_prefix_path}meshes/grav/visual/base.stl" scale="0.001 0.001 0.001" />
-        </geometry>
-        <material name="flexiv_black" />
-      </visual>
-      <collision>
-        <origin rpy="0 0 1.5707963267948966" xyz="0 0 0" />
-        <geometry>
-          <mesh filename="${mesh_prefix_path}meshes/grav/collision/base.stl" scale="0.001 0.001 0.001" />
+          <mesh filename="${mesh_prefix_path}meshes/Grav/visual/base.stl" scale="0.001 0.001 0.001" />
+        </geometry>
+        <material name="flexiv_black" />
+      </visual>
+      <collision>
+        <origin rpy="0 0 1.5707963267948966" xyz="0 0 0" />
+        <geometry>
+          <mesh filename="${mesh_prefix_path}meshes/Grav/collision/base.stl" scale="0.001 0.001 0.001" />
         </geometry>
       </collision>
@@ -33,13 +33,13 @@
         <origin rpy="0 0 1.5707963267948966" xyz="0 0 0" />
         <geometry>
-          <mesh filename="${mesh_prefix_path}meshes/grav/visual/outer_bar.stl"
-            scale="0.001 0.001 0.001" />
-        </geometry>
-        <material name="flexiv_black" />
-      </visual>
-      <collision>
-        <origin rpy="0 0 1.5707963267948966" xyz="0 0 0" />
-        <geometry>
-          <mesh filename="${mesh_prefix_path}meshes/grav/collision/outer_bar.stl"
+          <mesh filename="${mesh_prefix_path}meshes/Grav/visual/outer_bar.stl"
+            scale="0.001 0.001 0.001" />
+        </geometry>
+        <material name="flexiv_black" />
+      </visual>
+      <collision>
+        <origin rpy="0 0 1.5707963267948966" xyz="0 0 0" />
+        <geometry>
+          <mesh filename="${mesh_prefix_path}meshes/Grav/collision/outer_bar.stl"
             scale="0.001 0.001 0.001" />
         </geometry>
@@ -55,13 +55,13 @@
         <origin rpy="0 0 1.5707963267948966" xyz="0 0 0" />
         <geometry>
-          <mesh filename="${mesh_prefix_path}meshes/grav/visual/inner_bar.stl"
-            scale="0.001 0.001 0.001" />
-        </geometry>
-        <material name="flexiv_black" />
-      </visual>
-      <collision>
-        <origin rpy="0 0 1.5707963267948966" xyz="0 0 0" />
-        <geometry>
-          <mesh filename="${mesh_prefix_path}meshes/grav/collision/inner_bar.stl"
+          <mesh filename="${mesh_prefix_path}meshes/Grav/visual/inner_bar.stl"
+            scale="0.001 0.001 0.001" />
+        </geometry>
+        <material name="flexiv_black" />
+      </visual>
+      <collision>
+        <origin rpy="0 0 1.5707963267948966" xyz="0 0 0" />
+        <geometry>
+          <mesh filename="${mesh_prefix_path}meshes/Grav/collision/inner_bar.stl"
             scale="0.001 0.001 0.001" />
         </geometry>
@@ -77,5 +77,5 @@
         <origin rpy="0 0 1.5707963267948966" xyz="0 0 0" />
         <geometry>
-          <mesh filename="${mesh_prefix_path}meshes/grav/visual/finger_mount.stl"
+          <mesh filename="${mesh_prefix_path}meshes/Grav/visual/finger_mount.stl"
             scale="0.001 0.001 0.001" />
         </geometry>
@@ -92,12 +92,12 @@
         <origin rpy="0 0 1.5707963267948966" xyz="0 0 0" />
         <geometry>
-          <mesh filename="${mesh_prefix_path}meshes/grav/visual/finger_tip.obj"
-            scale="0.001 0.001 0.001" />
-        </geometry>
-      </visual>
-      <collision>
-        <origin rpy="0 0 1.5707963267948966" xyz="0 0 0" />
-        <geometry>
-          <mesh filename="${mesh_prefix_path}meshes/grav/collision/finger_tip.stl"
+          <mesh filename="${mesh_prefix_path}meshes/Grav/visual/finger_tip.obj"
+            scale="0.001 0.001 0.001" />
+        </geometry>
+      </visual>
+      <collision>
+        <origin rpy="0 0 1.5707963267948966" xyz="0 0 0" />
+        <geometry>
+          <mesh filename="${mesh_prefix_path}meshes/Grav/collision/finger_tip.stl"
             scale="0.001 0.001 0.001" />
         </geometry>
@@ -114,13 +114,13 @@
         <origin rpy="0 0 1.5707963267948966" xyz="0 0 0" />
         <geometry>
-          <mesh filename="${mesh_prefix_path}meshes/grav/visual/outer_bar.stl"
-            scale="0.001 0.001 0.001" />
-        </geometry>
-        <material name="flexiv_black" />
-      </visual>
-      <collision>
-        <origin rpy="0 0 1.5707963267948966" xyz="0 0 0" />
-        <geometry>
-          <mesh filename="${mesh_prefix_path}meshes/grav/collision/outer_bar.stl"
+          <mesh filename="${mesh_prefix_path}meshes/Grav/visual/outer_bar.stl"
+            scale="0.001 0.001 0.001" />
+        </geometry>
+        <material name="flexiv_black" />
+      </visual>
+      <collision>
+        <origin rpy="0 0 1.5707963267948966" xyz="0 0 0" />
+        <geometry>
+          <mesh filename="${mesh_prefix_path}meshes/Grav/collision/outer_bar.stl"
             scale="0.001 0.001 0.001" />
         </geometry>
@@ -136,13 +136,13 @@
         <origin rpy="0 0 1.5707963267948966" xyz="0 0 0" />
         <geometry>
-          <mesh filename="${mesh_prefix_path}meshes/grav/visual/inner_bar.stl"
-            scale="0.001 0.001 0.001" />
-        </geometry>
-        <material name="flexiv_black" />
-      </visual>
-      <collision>
-        <origin rpy="0 0 1.5707963267948966" xyz="0 0 0" />
-        <geometry>
-          <mesh filename="${mesh_prefix_path}meshes/grav/collision/inner_bar.stl"
+          <mesh filename="${mesh_prefix_path}meshes/Grav/visual/inner_bar.stl"
+            scale="0.001 0.001 0.001" />
+        </geometry>
+        <material name="flexiv_black" />
+      </visual>
+      <collision>
+        <origin rpy="0 0 1.5707963267948966" xyz="0 0 0" />
+        <geometry>
+          <mesh filename="${mesh_prefix_path}meshes/Grav/collision/inner_bar.stl"
             scale="0.001 0.001 0.001" />
         </geometry>
@@ -158,5 +158,5 @@
         <origin rpy="0 0 1.5707963267948966" xyz="0 0 0" />
         <geometry>
-          <mesh filename="${mesh_prefix_path}meshes/grav/visual/finger_mount.stl"
+          <mesh filename="${mesh_prefix_path}meshes/Grav/visual/finger_mount.stl"
             scale="0.001 0.001 0.001" />
         </geometry>
@@ -173,12 +173,12 @@
         <origin rpy="0 0 1.5707963267948966" xyz="0 0 0" />
         <geometry>
-          <mesh filename="${mesh_prefix_path}meshes/grav/visual/finger_tip.obj"
-            scale="0.001 0.001 0.001" />
-        </geometry>
-      </visual>
-      <collision>
-        <origin rpy="0 0 1.5707963267948966" xyz="0 0 0" />
-        <geometry>
-          <mesh filename="${mesh_prefix_path}meshes/grav/collision/finger_tip.stl"
+          <mesh filename="${mesh_prefix_path}meshes/Grav/visual/finger_tip.obj"
+            scale="0.001 0.001 0.001" />
+        </geometry>
+      </visual>
+      <collision>
+        <origin rpy="0 0 1.5707963267948966" xyz="0 0 0" />
+        <geometry>
+          <mesh filename="${mesh_prefix_path}meshes/Grav/collision/finger_tip.stl"
             scale="0.001 0.001 0.001" />
         </geometry>
