Commit message: Remove initial_positions xacro parameter

File: flexiv_description/urdf/rizon.urdf.xacro (robot description, xacro)
@@ -14,7 +14,4 @@
   <xacro:arg name="use_fake_hardware" default="false" />
   <xacro:arg name="fake_sensor_commands" default="false" />
-  <xacro:arg name="initial_positions_file" default="$(find flexiv_description)/config/initial_positions.yaml"/>
-  <!-- convert to property to use substitution in function -->
-  <xacro:property name="initial_positions_file" default="$(arg initial_positions_file)"/>
   <xacro:rizon_robot
     rizon_type="$(arg rizon_type)"
@@ -24,6 +21,5 @@
     gripper_name="$(arg gripper_name)"
     use_fake_hardware="$(arg use_fake_hardware)"
-    fake_sensor_commands="$(arg fake_sensor_commands)"
-    initial_positions="${xacro.load_yaml(initial_positions_file)}">
+    fake_sensor_commands="$(arg fake_sensor_commands)">
   </xacro:rizon_robot>
 </robot>

File: flexiv_description/urdf/rizon10.ros2_control.xacro (robot description, xacro)
@@ -6,5 +6,4 @@
     use_fake_hardware:=false
     fake_sensor_commands:=false
-    initial_positions:=${dict(joint1=0.0,joint2=-0.69813,joint3=0.0,joint4=1.570796,joint5=0.0,joint6=0.69813,joint7=0.0)}
     ">
     <ros2_control name="FlexivHardwareInterface" type="system">
@@ -33,5 +32,5 @@
         <state_interface name="position">
           <!-- initial position for the FakeSystem -->
-          <param name="initial_value">${initial_positions['joint1']}</param>
+          <param name="initial_value">0.0</param>
         </state_interface>
         <state_interface name="velocity"/>
@@ -50,5 +49,5 @@
         <state_interface name="position">
           <!-- initial position for the FakeSystem -->
-          <param name="initial_value">${initial_positions['joint2']}</param>
+          <param name="initial_value">-0.69813</param>
         </state_interface>
         <state_interface name="velocity"/>
@@ -67,5 +66,5 @@
         <state_interface name="position">
           <!-- initial position for the FakeSystem -->
-          <param name="initial_value">${initial_positions['joint3']}</param>
+          <param name="initial_value">0.0</param>
         </state_interface>
         <state_interface name="velocity"/>
@@ -84,5 +83,5 @@
         <state_interface name="position">
           <!-- initial position for the FakeSystem -->
-          <param name="initial_value">${initial_positions['joint4']}</param>
+          <param name="initial_value">1.570796</param>
         </state_interface>
         <state_interface name="velocity"/>
@@ -101,5 +100,5 @@
         <state_interface name="position">
           <!-- initial position for the FakeSystem -->
-          <param name="initial_value">${initial_positions['joint5']}</param>
+          <param name="initial_value">0.0</param>
         </state_interface>
         <state_interface name="velocity"/>
@@ -118,5 +117,5 @@
         <state_interface name="position">
           <!-- initial position for the FakeSystem -->
-          <param name="initial_value">${initial_positions['joint6']}</param>
+          <param name="initial_value">0.69813</param>
         </state_interface>
         <state_interface name="velocity"/>
@@ -135,5 +134,5 @@
         <state_interface name="position">
           <!-- initial position for the FakeSystem -->
-          <param name="initial_value">${initial_positions['joint7']}</param>
+          <param name="initial_value">0.0</param>
         </state_interface>
         <state_interface name="velocity"/>

File: flexiv_description/urdf/rizon4.ros2_control.xacro (robot description, xacro)
@@ -6,5 +6,4 @@
     use_fake_hardware:=false
     fake_sensor_commands:=false
-    initial_positions:=${dict(joint1=0.0,joint2=-0.69813,joint3=0.0,joint4=1.570796,joint5=0.0,joint6=0.69813,joint7=0.0)}
     ">
     <ros2_control name="FlexivHardwareInterface" type="system">
@@ -33,5 +32,5 @@
         <state_interface name="position">
           <!-- initial position for the FakeSystem -->
-          <param name="initial_value">${initial_positions['joint1']}</param>
+          <param name="initial_value">0.0</param>
         </state_interface>
         <state_interface name="velocity"/>
@@ -50,5 +49,5 @@
         <state_interface name="position">
           <!-- initial position for the FakeSystem -->
-          <param name="initial_value">${initial_positions['joint2']}</param>
+          <param name="initial_value">-0.69813</param>
         </state_interface>
         <state_interface name="velocity"/>
@@ -67,5 +66,5 @@
         <state_interface name="position">
           <!-- initial position for the FakeSystem -->
-          <param name="initial_value">${initial_positions['joint3']}</param>
+          <param name="initial_value">0.0</param>
         </state_interface>
         <state_interface name="velocity"/>
@@ -84,5 +83,5 @@
         <state_interface name="position">
           <!-- initial position for the FakeSystem -->
-          <param name="initial_value">${initial_positions['joint4']}</param>
+          <param name="initial_value">1.570796</param>
         </state_interface>
         <state_interface name="velocity"/>
@@ -101,5 +100,5 @@
         <state_interface name="position">
           <!-- initial position for the FakeSystem -->
-          <param name="initial_value">${initial_positions['joint5']}</param>
+          <param name="initial_value">0.0</param>
         </state_interface>
         <state_interface name="velocity"/>
@@ -118,5 +117,5 @@
         <state_interface name="position">
           <!-- initial position for the FakeSystem -->
-          <param name="initial_value">${initial_positions['joint6']}</param>
+          <param name="initial_value">0.69813</param>
         </state_interface>
         <state_interface name="velocity"/>
@@ -135,5 +134,5 @@
         <state_interface name="position">
           <!-- initial position for the FakeSystem -->
-          <param name="initial_value">${initial_positions['joint7']}</param>
+          <param name="initial_value">0.0</param>
         </state_interface>
         <state_interface name="velocity"/>

File: flexiv_description/urdf/rizon_macro.xacro (robot description, xacro)
@@ -9,5 +9,4 @@
     use_fake_hardware:=false
     fake_sensor_commands:=false
-    initial_positions:=${dict(joint1=0.0,joint2=-0.69813,joint3=0.0,joint4=1.570796,joint5=0.0,joint6=0.69813,joint7=0.0)}
     ">
     <!-- Load gripper -->
@@ -21,24 +20,24 @@
     <xacro:if value="${rizon_type=='rizon4' or rizon_type=='rizon4s'}">
       <xacro:include filename="$(find flexiv_description)/urdf/rizon4_joints_links.xacro" />
-      <xacro:rizon4_joints_links rizon_type="${rizon_type}" prefix="${prefix}" mesh_prefix_path="package://flexiv_description/" />
+      <xacro:rizon4_joints_links rizon_type="${rizon_type}" prefix="${prefix}"
+        robot_sn="${robot_sn}" mesh_prefix_path="package://flexiv_description/" />
       <!-- ros2 control include -->
-      <xacro:include filename="$(find flexiv_description)/urdf/rizon4.ros2_control.xacro"/>
+      <xacro:include filename="$(find flexiv_description)/urdf/rizon4.ros2_control.xacro" />
       <xacro:rizon4_ros2_control prefix="${prefix}" robot_sn="${robot_sn}"
         use_fake_hardware="${use_fake_hardware}"
         fake_sensor_commands="${fake_sensor_commands}"
-        initial_positions="${initial_positions}"
-        />
+      />
     </xacro:if>
     <!-- Rizon 10 or 10s-->
     <xacro:if value="${rizon_type=='rizon10' or rizon_type=='rizon10s'}">
       <xacro:include filename="$(find flexiv_description)/urdf/rizon10_joints_links.xacro" />
-      <xacro:rizon10_joints_links rizon_type="${rizon_type}" prefix="${prefix}" mesh_prefix_path="package://flexiv_description/" />
+      <xacro:rizon10_joints_links rizon_type="${rizon_type}" prefix="${prefix}"
+        robot_sn="${robot_sn}" mesh_prefix_path="package://flexiv_description/" />
       <!-- ros2 control include -->
-      <xacro:include filename="$(find flexiv_description)/urdf/rizon10.ros2_control.xacro"/>
+      <xacro:include filename="$(find flexiv_description)/urdf/rizon10.ros2_control.xacro" />
       <xacro:rizon10_ros2_control prefix="${prefix}" robot_sn="${robot_sn}"
         use_fake_hardware="${use_fake_hardware}"
         fake_sensor_commands="${fake_sensor_commands}"
-        initial_positions="${initial_positions}"
-        />
+      />
     </xacro:if>
   </xacro:macro>

Commit message: Remove name and add robot_sn as joint name prefix

File: flexiv_description/urdf/rizon.urdf.xacro (robot description, xacro)
@@ -1,6 +1,4 @@
 <?xml version="1.0" encoding="utf-8"?>
-<robot xmlns:xacro="http://www.ros.org/wiki/xacro" name="$(arg name)">
-  <!-- Enable setting arguments from the launch file -->
-  <xacro:arg name="name" default="rizon"/>
+<robot xmlns:xacro="http://www.ros.org/wiki/xacro" name="rizon">
   <!-- 'rizon_type' values: rizon4, rizon4s, rizon10, rizon10s -->
   <xacro:arg name="rizon_type" default="rizon4"/>
@@ -8,5 +6,5 @@
   <xacro:include filename="$(find flexiv_description)/urdf/rizon_macro.xacro"/>
   <!-- parameters -->
-  <xacro:arg name="prefix" default="" />
+  <xacro:arg name="arm_prefix" default="" />
   <xacro:arg name="robot_sn" default="" />
   <xacro:arg name="load_gripper" default="false" />
@@ -16,5 +14,5 @@
   <xacro:rizon_robot
     rizon_type="$(arg rizon_type)"
-    prefix="$(arg prefix)"
+    arm_prefix="$(arg arm_prefix)"
     robot_sn="$(arg robot_sn)"
     load_gripper="$(arg load_gripper)"

File: flexiv_description/urdf/rizon_macro.xacro (robot description, xacro)
@@ -1,7 +1,8 @@
 <?xml version="1.0"?>
 <robot xmlns:xacro="http://wiki.ros.org/xacro">
-  <xacro:macro name="rizon_robot" params="
+  <xacro:macro name="rizon_robot"
+    params="
     rizon_type
-    prefix
+    arm_prefix
     robot_sn
     load_gripper:=false
@@ -10,4 +11,6 @@
     fake_sensor_commands:=false
     ">
+    <!-- Prefix defaults to 'arm_prefix_robot_sn' -->
+    <xacro:property name="prefix" value="${arm_prefix + robot_sn + '_'}" />
     <!-- Load gripper -->
     <xacro:if value="${load_gripper and gripper_name=='Flexiv-GN01'}">
@@ -21,5 +24,5 @@
       <xacro:include filename="$(find flexiv_description)/urdf/rizon4_joints_links.xacro" />
       <xacro:rizon4_joints_links rizon_type="${rizon_type}" prefix="${prefix}"
-        robot_sn="${robot_sn}" mesh_prefix_path="package://flexiv_description/" />
+        mesh_prefix_path="package://flexiv_description/" />
       <!-- ros2 control include -->
       <xacro:include filename="$(find flexiv_description)/urdf/rizon4.ros2_control.xacro" />
@@ -33,5 +36,5 @@
       <xacro:include filename="$(find flexiv_description)/urdf/rizon10_joints_links.xacro" />
       <xacro:rizon10_joints_links rizon_type="${rizon_type}" prefix="${prefix}"
-        robot_sn="${robot_sn}" mesh_prefix_path="package://flexiv_description/" />
+        mesh_prefix_path="package://flexiv_description/" />
       <!-- ros2 control include -->
       <xacro:include filename="$(find flexiv_description)/urdf/rizon10.ros2_control.xacro" />

File: flexiv_moveit_config/srdf/rizon_macro.srdf.xacro (robot description, xacro)
@@ -1,6 +1,6 @@
 <?xml version="1.0" encoding="UTF-8"?>
 <robot xmlns:xacro="http://www.ros.org/wiki/xacro">
-    <xacro:macro name="rizon_srdf" params="name prefix">
-        <group name="${prefix}${name}_arm">
+    <xacro:macro name="rizon_srdf" params="prefix robot_sn">
+        <group name="${prefix}${robot_sn}_arm">
             <chain base_link="${prefix}base_link" tip_link="${prefix}flange" />
         </group>
