Commit message: Add support for Rizon4R robot model and update existing Rizon4 configurations

File: flexiv_description/urdf/rizon.urdf.xacro (robot description, xacro)
@@ -1,6 +1,6 @@
 <?xml version="1.0" encoding="utf-8"?>
 <robot xmlns:xacro="http://www.ros.org/wiki/xacro" name="rizon">
-  <!-- 'rizon_type' values: rizon4, rizon4s, rizon10, rizon10s -->
-  <xacro:arg name="rizon_type" default="rizon4"/>
+  <!-- 'rizon_type' values: Rizon4, Rizon4s, Rizon10, Rizon10s -->
+  <xacro:arg name="rizon_type" default="Rizon4"/>
   <!-- import main macro -->
   <xacro:include filename="$(find flexiv_description)/urdf/rizon_macro.xacro"/>

File: flexiv_description/urdf/rizon4r_joints_links.xacro (robot description, xacro)
@@ -2,10 +2,10 @@
 <robot xmlns:xacro="http://www.ros.org/wiki/xacro">
   <!--
-    rizon_type = "Rizon4", "Rizon4M", "Rizon4s"
+    rizon_type = "Rizon4R"
     prefix = "Rizon4-123456_"
     mesh_prefix_path = "", "package://flexiv_description/"
     NOTE: accurate kinematic but approximated dynamics parameters
   -->
-  <xacro:macro name="rizon4_joints_links" params="rizon_type prefix mesh_prefix_path">
+  <xacro:macro name="rizon4r_joints_links" params="rizon_type prefix mesh_prefix_path">
     <!-- JOINTS-->
     <joint name="${prefix}base_joint" type="fixed">
@@ -17,5 +17,5 @@
       <parent link="${prefix}base_link" />
       <child link="${prefix}link1" />
-      <origin xyz="0.0 0.0 0.155" rpy="0 0 ${-pi}" />
+      <origin xyz="0.0 0.0 0.155" rpy="${pi} 0 ${-pi}" />
       <axis xyz="0 0 1" />
       <limit effort="123" lower="-2.8798" upper="2.8798" velocity="2.0944" />
@@ -26,5 +26,5 @@
       <parent link="${prefix}link1" />
       <child link="${prefix}link2" />
-      <origin xyz="0.0 0.03 0.210" rpy="0 0 0" />
+      <origin xyz="0.0 0.03 -0.210" rpy="0 0 ${-pi}" />
       <axis xyz="0 1 0" />
       <limit effort="123" lower="-2.3562" upper="2.3562" velocity="2.0944" />
@@ -35,5 +35,5 @@
       <parent link="${prefix}link2" />
       <child link="${prefix}link3" />
-      <origin xyz="0.0 0.035 0.205" rpy="0 0 0" />
+      <origin xyz="0.0 -0.035 -0.205" rpy="0 0 ${-pi}" />
       <axis xyz="0 0 1" />
       <limit effort="64" lower="-3.0543" upper="3.0543" velocity="2.4435" />
@@ -44,5 +44,5 @@
       <parent link="${prefix}link3" />
       <child link="${prefix}link4" />
-      <origin xyz="-0.02 -0.03 0.19" rpy="0 0 ${-pi}" />
+      <origin xyz="-0.02 -0.03 -0.19" rpy="0 0 0" />
       <axis xyz="0 1 0" />
       <limit effort="64" lower="-1.9548" upper="2.7751" velocity="2.4435" />
@@ -53,5 +53,5 @@
       <parent link="${prefix}link4" />
       <child link="${prefix}link5" />
-      <origin xyz="-0.02 0.025 0.195" rpy="0 0 ${-pi}" />
+      <origin xyz="0.02 -0.025 -0.195" rpy="0 0 0" />
       <axis xyz="0 0 1" />
       <limit effort="39" lower="-3.0543" upper="3.0543" velocity="4.8869" />
@@ -62,5 +62,5 @@
       <parent link="${prefix}link5" />
       <child link="${prefix}link6" />
-      <origin xyz="0.0 0.03 0.19" rpy="0 0 0" />
+      <origin xyz="0.0 0.03 -0.19" rpy="0 0 ${-pi}" />
       <axis xyz="0 1 0" />
       <limit effort="39" lower="-1.4835" upper="4.6251" velocity="4.8869" />
@@ -71,5 +71,5 @@
       <parent link="${prefix}link6" />
       <child link="${prefix}link7" />
-      <origin xyz="-0.015 0.073 0.11" rpy="0 ${-pi/2} 0" />
+      <origin xyz="0.015 -0.073 -0.11" rpy="0 ${-pi/2} 0" />
       <axis xyz="0 0 1" />
       <limit effort="39" lower="-3.0543" upper="3.0543" velocity="4.8869" />
@@ -80,10 +80,5 @@
       <parent link="${prefix}link7" />
       <child link="${prefix}flange" />
-      <xacro:if value="${rizon_type=='Rizon4' or rizon_type=='Rizon4M'}">
-        <origin xyz="0.0 0.0 0.081" rpy="0 0 ${-pi}" />
-      </xacro:if>
-      <xacro:if value="${rizon_type=='Rizon4s'}">
-        <origin xyz="0.0 0.0 0.124" rpy="0 0 ${-pi}" />
-      </xacro:if>
+      <origin xyz="0.0 0.0 -0.081" rpy="${pi} 0 0" />
     </joint>
     <!-- LINKS -->
@@ -92,10 +87,10 @@
     <link name="${prefix}base_link">
       <inertial>
-        <mass value="3.8" />
-        <origin rpy="0 0 0" xyz="0.0 -0.0 0.09" />
-        <inertia ixx="0.02" ixy="0.0" ixz="0.0" iyy="0.02" iyz="0.0" izz="0.01" />
-      </inertial>
-      <visual name="shell">
-        <origin xyz="0 0 0" rpy="0 0 0" />
+        <mass value="3.7" />
+        <origin rpy="0 0 0" xyz="-0.0 0.0 0.09" />
+        <inertia ixx="0.02" ixy="0.0" ixz="0.0" iyy="0.02" iyz="-0.0" izz="0.01" />
+      </inertial>
+      <visual name="shell">
+        <origin xyz="0 0 0" rpy="0 0 ${pi}" />
         <geometry>
           <mesh filename="${mesh_prefix_path}meshes/${rizon_type}/visual/link0.obj" />
@@ -103,5 +98,5 @@
       </visual>
       <collision name="convex_mesh">
-        <origin xyz="0 0 0" rpy="0 0 0" />
+        <origin xyz="0 0 0" rpy="0 0 ${pi}" />
         <geometry>
           <mesh filename="${mesh_prefix_path}meshes/${rizon_type}/collision/link0.stl" />
@@ -117,10 +112,10 @@
     <link name="${prefix}link1">
       <inertial>
-        <mass value="3.6" />
-        <origin rpy="0 0 0" xyz="0.0 0.0 0.15" />
+        <mass value="3.7" />
+        <origin rpy="0 0 0" xyz="0.0 0.01 -0.15" />
         <inertia ixx="0.03" ixy="0.0" ixz="0.0" iyy="0.03" iyz="0.0" izz="0.01" />
       </inertial>
       <visual name="shell">
-        <origin xyz="0 0 0" rpy="0 0 0" />
+        <origin xyz="0 0 0" rpy="0 ${pi} 0" />
         <geometry>
           <mesh filename="${mesh_prefix_path}meshes/${rizon_type}/visual/link1.obj" />
@@ -128,5 +123,5 @@
       </visual>
       <visual name="ring">
-        <origin rpy="0 0 0" xyz="0 0 -0.0025" />
+        <origin rpy="0 0 0" xyz="0 0 0.0025" />
         <geometry>
           <mesh filename="${mesh_prefix_path}meshes/${rizon_type}/visual/ring.obj"
@@ -135,5 +130,5 @@
       </visual>
       <collision name="convex_mesh">
-        <origin xyz="0 0 0" rpy="0 0 0" />
+        <origin xyz="0 0 0" rpy="0 ${pi} 0" />
         <geometry>
           <mesh filename="${mesh_prefix_path}meshes/${rizon_type}/collision/link1.stl" />
@@ -144,9 +139,9 @@
       <inertial>
         <mass value="2.7" />
-        <origin rpy="0 0 0" xyz="-0.0 0.04 0.1" />
+        <origin rpy="0 0 0" xyz="0.0 -0.04 -0.1" />
         <inertia ixx="0.02" ixy="0.0" ixz="0.0" iyy="0.02" iyz="-0.0003" izz="0.004" />
       </inertial>
       <visual name="shell">
-        <origin xyz="0 0 0" rpy="0 0 0" />
+        <origin xyz="0 0 0" rpy="${pi} 0 0" />
         <geometry>
           <mesh filename="${mesh_prefix_path}meshes/${rizon_type}/visual/link2.obj" />
@@ -154,5 +149,5 @@
       </visual>
       <visual name="ring">
-        <origin rpy="${pi/2} 0 0" xyz="0 -0.0025 0" />
+        <origin rpy="${pi/2} 0 0" xyz="0 0.0025 0" />
         <geometry>
           <mesh filename="${mesh_prefix_path}meshes/${rizon_type}/visual/ring.obj"
@@ -161,5 +156,5 @@
       </visual>
       <collision name="convex_mesh">
-        <origin xyz="0 0 0" rpy="0 0 0" />
+        <origin xyz="0 0 0" rpy="${pi} 0 0" />
         <geometry>
           <mesh filename="${mesh_prefix_path}meshes/${rizon_type}/collision/link2.stl" />
@@ -170,24 +165,24 @@
       <inertial>
         <mass value="2.4" />
-        <origin rpy="0 0 0" xyz="-0.01 -0.0 0.14" />
-        <inertia ixx="0.01" ixy="0.0" ixz="-0.001" iyy="0.01" iyz="-0.0007" izz="0.004" />
-      </inertial>
-      <visual name="shell">
-        <origin xyz="0 0 0" rpy="0 0 0" />
-        <geometry>
-          <mesh filename="${mesh_prefix_path}meshes/${rizon_type}/visual/link3.obj" />
-        </geometry>
-      </visual>
-      <visual name="ring">
-        <origin rpy="0 0 0" xyz="0 0 -0.0025" />
-        <geometry>
-          <mesh filename="${mesh_prefix_path}meshes/${rizon_type}/visual/ring.obj"
-            scale="0.051 0.051 0.002" />
-        </geometry>
-      </visual>
-      <collision name="convex_mesh">
-        <origin xyz="0 0 0" rpy="0 0 0" />
-        <geometry>
-          <mesh filename="${mesh_prefix_path}meshes/${rizon_type}/collision/link3.stl" />
+        <origin rpy="0 0 0" xyz="-0.01 -0.0 -0.13" />
+        <inertia ixx="0.01" ixy="0.0" ixz="0.001" iyy="0.01" iyz="0.0007" izz="0.004" />
+      </inertial>
+      <visual name="shell">
+        <origin xyz="0 0 0" rpy="0 ${pi} 0" />
+        <geometry>
+          <mesh filename="${mesh_prefix_path}meshes/${rizon_type}/visual/link3r.obj" />
+        </geometry>
+      </visual>
+      <visual name="ring">
+        <origin rpy="0 0 0" xyz="0 0 0.0025" />
+        <geometry>
+          <mesh filename="${mesh_prefix_path}meshes/${rizon_type}/visual/ring.obj"
+            scale="0.051 0.051 0.002" />
+        </geometry>
+      </visual>
+      <collision name="convex_mesh">
+        <origin xyz="0 0 0" rpy="0 ${pi} 0" />
+        <geometry>
+          <mesh filename="${mesh_prefix_path}meshes/${rizon_type}/collision/link3r.stl" />
         </geometry>
       </collision>
@@ -196,24 +191,24 @@
       <inertial>
         <mass value="2.4" />
-        <origin rpy="0 0 0" xyz="-0.01 0.03 0.1" />
+        <origin rpy="0 0 0" xyz="0.01 -0.03 -0.1" />
         <inertia ixx="0.02" ixy="0.0" ixz="-0.002" iyy="0.02" iyz="-0.001" izz="0.003" />
       </inertial>
       <visual name="shell">
-        <origin xyz="0 0 0" rpy="0 0 0" />
-        <geometry>
-          <mesh filename="${mesh_prefix_path}meshes/${rizon_type}/visual/link4.obj" />
-        </geometry>
-      </visual>
-      <visual name="ring">
-        <origin rpy="${pi/2} 0 0" xyz="0 -0.0025 0" />
-        <geometry>
-          <mesh filename="${mesh_prefix_path}meshes/${rizon_type}/visual/ring.obj"
-            scale="0.051 0.051 0.002" />
-        </geometry>
-      </visual>
-      <collision name="convex_mesh">
-        <origin xyz="0 0 0" rpy="0 0 0" />
-        <geometry>
-          <mesh filename="${mesh_prefix_path}meshes/${rizon_type}/collision/link4.stl" />
+        <origin xyz="0 0 0" rpy="${pi} 0 0" />
+        <geometry>
+          <mesh filename="${mesh_prefix_path}meshes/${rizon_type}/visual/link4r.obj" />
+        </geometry>
+      </visual>
+      <visual name="ring">
+        <origin rpy="${pi/2} 0 0" xyz="0 0.0025 0" />
+        <geometry>
+          <mesh filename="${mesh_prefix_path}meshes/${rizon_type}/visual/ring.obj"
+            scale="0.051 0.051 0.002" />
+        </geometry>
+      </visual>
+      <collision name="convex_mesh">
+        <origin xyz="0 0 0" rpy="${pi} 0 0" />
+        <geometry>
+          <mesh filename="${mesh_prefix_path}meshes/${rizon_type}/collision/link4r.stl" />
         </geometry>
       </collision>
@@ -221,10 +216,10 @@
     <link name="${prefix}link5">
       <inertial>
-        <mass value="2.3" />
-        <origin rpy="0 0 0" xyz="0.0 0.0 0.14" />
-        <inertia ixx="0.01" ixy="0.0" ixz="0.0" iyy="0.01" iyz="0.001" izz="0.004" />
-      </inertial>
-      <visual name="shell">
-        <origin xyz="0 0 0" rpy="0 0 0" />
+        <mass value="2.4" />
+        <origin rpy="0 0 0" xyz="0.0 0.0 -0.13" />
+        <inertia ixx="0.01" ixy="0.0" ixz="0.0" iyy="0.01" iyz="-0.001" izz="0.004" />
+      </inertial>
+      <visual name="shell">
+        <origin xyz="0 0 0" rpy="0 ${pi} 0" />
         <geometry>
           <mesh filename="${mesh_prefix_path}meshes/${rizon_type}/visual/link5.obj" />
@@ -232,12 +227,12 @@
       </visual>
       <visual name="ring">
-        <origin rpy="0 0 0" xyz="0 0 -0.0025" />
-        <geometry>
-          <mesh filename="${mesh_prefix_path}meshes/${rizon_type}/visual/ring.obj"
-            scale="0.051 0.051 0.002" />
-        </geometry>
-      </visual>
-      <collision name="convex_mesh">
-        <origin xyz="0 0 0" rpy="0 0 0" />
+        <origin rpy="0 0 0" xyz="0 0 0.0025" />
+        <geometry>
+          <mesh filename="${mesh_prefix_path}meshes/${rizon_type}/visual/ring.obj"
+            scale="0.051 0.051 0.002" />
+        </geometry>
+      </visual>
+      <collision name="convex_mesh">
+        <origin xyz="0 0 0" rpy="0 ${pi} 0" />
         <geometry>
           <mesh filename="${mesh_prefix_path}meshes/${rizon_type}/collision/link5.stl" />
@@ -248,80 +243,52 @@
       <inertial>
         <mass value="2.2" />
-        <origin rpy="0 0 0" xyz="0.02 0.06 0.07" />
+        <origin rpy="0 0 0" xyz="-0.02 -0.06 -0.07" />
         <inertia ixx="0.01" ixy="0.0" ixz="-0.001" iyy="0.01" iyz="0.002" izz="0.004" />
       </inertial>
       <visual name="shell">
-        <origin xyz="0 0 0" rpy="0 0 0" />
-        <geometry>
-          <mesh filename="${mesh_prefix_path}meshes/${rizon_type}/visual/link6.obj" />
-        </geometry>
-      </visual>
-      <visual name="ring">
-        <origin rpy="${pi/2} 0 0" xyz="0 -0.0025 0" />
-        <geometry>
-          <mesh filename="${mesh_prefix_path}meshes/${rizon_type}/visual/ring.obj"
-            scale="0.051 0.051 0.002" />
-        </geometry>
-      </visual>
-      <collision name="convex_mesh">
-        <origin xyz="0 0 0" rpy="0 0 0" />
-        <geometry>
-          <mesh filename="${mesh_prefix_path}meshes/${rizon_type}/collision/link6.stl" />
+        <origin xyz="0 0 0" rpy="0 ${pi} 0" />
+        <geometry>
+          <mesh filename="${mesh_prefix_path}meshes/${rizon_type}/visual/link6r.obj" />
+        </geometry>
+      </visual>
+      <visual name="ring">
+        <origin rpy="${pi/2} 0 0" xyz="0 0.0025 0" />
+        <geometry>
+          <mesh filename="${mesh_prefix_path}meshes/${rizon_type}/visual/ring.obj"
+            scale="0.051 0.051 0.002" />
+        </geometry>
+      </visual>
+      <collision name="convex_mesh">
+        <origin xyz="0 0 0" rpy="0 ${pi} 0" />
+        <geometry>
+          <mesh filename="${mesh_prefix_path}meshes/${rizon_type}/collision/link6r.stl" />
         </geometry>
       </collision>
     </link>
     <link name="${prefix}link7">
-      <xacro:if value="${rizon_type=='Rizon4' or rizon_type=='Rizon4M'}">
-        <inertial>
-          <mass value="0.8" />
-          <origin rpy="0 0 0" xyz="0.0 0.0 0.03" />
-          <inertia ixx="0.001" ixy="0.0" ixz="0.0" iyy="0.001" iyz="0.0" izz="0.001" />
-        </inertial>
-        <visual name="shell">
-          <origin xyz="0 0 0" rpy="0 0 0" />
-          <geometry>
-            <mesh filename="${mesh_prefix_path}meshes/${rizon_type}/visual/link7.obj" />
-          </geometry>
-        </visual>
-        <visual name="ring">
-          <origin rpy="0 0 0" xyz="0 0 -0.0025" />
-          <geometry>
-            <mesh filename="${mesh_prefix_path}meshes/${rizon_type}/visual/ring.obj"
-              scale="0.051 0.051 0.002" />
-          </geometry>
-        </visual>
-        <collision name="convex_mesh">
-          <origin xyz="0 0 0" rpy="0 0 0" />
-          <geometry>
-            <mesh filename="${mesh_prefix_path}meshes/${rizon_type}/collision/link7.stl" />
-          </geometry>
-        </collision>
-      </xacro:if>
-      <xacro:if value="${rizon_type=='Rizon4s'}">
-        <inertial>
-          <mass value="1.4" />
-          <origin xyz="0.0 0.0 0.05" rpy="0 0 0" />
-          <inertia ixx="0.001" ixy="0.0" ixz="0.0" iyy="0.001" iyz="0.0" izz="0.001" />
-        </inertial>
-        <visual name="shell">
-          <origin xyz="0 0 0" rpy="0 0 0" />
-          <geometry>
-            <mesh filename="${mesh_prefix_path}meshes/${rizon_type}/visual/link7.obj" />
-          </geometry>
-        </visual>
-        <visual name="ring">
-          <origin rpy="0 0 0" xyz="0 0 -0.0025" />
-          <geometry>
-            <mesh filename="${mesh_prefix_path}meshes/${rizon_type}/visual/ring.obj"
-              scale="0.051 0.051 0.002" />
-          </geometry>
-        </visual>
-        <collision name="hull">
-          <origin xyz="0 0 0" rpy="0 0 0" />
-          <geometry>
-            <mesh filename="${mesh_prefix_path}meshes/${rizon_type}/collision/link7.stl" />
-          </geometry>
-        </collision>
-      </xacro:if>
+      <inertial>
+        <mass value="0.8" />
+        <origin rpy="0 0 0" xyz="0.0 -0.0 0.03" />
+        <inertia ixx="0.001" ixy="0.0" ixz="0.0" iyy="0.001" iyz="0.0" izz="0.001" />
+      </inertial>
+      <visual name="shell">
+        <origin xyz="0 0 0" rpy="${pi} 0 0" />
+        <geometry>
+          <mesh filename="${mesh_prefix_path}meshes/${rizon_type}/visual/link7.obj" />
+        </geometry>
+      </visual>
+      <visual name="ring">
+        <origin rpy="0 0 0" xyz="0 0 0.0025" />
+        <geometry>
+          <mesh filename="${mesh_prefix_path}meshes/${rizon_type}/visual/ring.obj"
+            scale="0.051 0.051 0.002" />
+        </geometry>
+      </visual>
+      <collision name="convex_mesh">
+        <origin xyz="0 0 0" rpy="${pi} 0 0" />
+        <geometry>
+          <mesh filename="${mesh_prefix_path}meshes/${rizon_type}/collision/link7.stl" />
+        </geometry>
+      </collision>
     </link>
     <link name="${prefix}flange">

File: flexiv_description/urdf/rizon_macro.xacro (robot description, xacro)
@@ -18,11 +18,19 @@
       <xacro:flexiv_GN01 prefix="${prefix}" mesh_prefix_path="package://flexiv_description/" />
     </xacro:if>
-    <!-- Import Rviz colors -->
-    <xacro:include filename="$(find flexiv_description)/urdf/flexiv_arm.materials.xacro" />
-    <!-- Rizon 4 or 4s-->
-    <xacro:if value="${rizon_type=='rizon4' or rizon_type=='rizon4s'}">
-      <xacro:include filename="$(find flexiv_description)/urdf/rizon4_joints_links.xacro" />
-      <xacro:rizon4_joints_links rizon_type="${rizon_type}" prefix="${prefix}"
-        mesh_prefix_path="package://flexiv_description/" />
+    <!-- Rizon4, Rizon4M, Rizon4R or Rizon4s -->
+    <xacro:if
+      value="${rizon_type=='Rizon4' or rizon_type=='Rizon4M' or rizon_type=='Rizon4R' or rizon_type=='Rizon4s'}">
+      <!-- Rizon4R -->
+      <xacro:if value="${rizon_type=='Rizon4R'}">
+        <xacro:include filename="$(find flexiv_description)/urdf/rizon4r_joints_links.xacro" />
+        <xacro:rizon4r_joints_links rizon_type="${rizon_type}" prefix="${prefix}"
+          mesh_prefix_path="package://flexiv_description/" />
+      </xacro:if>
+      <!-- Rizon4, Rizon4M or Rizon4s -->
+      <xacro:unless value="${rizon_type=='Rizon4R'}">
+        <xacro:include filename="$(find flexiv_description)/urdf/rizon4_joints_links.xacro" />
+        <xacro:rizon4_joints_links rizon_type="${rizon_type}" prefix="${prefix}"
+          mesh_prefix_path="package://flexiv_description/" />
+      </xacro:unless>
       <!-- ros2 control include -->
       <xacro:include filename="$(find flexiv_description)/urdf/rizon4.ros2_control.xacro" />
@@ -32,6 +40,6 @@
       />
     </xacro:if>
-    <!-- Rizon 10 or 10s-->
-    <xacro:if value="${rizon_type=='rizon10' or rizon_type=='rizon10s'}">
+    <!-- Rizon10 or 10s-->
+    <xacro:if value="${rizon_type=='Rizon10' or rizon_type=='Rizon10s'}">
       <xacro:include filename="$(find flexiv_description)/urdf/rizon10_joints_links.xacro" />
       <xacro:rizon10_joints_links rizon_type="${rizon_type}" prefix="${prefix}"
