Commit message: Add FT03-D1 sensor loading to Rizon4, Rizon4R and Rizon10 models

File: flexiv_description/urdf/rizon.urdf.xacro (robot description, xacro)
@@ -2,7 +2,7 @@
 <robot xmlns:xacro="http://www.ros.org/wiki/xacro" name="rizon">
   <!-- 'rizon_type' values: Rizon4, Rizon4s, Rizon10, Rizon10s -->
-  <xacro:arg name="rizon_type" default="Rizon4"/>
+  <xacro:arg name="rizon_type" default="Rizon4" />
   <!-- import main macro -->
-  <xacro:include filename="$(find flexiv_description)/urdf/rizon_macro.xacro"/>
+  <xacro:include filename="$(find flexiv_description)/urdf/rizon_macro.xacro" />
   <!-- parameters -->
   <xacro:arg name="arm_prefix" default="" />
@@ -10,4 +10,5 @@
   <xacro:arg name="load_gripper" default="false" />
   <xacro:arg name="gripper_name" default="Flexiv-GN01" />
+  <xacro:arg name="load_mounted_ft_sensor" default="false" />
   <xacro:arg name="use_fake_hardware" default="false" />
   <xacro:arg name="fake_sensor_commands" default="false" />
@@ -19,4 +20,5 @@
     gripper_name="$(arg gripper_name)"
     use_fake_hardware="$(arg use_fake_hardware)"
+    load_mounted_ft_sensor="$(arg load_mounted_ft_sensor)"
     fake_sensor_commands="$(arg fake_sensor_commands)">
   </xacro:rizon_robot>

File: flexiv_description/urdf/rizon10_joints_links.xacro (robot description, xacro)
@@ -4,8 +4,10 @@
     rizon_type = "Rizon10", "Rizon10s"
     prefix = "Rizon10-123456_"
+    load_mounted_ft_sensor = false
     mesh_prefix_path = "", "package://flexiv_description/"
     NOTE: accurate kinematic but approximated dynamics parameters
   -->
-  <xacro:macro name="rizon10_joints_links" params="rizon_type prefix mesh_prefix_path">
+  <xacro:macro name="rizon10_joints_links"
+    params="rizon_type prefix load_mounted_ft_sensor mesh_prefix_path">
     <!-- JOINTS-->
     <joint name="${prefix}base_joint" type="fixed">
@@ -79,5 +81,10 @@
     <joint name="${prefix}link7_to_flange" type="fixed">
       <parent link="${prefix}link7" />
-      <child link="${prefix}flange" />
+      <xacro:if value="${load_mounted_ft_sensor}">
+        <child link="${prefix}wrist-sensor.base_link" />
+      </xacro:if>
+      <xacro:unless value="${load_mounted_ft_sensor}">
+        <child link="${prefix}flange" />
+      </xacro:unless>
       <xacro:if value="${rizon_type=='Rizon10'}">
         <origin xyz="0.0 0.0 0.081" rpy="0 0 ${-pi}" />
@@ -325,4 +332,77 @@
       </xacro:if>
     </link>
+    <!-- FT03-D1 wrist sensor -->
+    <xacro:if value="${load_mounted_ft_sensor}">
+      <joint name="${prefix}wrist-sensor.remove_rizon_flange_body" type="fixed">
+        <origin rpy="0 0 0" xyz="0 0 -0.016" />
+        <parent link="${prefix}wrist-sensor.base_link" />
+        <child link="${prefix}wrist-sensor.proximal_link" />
+        <axis xyz="0 0 1" />
+      </joint>
+      <joint name="${prefix}wrist-sensor.proximal_link_to_sensing_frame" type="fixed">
+        <origin rpy="0 0 0" xyz="0 0 0.0235" />
+        <parent link="${prefix}wrist-sensor.proximal_link" />
+        <child link="${prefix}wrist-sensor.distal_link" />
+        <axis xyz="0 0 1" />
+      </joint>
+      <joint name="${prefix}wrist-sensor.sensing_frame_to_flange" type="fixed">
+        <parent link="${prefix}wrist-sensor.distal_link" />
+        <child link="${prefix}flange" />
+        <origin rpy="0 0 0" xyz="0.0 0.0 0.0285" />
+      </joint>
+      <link name="${prefix}wrist-sensor.base_link">
+        <inertial>
+          <mass value="0.0" />
+          <origin rpy="0 0 0" xyz="0.0 0.0 0.0" />
+          <inertia ixx="0.0" ixy="0.0" ixz="0.0" iyy="0.0" iyz="0.0" izz="0.0" />
+        </inertial>
+      </link>
+      <link name="${prefix}wrist-sensor.proximal_link">
+        <inertial>
+          <origin rpy="0 0 0" xyz="0 0 0.01955" />
+          <mass value="0.149" />
+          <inertia ixx="0.0" ixy="0.0" ixz="0.0" iyy="0.0" iyz="0.0" izz="0.0" />
+        </inertial>
+        <visual name="shell">
+          <origin rpy="0 0 0" xyz="0 0 0" />
+          <geometry>
+            <mesh filename="${mesh_prefix_path}meshes/FT03-D1/visual/proximal.obj"
+              scale="1 1 1" />
+          </geometry>
+        </visual>
+        <collision name="convex_mesh">
+          <origin xyz="0 0 0" rpy="0 0 0" />
+          <geometry>
+            <mesh filename="${mesh_prefix_path}meshes/FT03-D1/collision/proximal.stl" />
+          </geometry>
+        </collision>
+      </link>
+      <link name="${prefix}wrist-sensor.distal_link">
+        <inertial>
+          <mass value="0.249" />
+          <origin rpy="0 0 0" xyz="0 0 0.0085" />
+          <inertia ixx="1.05E-4" ixy="0" ixz="0" iyy="1.05E-4" iyz="-0" izz="1.81E-4" />
+        </inertial>
+        <visual name="shell">
+          <origin rpy="0 0 0" xyz="0 0 0" />
+          <geometry>
+            <mesh filename="${mesh_prefix_path}meshes/FT03-D1/visual/distal.obj" />
+          </geometry>
+        </visual>
+        <visual name="ring">
+          <origin rpy="0 0 0" xyz="0 0 0" />
+          <geometry>
+            <mesh filename="${mesh_prefix_path}meshes/FT03-D1/visual/ring.obj"
+              scale="0.039 0.039 0.002" />
+          </geometry>
+        </visual>
+        <collision name="convex_mesh">
+          <origin xyz="0 0 0" rpy="0 0 0" />
+          <geometry>
+            <mesh filename="${mesh_prefix_path}meshes/FT03-D1/collision/distal.stl" />
+          </geometry>
+        </collision>
+      </link>
+    </xacro:if>
     <link name="${prefix}flange">
       <inertial>

File: flexiv_description/urdf/rizon4_joints_links.xacro (robot description, xacro)
@@ -4,8 +4,10 @@
     rizon_type = "Rizon4", "Rizon4M", "Rizon4s"
     prefix = "Rizon4-123456_"
+    load_mounted_ft_sensor = false
     mesh_prefix_path = "", "package://flexiv_description/"
     NOTE: accurate kinematic but approximated dynamics parameters
   -->
-  <xacro:macro name="rizon4_joints_links" params="rizon_type prefix mesh_prefix_path">
+  <xacro:macro name="rizon4_joints_links"
+    params="rizon_type prefix load_mounted_ft_sensor mesh_prefix_path">
     <!-- JOINTS-->
     <joint name="${prefix}base_joint" type="fixed">
@@ -79,5 +81,10 @@
     <joint name="${prefix}link7_to_flange" type="fixed">
       <parent link="${prefix}link7" />
-      <child link="${prefix}flange" />
+      <xacro:if value="${load_mounted_ft_sensor}">
+        <child link="${prefix}wrist-sensor.base_link" />
+      </xacro:if>
+      <xacro:unless value="${load_mounted_ft_sensor}">
+        <child link="${prefix}flange" />
+      </xacro:unless>
       <xacro:if value="${rizon_type=='Rizon4' or rizon_type=='Rizon4M'}">
         <origin xyz="0.0 0.0 0.081" rpy="0 0 ${-pi}" />
@@ -325,4 +332,77 @@
       </xacro:if>
     </link>
+    <!-- FT03-D1 wrist sensor -->
+    <xacro:if value="${load_mounted_ft_sensor}">
+      <joint name="${prefix}wrist-sensor.remove_rizon_flange_body" type="fixed">
+        <origin rpy="0 0 0" xyz="0 0 -0.016" />
+        <parent link="${prefix}wrist-sensor.base_link" />
+        <child link="${prefix}wrist-sensor.proximal_link" />
+        <axis xyz="0 0 1" />
+      </joint>
+      <joint name="${prefix}wrist-sensor.proximal_link_to_sensing_frame" type="fixed">
+        <origin rpy="0 0 0" xyz="0 0 0.0235" />
+        <parent link="${prefix}wrist-sensor.proximal_link" />
+        <child link="${prefix}wrist-sensor.distal_link" />
+        <axis xyz="0 0 1" />
+      </joint>
+      <joint name="${prefix}wrist-sensor.sensing_frame_to_flange" type="fixed">
+        <parent link="${prefix}wrist-sensor.distal_link" />
+        <child link="${prefix}flange" />
+        <origin rpy="0 0 0" xyz="0.0 0.0 0.0285" />
+      </joint>
+      <link name="${prefix}wrist-sensor.base_link">
+        <inertial>
+          <mass value="0.0" />
+          <origin rpy="0 0 0" xyz="0.0 0.0 0.0" />
+          <inertia ixx="0.0" ixy="0.0" ixz="0.0" iyy="0.0" iyz="0.0" izz="0.0" />
+        </inertial>
+      </link>
+      <link name="${prefix}wrist-sensor.proximal_link">
+        <inertial>
+          <origin rpy="0 0 0" xyz="0 0 0.01955" />
+          <mass value="0.149" />
+          <inertia ixx="0.0" ixy="0.0" ixz="0.0" iyy="0.0" iyz="0.0" izz="0.0" />
+        </inertial>
+        <visual name="shell">
+          <origin rpy="0 0 0" xyz="0 0 0" />
+          <geometry>
+            <mesh filename="${mesh_prefix_path}meshes/FT03-D1/visual/proximal.obj"
+              scale="1 1 1" />
+          </geometry>
+        </visual>
+        <collision name="convex_mesh">
+          <origin xyz="0 0 0" rpy="0 0 0" />
+          <geometry>
+            <mesh filename="${mesh_prefix_path}meshes/FT03-D1/collision/proximal.stl" />
+          </geometry>
+        </collision>
+      </link>
+      <link name="${prefix}wrist-sensor.distal_link">
+        <inertial>
+          <mass value="0.249" />
+          <origin rpy="0 0 0" xyz="0 0 0.0085" />
+          <inertia ixx="1.05E-4" ixy="0" ixz="0" iyy="1.05E-4" iyz="-0" izz="1.81E-4" />
+        </inertial>
+        <visual name="shell">
+          <origin rpy="0 0 0" xyz="0 0 0" />
+          <geometry>
+            <mesh filename="${mesh_prefix_path}meshes/FT03-D1/visual/distal.obj" />
+          </geometry>
+        </visual>
+        <visual name="ring">
+          <origin rpy="0 0 0" xyz="0 0 0" />
+          <geometry>
+            <mesh filename="${mesh_prefix_path}meshes/FT03-D1/visual/ring.obj"
+              scale="0.039 0.039 0.002" />
+          </geometry>
+        </visual>
+        <collision name="convex_mesh">
+          <origin xyz="0 0 0" rpy="0 0 0" />
+          <geometry>
+            <mesh filename="${mesh_prefix_path}meshes/FT03-D1/collision/distal.stl" />
+          </geometry>
+        </collision>
+      </link>
+    </xacro:if>
     <link name="${prefix}flange">
       <inertial>

File: flexiv_description/urdf/rizon4r_joints_links.xacro (robot description, xacro)
@@ -4,8 +4,10 @@
     rizon_type = "Rizon4R"
     prefix = "Rizon4R-123456_"
+    load_mounted_ft_sensor = false
     mesh_prefix_path = "", "package://flexiv_description/"
     NOTE: accurate kinematic but approximated dynamics parameters
   -->
-  <xacro:macro name="rizon4r_joints_links" params="rizon_type prefix mesh_prefix_path">
+  <xacro:macro name="rizon4r_joints_links"
+    params="rizon_type prefix load_mounted_ft_sensor mesh_prefix_path">
     <!-- JOINTS-->
     <joint name="${prefix}base_joint" type="fixed">
@@ -79,5 +81,10 @@
     <joint name="${prefix}link7_to_flange" type="fixed">
       <parent link="${prefix}link7" />
-      <child link="${prefix}flange" />
+      <xacro:if value="${load_mounted_ft_sensor}">
+        <child link="${prefix}wrist-sensor.base_link" />
+      </xacro:if>
+      <xacro:unless value="${load_mounted_ft_sensor}">
+        <child link="${prefix}flange" />
+      </xacro:unless>
       <origin xyz="0.0 0.0 -0.081" rpy="${pi} 0 0" />
     </joint>
@@ -292,4 +299,77 @@
       </collision>
     </link>
+    <!-- FT03-D1 wrist sensor -->
+    <xacro:if value="${load_mounted_ft_sensor}">
+      <joint name="${prefix}wrist-sensor.remove_rizon_flange_body" type="fixed">
+        <origin rpy="0 0 0" xyz="0 0 -0.016" />
+        <parent link="${prefix}wrist-sensor.base_link" />
+        <child link="${prefix}wrist-sensor.proximal_link" />
+        <axis xyz="0 0 1" />
+      </joint>
+      <joint name="${prefix}wrist-sensor.proximal_link_to_sensing_frame" type="fixed">
+        <origin rpy="0 0 0" xyz="0 0 0.0235" />
+        <parent link="${prefix}wrist-sensor.proximal_link" />
+        <child link="${prefix}wrist-sensor.distal_link" />
+        <axis xyz="0 0 1" />
+      </joint>
+      <joint name="${prefix}wrist-sensor.sensing_frame_to_flange" type="fixed">
+        <parent link="${prefix}wrist-sensor.distal_link" />
+        <child link="${prefix}flange" />
+        <origin rpy="0 0 0" xyz="0.0 0.0 0.0285" />
+      </joint>
+      <link name="${prefix}wrist-sensor.base_link">
+        <inertial>
+          <mass value="0.0" />
+          <origin rpy="0 0 0" xyz="0.0 0.0 0.0" />
+          <inertia ixx="0.0" ixy="0.0" ixz="0.0" iyy="0.0" iyz="0.0" izz="0.0" />
+        </inertial>
+      </link>
+      <link name="${prefix}wrist-sensor.proximal_link">
+        <inertial>
+          <origin rpy="0 0 0" xyz="0 0 0.01955" />
+          <mass value="0.149" />
+          <inertia ixx="0.0" ixy="0.0" ixz="0.0" iyy="0.0" iyz="0.0" izz="0.0" />
+        </inertial>
+        <visual name="shell">
+          <origin rpy="0 0 0" xyz="0 0 0" />
+          <geometry>
+            <mesh filename="${mesh_prefix_path}meshes/FT03-D1/visual/proximal.obj"
+              scale="1 1 1" />
+          </geometry>
+        </visual>
+        <collision name="convex_mesh">
+          <origin xyz="0 0 0" rpy="0 0 0" />
+          <geometry>
+            <mesh filename="${mesh_prefix_path}meshes/FT03-D1/collision/proximal.stl" />
+          </geometry>
+        </collision>
+      </link>
+      <link name="${prefix}wrist-sensor.distal_link">
+        <inertial>
+          <mass value="0.249" />
+          <origin rpy="0 0 0" xyz="0 0 0.0085" />
+          <inertia ixx="1.05E-4" ixy="0" ixz="0" iyy="1.05E-4" iyz="-0" izz="1.81E-4" />
+        </inertial>
+        <visual name="shell">
+          <origin rpy="0 0 0" xyz="0 0 0" />
+          <geometry>
+            <mesh filename="${mesh_prefix_path}meshes/FT03-D1/visual/distal.obj" />
+          </geometry>
+        </visual>
+        <visual name="ring">
+          <origin rpy="0 0 0" xyz="0 0 0" />
+          <geometry>
+            <mesh filename="${mesh_prefix_path}meshes/FT03-D1/visual/ring.obj"
+              scale="0.039 0.039 0.002" />
+          </geometry>
+        </visual>
+        <collision name="convex_mesh">
+          <origin xyz="0 0 0" rpy="0 0 0" />
+          <geometry>
+            <mesh filename="${mesh_prefix_path}meshes/FT03-D1/collision/distal.stl" />
+          </geometry>
+        </collision>
+      </link>
+    </xacro:if>
     <link name="${prefix}flange">
       <inertial>

File: flexiv_description/urdf/rizon_macro.xacro (robot description, xacro)
@@ -8,4 +8,5 @@
     load_gripper:=false
     gripper_name:='Flexiv-GN01'
+    load_mounted_ft_sensor:=false
     use_fake_hardware:=false
     fake_sensor_commands:=false
@@ -13,4 +14,8 @@
     <!-- Prefix defaults to 'arm_prefix_robot_sn' -->
     <xacro:property name="prefix" value="${arm_prefix + robot_sn + '_'}" />
+    <!-- FT sensor mounting only supported for Rizon4, Rizon4R and Rizon10 -->
+    <xacro:unless value="${rizon_type=='Rizon4' or rizon_type=='Rizon4R' or rizon_type=='Rizon10'}">
+      <xacro:property name="load_mounted_ft_sensor" value="false" />
+    </xacro:unless>
     <!-- Load gripper -->
     <xacro:if value="${load_gripper and gripper_name=='Flexiv-GN01'}">
@@ -25,4 +30,5 @@
         <xacro:include filename="$(find flexiv_description)/urdf/rizon4r_joints_links.xacro" />
         <xacro:rizon4r_joints_links rizon_type="${rizon_type}" prefix="${prefix}"
+          load_mounted_ft_sensor="${load_mounted_ft_sensor}"
           mesh_prefix_path="package://flexiv_description/" />
       </xacro:if>
@@ -31,4 +37,5 @@
         <xacro:include filename="$(find flexiv_description)/urdf/rizon4_joints_links.xacro" />
         <xacro:rizon4_joints_links rizon_type="${rizon_type}" prefix="${prefix}"
+          load_mounted_ft_sensor="${load_mounted_ft_sensor}"
           mesh_prefix_path="package://flexiv_description/" />
       </xacro:unless>
@@ -44,4 +51,5 @@
       <xacro:include filename="$(find flexiv_description)/urdf/rizon10_joints_links.xacro" />
       <xacro:rizon10_joints_links rizon_type="${rizon_type}" prefix="${prefix}"
+        load_mounted_ft_sensor="${load_mounted_ft_sensor}"
         mesh_prefix_path="package://flexiv_description/" />
       <!-- ros2 control include -->
