Commit message: Sync launch files and configs, fix AICO1-4-V2 actuated joints and SRDF collisions, and update dependencies, CI and docs

File: flexiv_moveit_config/srdf/rizon_macro.srdf.xacro (robot description, xacro)
@@ -17,5 +17,5 @@
     </xacro:macro>
     <!-- 'prefix' is the fully-formed prefix, normally from compute_prefix above. -->
-    <xacro:macro name="rizon_srdf" params="prefix load_mounted_ft_sensor use_virtual_joint:=true">
+    <xacro:macro name="rizon_srdf" params="prefix load_mounted_ft_sensor">
         <group name="${prefix}arm">
             <chain base_link="${prefix}base_link" tip_link="${prefix}flange" />
@@ -30,8 +30,4 @@
             <joint name="${prefix}joint7" value="0" />
         </group_state>
-        <xacro:if value="${use_virtual_joint}">
-            <virtual_joint name="virtual_joint" type="fixed" parent_frame="world"
-                child_link="${prefix}base_link" />
-        </xacro:if>
         <disable_collisions link1="${prefix}base_link" link2="${prefix}link1" reason="Adjacent" />
         <disable_collisions link1="${prefix}base_link" link2="${prefix}link2" reason="Never" />
