Commit message: Add MoveIt configuration files for AICO robots and update SRDF for dual arms

File: flexiv_moveit_config/srdf/aico1.srdf.xacro (robot description, xacro)
@@ -13,5 +13,5 @@
         load_mounted_ft_sensor="$(arg load_mounted_ft_sensor)" use_virtual_joint="false" />
     <!-- Prefixes -->
-    <xacro:property name="prefix" value="${arm_prefix + robot_sn + '_'}" />
+    <xacro:property name="prefix" value="$(arg arm_prefix)$(arg robot_sn)_" />
     <xacro:property name="platform_prefix" value="$(arg platform_prefix)" />
     <!-- Virtual Joint and Platform Group -->
@@ -19,12 +19,14 @@
         <virtual_joint name="virtual_joint" type="fixed" parent_frame="world"
             child_link="${platform_prefix}aico1_x1_base_link" />
-        <group name="aico1_x1_platform">
-            <chain base_link="${platform_prefix}aico1_x1_base_link" tip_link="${prefix}base_link" />
+        <group name="${platform_prefix}aico1_x1_platform_${prefix}arm">
+            <chain base_link="${platform_prefix}aico1_x1_base_link" tip_link="${prefix}flange" />
+        </group>
     </xacro:if>
     <xacro:if value="${'$(arg platform_type)' == 'X2'}">
         <virtual_joint name="virtual_joint" type="fixed" parent_frame="world"
             child_link="${platform_prefix}aico1_x2_agv" />
-        <group name="aico1_x2_platform">
-            <chain base_link="${platform_prefix}aico1_x2_base_link" tip_link="${prefix}base_link" />
+        <group name="${platform_prefix}aico1_x2_platform_${prefix}arm">
+            <chain base_link="${platform_prefix}aico1_x2_base_link" tip_link="${prefix}flange" />
+        </group>
     </xacro:if>
     <!-- Platform Collisions -->

File: flexiv_moveit_config/srdf/aico2.srdf.xacro (robot description, xacro)
@@ -10,16 +10,16 @@
     <xacro:arg name="load_mounted_ft_sensor_left" default="false" />
     <xacro:arg name="load_mounted_ft_sensor_right" default="false" />
-    <xacro:arg name="prefix_left" default="left_" />
-    <xacro:arg name="prefix_right" default="right_" />
+    <xacro:arg name="arm_prefix_left" default="left_" />
+    <xacro:arg name="arm_prefix_right" default="right_" />
     <xacro:include filename="$(find flexiv_moveit_config)/srdf/rizon_macro.srdf.xacro" />
     <!-- Left Arm -->
-    <xacro:rizon_srdf arm_prefix="$(arg prefix_left)" robot_sn="$(arg robot_sn_left)"
+    <xacro:rizon_srdf arm_prefix="$(arg arm_prefix_left)" robot_sn="$(arg robot_sn_left)"
         load_mounted_ft_sensor="$(arg load_mounted_ft_sensor_left)" use_virtual_joint="false" />
     <!-- Right Arm -->
-    <xacro:rizon_srdf arm_prefix="$(arg prefix_right)" robot_sn="$(arg robot_sn_right)"
+    <xacro:rizon_srdf arm_prefix="$(arg arm_prefix_right)" robot_sn="$(arg robot_sn_right)"
         load_mounted_ft_sensor="$(arg load_mounted_ft_sensor_right)" use_virtual_joint="false" />
     <!-- Prefixes -->
-    <xacro:property name="prefix_left" value="${prefix_left + robot_sn_left + '_'}" />
-    <xacro:property name="prefix_right" value="${prefix_right + robot_sn_right + '_'}" />
+    <xacro:property name="prefix_left" value="$(arg arm_prefix_left)$(arg robot_sn_left)_" />
+    <xacro:property name="prefix_right" value="$(arg arm_prefix_right)$(arg robot_sn_right)_" />
     <xacro:property name="platform_prefix" value="$(arg platform_prefix)" />
     <!-- Virtual Joint and Platform Group -->
@@ -27,12 +27,14 @@
         <virtual_joint name="virtual_joint" type="fixed" parent_frame="world"
             child_link="${platform_prefix}aico2_x1_base_link" />
-        <group name="aico2_x1_platform">
-            <chain base_link="${platform_prefix}aico2_x1_base_link" tip_link="${prefix_left}base_link" />
+        <group name="${platform_prefix}aico2_x1_platform_${prefix_left}arm">
+            <chain base_link="${platform_prefix}aico2_x1_base_link" tip_link="${prefix_left}flange" />
+        </group>
     </xacro:if>
     <xacro:if value="${'$(arg platform_type)' == 'X2'}">
         <virtual_joint name="virtual_joint" type="fixed" parent_frame="world"
             child_link="${platform_prefix}aico2_x2_base_link" />
-        <group name="aico2_x2_platform">
-            <chain base_link="${platform_prefix}aico2_x2_base_link" tip_link="${prefix_left}base_link" />
+        <group name="${platform_prefix}aico2_x2_platform_${prefix_left}arm">
+            <chain base_link="${platform_prefix}aico2_x2_base_link" tip_link="${prefix_left}flange" />
+        </group>
     </xacro:if>
     <!-- Platform Collisions -->
@@ -52,4 +54,7 @@
         <disable_collisions link1="${prefix_right}link1" link2="${platform_prefix}aico2_x1_link1" reason="Never" />
         <disable_collisions link1="${prefix_right}link1" link2="${platform_prefix}aico2_x1_base_link" reason="Never" />
+        <!-- Left and Right Arms -->
+        <disable_collisions link1="${prefix_left}base_link" link2="${prefix_right}base_link" reason="Never" />
+        <disable_collisions link1="${prefix_left}link1" link2="${prefix_right}link1" reason="Never" />
         <!-- Platform internal -->
         <disable_collisions link1="${platform_prefix}aico2_x1_base_link" link2="${platform_prefix}aico2_x1_link1" reason="Adjacent" />

File: flexiv_moveit_config/srdf/rizon_dual.srdf.xacro (robot description, xacro)
@@ -17,4 +17,7 @@
     <xacro:rizon_srdf arm_prefix="$(arg prefix_right)" robot_sn="$(arg robot_sn_right)"
         load_mounted_ft_sensor="$(arg load_mounted_ft_sensor_right)" />
+    <!-- Left and Right Arms Collisions -->
+    <disable_collisions link1="${prefix_left}base_link" link2="${prefix_right}base_link" reason="Never" />
+    <disable_collisions link1="${prefix_left}link1" link2="${prefix_right}link1" reason="Never" />
     <!-- Load grippers -->
     <xacro:if value="$(arg load_gripper_left)">
