Commit message: Update AICO launch files to use external axis parameters

File: flexiv_moveit_config/srdf/aico1.srdf.xacro (robot description, xacro)
@@ -2,6 +2,6 @@
 <robot xmlns:xacro="http://wiki.ros.org/xacro" name="aico1">
     <!-- parameters -->
-    <xacro:arg name="platform_type" default="X1" />
-    <xacro:arg name="platform_prefix" default="" />
+    <xacro:arg name="external_axis_type" default="aico1_platform_x1" />
+    <xacro:arg name="external_axis_prefix" default="" />
     <xacro:arg name="arm_prefix" default="" />
     <xacro:arg name="robot_sn" default="" />
@@ -14,45 +14,45 @@
     <!-- Prefixes -->
     <xacro:property name="prefix" value="$(arg arm_prefix)$(arg robot_sn)_" />
-    <xacro:property name="platform_prefix" value="$(arg platform_prefix)" />
+    <xacro:property name="external_axis_prefix" value="$(arg external_axis_prefix)" />
     <!-- Virtual Joint and Platform Group -->
-    <xacro:if value="${'$(arg platform_type)' == 'X1'}">
+    <xacro:if value="${'$(arg external_axis_type)' == 'aico1_platform_x1'}">
         <virtual_joint name="virtual_joint" type="fixed" parent_frame="world"
-            child_link="${platform_prefix}aico1_x1_base_link" />
-        <group name="${platform_prefix}aico1_x1_platform_${prefix}arm">
-            <chain base_link="${platform_prefix}aico1_x1_base_link" tip_link="${prefix}flange" />
+            child_link="${external_axis_prefix}aico1_x1_base_link" />
+        <group name="${external_axis_prefix}aico1_x1_platform_${prefix}arm">
+            <chain base_link="${external_axis_prefix}aico1_x1_base_link" tip_link="${prefix}flange" />
         </group>
     </xacro:if>
-    <xacro:if value="${'$(arg platform_type)' == 'X2'}">
+    <xacro:if value="${'$(arg external_axis_type)' == 'aico1_platform_x2'}">
         <virtual_joint name="virtual_joint" type="fixed" parent_frame="world"
-            child_link="${platform_prefix}aico1_x2_agv" />
-        <group name="${platform_prefix}aico1_x2_platform_${prefix}arm">
-            <chain base_link="${platform_prefix}aico1_x2_base_link" tip_link="${prefix}flange" />
+            child_link="${external_axis_prefix}aico1_x2_agv" />
+        <group name="${external_axis_prefix}aico1_x2_platform_${prefix}arm">
+            <chain base_link="${external_axis_prefix}aico1_x2_base_link" tip_link="${prefix}flange" />
         </group>
     </xacro:if>
     <!-- Platform Collisions -->
-    <xacro:if value="${'$(arg platform_type)' == 'X1'}">
-        <disable_collisions link1="${prefix}base_link" link2="${platform_prefix}aico1_x1_link2" reason="Adjacent" />
-        <disable_collisions link1="${prefix}base_link" link2="${platform_prefix}aico1_x1_link1" reason="Never" />
-        <disable_collisions link1="${prefix}base_link" link2="${platform_prefix}aico1_x1_base_link" reason="Never" />
-        <disable_collisions link1="${prefix}link1" link2="${platform_prefix}aico1_x1_link2" reason="Never" />
-        <disable_collisions link1="${prefix}link1" link2="${platform_prefix}aico1_x1_link1" reason="Never" />
-        <disable_collisions link1="${prefix}link1" link2="${platform_prefix}aico1_x1_base_link" reason="Never" />
-        <disable_collisions link1="${platform_prefix}aico1_x1_base_link" link2="${platform_prefix}aico1_x1_link1" reason="Adjacent" />
-        <disable_collisions link1="${platform_prefix}aico1_x1_base_link" link2="${platform_prefix}aico1_x1_link2" reason="Never" />
-        <disable_collisions link1="${platform_prefix}aico1_x1_link1" link2="${platform_prefix}aico1_x1_link2" reason="Adjacent" />
+    <xacro:if value="${'$(arg external_axis_type)' == 'aico1_platform_x1'}">
+        <disable_collisions link1="${prefix}base_link" link2="${external_axis_prefix}aico1_x1_link2" reason="Adjacent" />
+        <disable_collisions link1="${prefix}base_link" link2="${external_axis_prefix}aico1_x1_link1" reason="Never" />
+        <disable_collisions link1="${prefix}base_link" link2="${external_axis_prefix}aico1_x1_base_link" reason="Never" />
+        <disable_collisions link1="${prefix}link1" link2="${external_axis_prefix}aico1_x1_link2" reason="Never" />
+        <disable_collisions link1="${prefix}link1" link2="${external_axis_prefix}aico1_x1_link1" reason="Never" />
+        <disable_collisions link1="${prefix}link1" link2="${external_axis_prefix}aico1_x1_base_link" reason="Never" />
+        <disable_collisions link1="${external_axis_prefix}aico1_x1_base_link" link2="${external_axis_prefix}aico1_x1_link1" reason="Adjacent" />
+        <disable_collisions link1="${external_axis_prefix}aico1_x1_base_link" link2="${external_axis_prefix}aico1_x1_link2" reason="Never" />
+        <disable_collisions link1="${external_axis_prefix}aico1_x1_link1" link2="${external_axis_prefix}aico1_x1_link2" reason="Adjacent" />
     </xacro:if>
-    <xacro:if value="${'$(arg platform_type)' == 'X2'}">
-        <disable_collisions link1="${prefix}base_link" link2="${platform_prefix}aico1_x2_link1" reason="Adjacent" />
-        <disable_collisions link1="${prefix}base_link" link2="${platform_prefix}aico1_x2_base_link" reason="Never" />
-        <disable_collisions link1="${prefix}base_link" link2="${platform_prefix}aico1_x2_neck_link" reason="Never" />
-        <disable_collisions link1="${prefix}base_link" link2="${platform_prefix}aico1_x2_head_link" reason="Never" />
-        <disable_collisions link1="${prefix}link1" link2="${platform_prefix}aico1_x2_link1" reason="Never" />
-        <disable_collisions link1="${prefix}link1" link2="${platform_prefix}aico1_x2_base_link" reason="Never" />
-        <disable_collisions link1="${prefix}link1" link2="${platform_prefix}aico1_x2_neck_link" reason="Never" />
-        <disable_collisions link1="${prefix}link1" link2="${platform_prefix}aico1_x2_head_link" reason="Never" />
-        <disable_collisions link1="${platform_prefix}aico1_x2_base_link" link2="${platform_prefix}aico1_x2_link1" reason="Adjacent" />
-        <disable_collisions link1="${platform_prefix}aico1_x2_base_link" link2="${platform_prefix}aico1_x2_neck_link" reason="Never" />
-        <disable_collisions link1="${platform_prefix}aico1_x2_link1" link2="${platform_prefix}aico1_x2_neck_link" reason="Adjacent" />
-        <disable_collisions link1="${platform_prefix}aico1_x2_neck_link" link2="${platform_prefix}aico1_x2_head_link" reason="Adjacent" />
+    <xacro:if value="${'$(arg external_axis_type)' == 'aico1_platform_x2'}">
+        <disable_collisions link1="${prefix}base_link" link2="${external_axis_prefix}aico1_x2_link1" reason="Adjacent" />
+        <disable_collisions link1="${prefix}base_link" link2="${external_axis_prefix}aico1_x2_base_link" reason="Never" />
+        <disable_collisions link1="${prefix}base_link" link2="${external_axis_prefix}aico1_x2_neck_link" reason="Never" />
+        <disable_collisions link1="${prefix}base_link" link2="${external_axis_prefix}aico1_x2_head_link" reason="Never" />
+        <disable_collisions link1="${prefix}link1" link2="${external_axis_prefix}aico1_x2_link1" reason="Never" />
+        <disable_collisions link1="${prefix}link1" link2="${external_axis_prefix}aico1_x2_base_link" reason="Never" />
+        <disable_collisions link1="${prefix}link1" link2="${external_axis_prefix}aico1_x2_neck_link" reason="Never" />
+        <disable_collisions link1="${prefix}link1" link2="${external_axis_prefix}aico1_x2_head_link" reason="Never" />
+        <disable_collisions link1="${external_axis_prefix}aico1_x2_base_link" link2="${external_axis_prefix}aico1_x2_link1" reason="Adjacent" />
+        <disable_collisions link1="${external_axis_prefix}aico1_x2_base_link" link2="${external_axis_prefix}aico1_x2_neck_link" reason="Never" />
+        <disable_collisions link1="${external_axis_prefix}aico1_x2_link1" link2="${external_axis_prefix}aico1_x2_neck_link" reason="Adjacent" />
+        <disable_collisions link1="${external_axis_prefix}aico1_x2_neck_link" link2="${external_axis_prefix}aico1_x2_head_link" reason="Adjacent" />
     </xacro:if>
     <!-- Load gripper -->

File: flexiv_moveit_config/srdf/aico2.srdf.xacro (robot description, xacro)
@@ -2,6 +2,6 @@
 <robot xmlns:xacro="http://wiki.ros.org/xacro" name="aico2">
     <!-- parameters -->
-    <xacro:arg name="platform_type" default="X1" />
-    <xacro:arg name="platform_prefix" default="" />
+    <xacro:arg name="external_axis_type" default="aico2_platform_x1" />
+    <xacro:arg name="external_axis_prefix" default="" />
     <xacro:arg name="robot_sn_left" default="" />
     <xacro:arg name="robot_sn_right" default="" />
@@ -22,63 +22,66 @@
     <xacro:property name="prefix_left" value="$(arg arm_prefix_left)$(arg robot_sn_left)_" />
     <xacro:property name="prefix_right" value="$(arg arm_prefix_right)$(arg robot_sn_right)_" />
-    <xacro:property name="platform_prefix" value="$(arg platform_prefix)" />
-    <!-- Virtual Joint and Platform Group -->
-    <xacro:if value="${'$(arg platform_type)' == 'X1'}">
+    <xacro:property name="external_axis_prefix" value="$(arg external_axis_prefix)" />
+    <!-- Virtual Joint and External Axis Group -->
+    <xacro:if value="${'$(arg external_axis_type)' == 'aico2_platform_x1'}">
         <virtual_joint name="virtual_joint" type="fixed" parent_frame="world"
-            child_link="${platform_prefix}aico2_x1_base_link" />
-        <group name="${platform_prefix}aico2_x1_platform_${prefix_left}arm">
-            <chain base_link="${platform_prefix}aico2_x1_base_link" tip_link="${prefix_left}flange" />
+            child_link="${external_axis_prefix}aico2_x1_base_link" />
+        <group name="${external_axis_prefix}aico2_x1_platform_${prefix_left}arm">
+            <chain base_link="${external_axis_prefix}aico2_x1_base_link" tip_link="${prefix_left}flange" />
         </group>
     </xacro:if>
-    <xacro:if value="${'$(arg platform_type)' == 'X2'}">
+    <xacro:if value="${'$(arg external_axis_type)' == 'aico2_platform_x2'}">
         <virtual_joint name="virtual_joint" type="fixed" parent_frame="world"
-            child_link="${platform_prefix}aico2_x2_base_link" />
-        <group name="${platform_prefix}aico2_x2_platform_${prefix_left}arm">
-            <chain base_link="${platform_prefix}aico2_x2_base_link" tip_link="${prefix_left}flange" />
+            child_link="${external_axis_prefix}aico2_x2_base_link" />
+        <group name="${external_axis_prefix}aico2_x2_platform_${prefix_left}arm">
+            <chain base_link="${external_axis_prefix}aico2_x2_base_link" tip_link="${prefix_left}flange" />
         </group>
     </xacro:if>
-    <!-- Platform Collisions -->
-    <xacro:if value="${'$(arg platform_type)' == 'X1'}">
+    <!-- External Axis Collisions -->
+    <xacro:if value="${'$(arg external_axis_type)' == 'aico2_platform_x1'}">
         <!-- Left Arm -->
-        <disable_collisions link1="${prefix_left}base_link" link2="${platform_prefix}aico2_x1_link2" reason="Adjacent" />
-        <disable_collisions link1="${prefix_left}base_link" link2="${platform_prefix}aico2_x1_link1" reason="Never" />
-        <disable_collisions link1="${prefix_left}base_link" link2="${platform_prefix}aico2_x1_base_link" reason="Never" />
-        <disable_collisions link1="${prefix_left}link1" link2="${platform_prefix}aico2_x1_link2" reason="Never" />
-        <disable_collisions link1="${prefix_left}link1" link2="${platform_prefix}aico2_x1_link1" reason="Never" />
-        <disable_collisions link1="${prefix_left}link1" link2="${platform_prefix}aico2_x1_base_link" reason="Never" />
+        <disable_collisions link1="${prefix_left}base_link" link2="${external_axis_prefix}aico2_x1_link2" reason="Adjacent" />
+        <disable_collisions link1="${prefix_left}base_link" link2="${external_axis_prefix}aico2_x1_link1" reason="Never" />
+        <disable_collisions link1="${prefix_left}base_link" link2="${external_axis_prefix}aico2_x1_base_link" reason="Never" />
+        <disable_collisions link1="${prefix_left}link1" link2="${external_axis_prefix}aico2_x1_link2" reason="Never" />
+        <disable_collisions link1="${prefix_left}link1" link2="${external_axis_prefix}aico2_x1_link1" reason="Never" />
+        <disable_collisions link1="${prefix_left}link1" link2="${external_axis_prefix}aico2_x1_base_link" reason="Never" />
         <!-- Right Arm -->
-        <disable_collisions link1="${prefix_right}base_link" link2="${platform_prefix}aico2_x1_link2" reason="Adjacent" />
-        <disable_collisions link1="${prefix_right}base_link" link2="${platform_prefix}aico2_x1_link1" reason="Never" />
-        <disable_collisions link1="${prefix_right}base_link" link2="${platform_prefix}aico2_x1_base_link" reason="Never" />
-        <disable_collisions link1="${prefix_right}link1" link2="${platform_prefix}aico2_x1_link2" reason="Never" />
-        <disable_collisions link1="${prefix_right}link1" link2="${platform_prefix}aico2_x1_link1" reason="Never" />
-        <disable_collisions link1="${prefix_right}link1" link2="${platform_prefix}aico2_x1_base_link" reason="Never" />
+        <disable_collisions link1="${prefix_right}base_link" link2="${external_axis_prefix}aico2_x1_link2" reason="Adjacent" />
+        <disable_collisions link1="${prefix_right}base_link" link2="${external_axis_prefix}aico2_x1_link1" reason="Never" />
+        <disable_collisions link1="${prefix_right}base_link" link2="${external_axis_prefix}aico2_x1_base_link" reason="Never" />
+        <disable_collisions link1="${prefix_right}link1" link2="${external_axis_prefix}aico2_x1_link2" reason="Never" />
+        <disable_collisions link1="${prefix_right}link1" link2="${external_axis_prefix}aico2_x1_link1" reason="Never" />
+        <disable_collisions link1="${prefix_right}link1" link2="${external_axis_prefix}aico2_x1_base_link" reason="Never" />
         <!-- Left and Right Arms -->
         <disable_collisions link1="${prefix_left}base_link" link2="${prefix_right}base_link" reason="Never" />
         <disable_collisions link1="${prefix_left}link1" link2="${prefix_right}link1" reason="Never" />
-        <!-- Platform internal -->
-        <disable_collisions link1="${platform_prefix}aico2_x1_base_link" link2="${platform_prefix}aico2_x1_link1" reason="Adjacent" />
-        <disable_collisions link1="${platform_prefix}aico2_x1_base_link" link2="${platform_prefix}aico2_x1_link2" reason="Never" />
-        <disable_collisions link1="${platform_prefix}aico2_x1_link1" link2="${platform_prefix}aico2_x1_link2" reason="Adjacent" />
+        <!-- External Axis internal -->
+        <disable_collisions link1="${external_axis_prefix}aico2_x1_base_link" link2="${external_axis_prefix}aico2_x1_link1" reason="Adjacent" />
+        <disable_collisions link1="${external_axis_prefix}aico2_x1_base_link" link2="${external_axis_prefix}aico2_x1_link2" reason="Never" />
+        <disable_collisions link1="${external_axis_prefix}aico2_x1_link1" link2="${external_axis_prefix}aico2_x1_link2" reason="Adjacent" />
     </xacro:if>
-    <xacro:if value="${'$(arg platform_type)' == 'X2'}">
+    <xacro:if value="${'$(arg external_axis_type)' == 'aico2_platform_x2'}">
         <!-- Left Arm -->
-        <disable_collisions link1="${prefix_left}base_link" link2="${platform_prefix}aico2_x2_link2" reason="Adjacent" />
-        <disable_collisions link1="${prefix_left}base_link" link2="${platform_prefix}aico2_x2_link1" reason="Never" />
-        <disable_collisions link1="${prefix_left}base_link" link2="${platform_prefix}aico2_x2_base_link" reason="Never" />
-        <disable_collisions link1="${prefix_left}link1" link2="${platform_prefix}aico2_x2_link2" reason="Never" />
-        <disable_collisions link1="${prefix_left}link1" link2="${platform_prefix}aico2_x2_link1" reason="Never" />
-        <disable_collisions link1="${prefix_left}link1" link2="${platform_prefix}aico2_x2_base_link" reason="Never" />
+        <disable_collisions link1="${prefix_left}base_link" link2="${external_axis_prefix}aico2_x2_link2" reason="Adjacent" />
+        <disable_collisions link1="${prefix_left}base_link" link2="${external_axis_prefix}aico2_x2_link1" reason="Never" />
+        <disable_collisions link1="${prefix_left}base_link" link2="${external_axis_prefix}aico2_x2_base_link" reason="Never" />
+        <disable_collisions link1="${prefix_left}link1" link2="${external_axis_prefix}aico2_x2_link2" reason="Never" />
+        <disable_collisions link1="${prefix_left}link1" link2="${external_axis_prefix}aico2_x2_link1" reason="Never" />
+        <disable_collisions link1="${prefix_left}link1" link2="${external_axis_prefix}aico2_x2_base_link" reason="Never" />
         <!-- Right Arm -->
-        <disable_collisions link1="${prefix_right}base_link" link2="${platform_prefix}aico2_x2_link2" reason="Adjacent" />
-        <disable_collisions link1="${prefix_right}base_link" link2="${platform_prefix}aico2_x2_link1" reason="Never" />
-        <disable_collisions link1="${prefix_right}base_link" link2="${platform_prefix}aico2_x2_base_link" reason="Never" />
-        <disable_collisions link1="${prefix_right}link1" link2="${platform_prefix}aico2_x2_link2" reason="Never" />
-        <disable_collisions link1="${prefix_right}link1" link2="${platform_prefix}aico2_x2_link1" reason="Never" />
-        <disable_collisions link1="${prefix_right}link1" link2="${platform_prefix}aico2_x2_base_link" reason="Never" />
-        <!-- Platform internal -->
-        <disable_collisions link1="${platform_prefix}aico2_x2_base_link" link2="${platform_prefix}aico2_x2_link1" reason="Adjacent" />
-        <disable_collisions link1="${platform_prefix}aico2_x2_base_link" link2="${platform_prefix}aico2_x2_link2" reason="Never" />
-        <disable_collisions link1="${platform_prefix}aico2_x2_link1" link2="${platform_prefix}aico2_x2_link2" reason="Adjacent" />
+        <disable_collisions link1="${prefix_right}base_link" link2="${external_axis_prefix}aico2_x2_link2" reason="Adjacent" />
+        <disable_collisions link1="${prefix_right}base_link" link2="${external_axis_prefix}aico2_x2_link1" reason="Never" />
+        <disable_collisions link1="${prefix_right}base_link" link2="${external_axis_prefix}aico2_x2_base_link" reason="Never" />
+        <disable_collisions link1="${prefix_right}link1" link2="${external_axis_prefix}aico2_x2_link2" reason="Never" />
+        <disable_collisions link1="${prefix_right}link1" link2="${external_axis_prefix}aico2_x2_link1" reason="Never" />
+        <disable_collisions link1="${prefix_right}link1" link2="${external_axis_prefix}aico2_x2_base_link" reason="Never" />
+        <!-- Left and Right Arms -->
+        <disable_collisions link1="${prefix_left}base_link" link2="${prefix_right}base_link" reason="Never" />
+        <disable_collisions link1="${prefix_left}link1" link2="${prefix_right}link1" reason="Never" />
+        <!-- External Axis internal -->
+        <disable_collisions link1="${external_axis_prefix}aico2_x2_base_link" link2="${external_axis_prefix}aico2_x2_link1" reason="Adjacent" />
+        <disable_collisions link1="${external_axis_prefix}aico2_x2_base_link" link2="${external_axis_prefix}aico2_x2_link2" reason="Never" />
+        <disable_collisions link1="${external_axis_prefix}aico2_x2_link1" link2="${external_axis_prefix}aico2_x2_link2" reason="Adjacent" />
     </xacro:if>
     <!-- Load grippers -->
