Commit message: Add configuration files for AICO robot kinematics, planning, and joint limits

File: flexiv_moveit_config/srdf/rizon_dual.srdf.xacro (robot description, xacro)
@@ -17,4 +17,7 @@
     <xacro:rizon_srdf arm_prefix="$(arg prefix_right)" robot_sn="$(arg robot_sn_right)"
         load_mounted_ft_sensor="$(arg load_mounted_ft_sensor_right)" />
+    <!-- Left and Right Arms Collisions -->
+    <disable_collisions link1="$(arg prefix_left)base_link" link2="$(arg prefix_right)base_link" reason="Never" />
+    <disable_collisions link1="$(arg prefix_left)link1" link2="$(arg prefix_right)link1" reason="Never" />
     <!-- Load grippers -->
     <xacro:if value="$(arg load_gripper_left)">

File: flexiv_moveit_config/srdf/rizon_macro.srdf.xacro (robot description, xacro)
@@ -1,5 +1,5 @@
 <?xml version="1.0" encoding="UTF-8"?>
 <robot xmlns:xacro="http://www.ros.org/wiki/xacro">
-    <xacro:macro name="rizon_srdf" params="arm_prefix robot_sn load_mounted_ft_sensor">
+    <xacro:macro name="rizon_srdf" params="arm_prefix robot_sn load_mounted_ft_sensor use_virtual_joint:=true">
         <!-- Prefix defaults to 'arm_prefix_robot_sn' -->
         <xacro:property name="prefix" value="${arm_prefix + robot_sn + '_'}" />
@@ -16,6 +16,8 @@
             <joint name="${prefix}joint7" value="0" />
         </group_state>
-        <virtual_joint name="virtual_joint" type="fixed" parent_frame="world"
-            child_link="${prefix}base_link" />
+        <xacro:if value="${use_virtual_joint}">
+            <virtual_joint name="virtual_joint" type="fixed" parent_frame="world"
+                child_link="${prefix}base_link" />
+        </xacro:if>
         <disable_collisions link1="${prefix}base_link" link2="${prefix}link1" reason="Adjacent" />
         <disable_collisions link1="${prefix}base_link" link2="${prefix}link2" reason="Never" />
@@ -40,16 +42,10 @@
         <xacro:if value="${load_mounted_ft_sensor}">
             <!-- Disable collisions for FT sensor fixed-link chain -->
-            <disable_collisions link1="${prefix}link7" link2="${prefix}wrist-sensor.base_link"
-                reason="Adjacent" />
-            <disable_collisions link1="${prefix}wrist-sensor.base_link"
-                link2="${prefix}wrist-sensor.proximal_link" reason="Adjacent" />
-            <disable_collisions link1="${prefix}wrist-sensor.proximal_link"
-                link2="${prefix}wrist-sensor.distal_link" reason="Adjacent" />
-            <disable_collisions link1="${prefix}wrist-sensor.distal_link" link2="${prefix}flange"
-                reason="Adjacent" />
-            <disable_collisions link1="${prefix}link7" link2="${prefix}wrist-sensor.proximal_link"
-                reason="Adjacent" />
-            <disable_collisions link1="${prefix}link7" link2="${prefix}wrist-sensor.distal_link"
-                reason="Adjacent" />
+            <disable_collisions link1="${prefix}link7" link2="${prefix}wrist-sensor.base_link" reason="Adjacent" />
+            <disable_collisions link1="${prefix}wrist-sensor.base_link" link2="${prefix}wrist-sensor.proximal_link" reason="Adjacent" />
+            <disable_collisions link1="${prefix}wrist-sensor.proximal_link" link2="${prefix}wrist-sensor.distal_link" reason="Adjacent" />
+            <disable_collisions link1="${prefix}wrist-sensor.distal_link" link2="${prefix}flange" reason="Adjacent" />
+            <disable_collisions link1="${prefix}link7" link2="${prefix}wrist-sensor.proximal_link" reason="Adjacent" />
+            <disable_collisions link1="${prefix}link7" link2="${prefix}wrist-sensor.distal_link" reason="Adjacent" />
         </xacro:if>
     </xacro:macro>

Commit message: Update rizon_dual SRDF to use dynamic arm prefixes for collision definitions

File: flexiv_moveit_config/srdf/rizon_dual.srdf.xacro (robot description, xacro)
@@ -17,7 +17,10 @@
     <xacro:rizon_srdf arm_prefix="$(arg prefix_right)" robot_sn="$(arg robot_sn_right)"
         load_mounted_ft_sensor="$(arg load_mounted_ft_sensor_right)" />
+    <!-- Arm Prefixes -->
+    <xacro:property name="left_arm_prefix" value="$(arg prefix_left)$(arg robot_sn_left)_" />
+    <xacro:property name="right_arm_prefix" value="$(arg prefix_right)$(arg robot_sn_right)_" />
     <!-- Left and Right Arms Collisions -->
-    <disable_collisions link1="$(arg prefix_left)base_link" link2="$(arg prefix_right)base_link" reason="Never" />
-    <disable_collisions link1="$(arg prefix_left)link1" link2="$(arg prefix_right)link1" reason="Never" />
+    <disable_collisions link1="${left_arm_prefix}base_link" link2="${right_arm_prefix}base_link" reason="Never" />
+    <disable_collisions link1="${left_arm_prefix}link1" link2="${right_arm_prefix}link1" reason="Never" />
     <!-- Load grippers -->
     <xacro:if value="$(arg load_gripper_left)">
