Commit message: Add robot_sn as naming prefix to MoveIt config files

File: flexiv_moveit_config/srdf/grav.srdf.xacro (robot description, xacro)
@@ -1,5 +1,7 @@
 <?xml version="1.0" encoding="UTF-8"?>
 <robot xmlns:xacro="http://www.ros.org/wiki/xacro">
-    <xacro:macro name="grav_srdf" params="name prefix">
+    <xacro:macro name="grav_srdf" params="arm_prefix robot_sn">
+        <!-- Prefix defaults to 'arm_prefix_robot_sn' -->
+        <xacro:property name="prefix" value="${arm_prefix + robot_sn + '_'}" />
         <group name="${prefix}grav_gripper">
             <joint name="${prefix}gripper_base_joint" />
@@ -30,5 +32,6 @@
             <joint name="${prefix}finger_width_joint" value="0.0" />
         </group_state>
-        <end_effector name="${prefix}grav_gripper" parent_link="${prefix}flange" group="${prefix}grav_gripper" parent_group="${prefix}${name}_arm"/>
+        <end_effector name="${prefix}grav_gripper" parent_link="${prefix}flange"
+            group="${prefix}grav_gripper" parent_group="${prefix}arm" />
         <disable_collisions link1="${prefix}grav_base_link" link2="${prefix}grav_tcp" reason="Never" />
         <disable_collisions link1="${prefix}grav_base_link" link2="${prefix}closed_fingers_tcp" reason="Never" />

File: flexiv_moveit_config/srdf/rizon.srdf.xacro (robot description, xacro)
@@ -1,16 +1,14 @@
 <?xml version="1.0" encoding="UTF-8"?>
-<robot xmlns:xacro="http://wiki.ros.org/xacro" name="(arg name)">
-    <!-- robot name parameter -->
-    <xacro:arg name="name" default="rizon" />
+<robot xmlns:xacro="http://wiki.ros.org/xacro" name="rizon">
     <!-- parameters -->
-    <xacro:arg name="prefix" default="" />
+    <xacro:arg name="arm_prefix" default="" />
+    <xacro:arg name="robot_sn" default="" />
     <xacro:arg name="load_gripper" default="false" />
-    <xacro:property name="name" value="$(arg name)"/>
     <xacro:include filename="$(find flexiv_moveit_config)/srdf/rizon_macro.srdf.xacro" />
-    <xacro:rizon_srdf name="${name}" prefix="$(arg prefix)" />
+    <xacro:rizon_srdf arm_prefix="$(arg arm_prefix)" robot_sn="$(arg robot_sn)" />
     <!-- Load gripper -->
     <xacro:if value="$(arg load_gripper)">
         <xacro:include filename="$(find flexiv_moveit_config)/srdf/grav.srdf.xacro" />
-        <xacro:grav_srdf name="${name}" prefix="$(arg prefix)" />
+        <xacro:grav_srdf arm_prefix="$(arg arm_prefix)" robot_sn="$(arg robot_sn)" />
     </xacro:if>
 </robot>

File: flexiv_moveit_config/srdf/rizon_macro.srdf.xacro (robot description, xacro)
@@ -1,38 +1,41 @@
 <?xml version="1.0" encoding="UTF-8"?>
 <robot xmlns:xacro="http://www.ros.org/wiki/xacro">
-    <xacro:macro name="rizon_srdf" params="prefix robot_sn">
-        <group name="${prefix}${robot_sn}_arm">
+    <xacro:macro name="rizon_srdf" params="arm_prefix robot_sn">
+        <!-- Prefix defaults to 'arm_prefix_robot_sn' -->
+        <xacro:property name="prefix" value="${arm_prefix + robot_sn + '_'}" />
+        <group name="${prefix}arm">
             <chain base_link="${prefix}base_link" tip_link="${prefix}flange" />
         </group>
-        <group_state name="${prefix}home" group="${prefix}${name}_arm">
-            <joint name="${prefix}joint1" value="0"/>
-            <joint name="${prefix}joint2" value="${-2*pi/9}"/>
-            <joint name="${prefix}joint3" value="0"/>
-            <joint name="${prefix}joint4" value="${pi/2}"/>
-            <joint name="${prefix}joint5" value="0"/>
-            <joint name="${prefix}joint6" value="${2*pi/9}"/>
-            <joint name="${prefix}joint7" value="0"/>
+        <group_state name="${prefix}home" group="${prefix}arm">
+            <joint name="${prefix}joint1" value="0" />
+            <joint name="${prefix}joint2" value="${-2*pi/9}" />
+            <joint name="${prefix}joint3" value="0" />
+            <joint name="${prefix}joint4" value="${pi/2}" />
+            <joint name="${prefix}joint5" value="0" />
+            <joint name="${prefix}joint6" value="${2*pi/9}" />
+            <joint name="${prefix}joint7" value="0" />
         </group_state>
-        <virtual_joint name="virtual_joint" type="fixed" parent_frame="world" child_link="${prefix}base_link"/>
-        <disable_collisions link1="${prefix}base_link" link2="${prefix}link1" reason="Adjacent"/>
-        <disable_collisions link1="${prefix}base_link" link2="${prefix}link2" reason="Never"/>
-        <disable_collisions link1="${prefix}base_link" link2="${prefix}link3" reason="Never"/>
-        <disable_collisions link1="${prefix}base_link" link2="${prefix}link4" reason="Never"/>
-        <disable_collisions link1="${prefix}link1" link2="${prefix}link2" reason="Adjacent"/>
-        <disable_collisions link1="${prefix}link1" link2="${prefix}link3" reason="Never"/>
-        <disable_collisions link1="${prefix}link1" link2="${prefix}link4" reason="Never"/>
-        <disable_collisions link1="${prefix}link2" link2="${prefix}link3" reason="Adjacent"/>
-        <disable_collisions link1="${prefix}link2" link2="${prefix}link4" reason="Never"/>
-        <disable_collisions link1="${prefix}link2" link2="${prefix}link5" reason="Never"/>
-        <disable_collisions link1="${prefix}link3" link2="${prefix}link4" reason="Adjacent"/>
-        <disable_collisions link1="${prefix}link3" link2="${prefix}link5" reason="Never"/>
-        <disable_collisions link1="${prefix}link3" link2="${prefix}link6" reason="Never"/>
-        <disable_collisions link1="${prefix}link3" link2="${prefix}link7" reason="Never"/>
-        <disable_collisions link1="${prefix}link4" link2="${prefix}link5" reason="Adjacent"/>
-        <disable_collisions link1="${prefix}link4" link2="${prefix}link6" reason="Never"/>
-        <disable_collisions link1="${prefix}link4" link2="${prefix}link7" reason="Never"/>
-        <disable_collisions link1="${prefix}link5" link2="${prefix}link6" reason="Adjacent"/>
-        <disable_collisions link1="${prefix}link6" link2="${prefix}link7" reason="Adjacent"/>
-        <disable_collisions link1="${prefix}link7" link2="${prefix}flange" reason="Adjacent"/>
+        <virtual_joint name="virtual_joint" type="fixed" parent_frame="world"
+            child_link="${prefix}base_link" />
+        <disable_collisions link1="${prefix}base_link" link2="${prefix}link1" reason="Adjacent" />
+        <disable_collisions link1="${prefix}base_link" link2="${prefix}link2" reason="Never" />
+        <disable_collisions link1="${prefix}base_link" link2="${prefix}link3" reason="Never" />
+        <disable_collisions link1="${prefix}base_link" link2="${prefix}link4" reason="Never" />
+        <disable_collisions link1="${prefix}link1" link2="${prefix}link2" reason="Adjacent" />
+        <disable_collisions link1="${prefix}link1" link2="${prefix}link3" reason="Never" />
+        <disable_collisions link1="${prefix}link1" link2="${prefix}link4" reason="Never" />
+        <disable_collisions link1="${prefix}link2" link2="${prefix}link3" reason="Adjacent" />
+        <disable_collisions link1="${prefix}link2" link2="${prefix}link4" reason="Never" />
+        <disable_collisions link1="${prefix}link2" link2="${prefix}link5" reason="Never" />
+        <disable_collisions link1="${prefix}link3" link2="${prefix}link4" reason="Adjacent" />
+        <disable_collisions link1="${prefix}link3" link2="${prefix}link5" reason="Never" />
+        <disable_collisions link1="${prefix}link3" link2="${prefix}link6" reason="Never" />
+        <disable_collisions link1="${prefix}link3" link2="${prefix}link7" reason="Never" />
+        <disable_collisions link1="${prefix}link4" link2="${prefix}link5" reason="Adjacent" />
+        <disable_collisions link1="${prefix}link4" link2="${prefix}link6" reason="Never" />
+        <disable_collisions link1="${prefix}link4" link2="${prefix}link7" reason="Never" />
+        <disable_collisions link1="${prefix}link5" link2="${prefix}link6" reason="Adjacent" />
+        <disable_collisions link1="${prefix}link6" link2="${prefix}link7" reason="Adjacent" />
+        <disable_collisions link1="${prefix}link7" link2="${prefix}flange" reason="Adjacent" />
     </xacro:macro>
 </robot>

Commit message: Add support for mounted force torque sensor in Rizon launch files

File: flexiv_moveit_config/srdf/grav.srdf.xacro (robot description, xacro)
@@ -1,5 +1,5 @@
 <?xml version="1.0" encoding="UTF-8"?>
 <robot xmlns:xacro="http://www.ros.org/wiki/xacro">
-    <xacro:macro name="grav_srdf" params="arm_prefix robot_sn">
+    <xacro:macro name="grav_srdf" params="arm_prefix robot_sn load_mounted_ft_sensor">
         <!-- Prefix defaults to 'arm_prefix_robot_sn' -->
         <xacro:property name="prefix" value="${arm_prefix + robot_sn + '_'}" />
@@ -35,31 +35,76 @@
             group="grav_gripper" parent_group="rizon_arm" />
         <disable_collisions link1="${prefix}grav_base_link" link2="${prefix}grav_tcp" reason="Never" />
-        <disable_collisions link1="${prefix}grav_base_link" link2="${prefix}closed_fingers_tcp" reason="Never" />
-        <disable_collisions link1="${prefix}grav_base_link" link2="${prefix}right_finger_tcp" reason="Never" />
-        <disable_collisions link1="${prefix}grav_base_link" link2="${prefix}left_finger_tcp" reason="Never" />
-        <disable_collisions link1="${prefix}grav_base_link" link2="${prefix}left_outer_bar" reason="Adjacent" />
-        <disable_collisions link1="${prefix}grav_base_link" link2="${prefix}left_inner_bar" reason="Adjacent" />
-        <disable_collisions link1="${prefix}grav_base_link" link2="${prefix}right_outer_bar" reason="Adjacent" />
-        <disable_collisions link1="${prefix}grav_base_link" link2="${prefix}right_inner_bar" reason="Adjacent" />
-        <disable_collisions link1="${prefix}grav_base_link" link2="${prefix}left_finger_mount" reason="Never" />
-        <disable_collisions link1="${prefix}grav_base_link" link2="${prefix}left_finger_tip" reason="Never" />
-        <disable_collisions link1="${prefix}grav_base_link" link2="${prefix}right_finger_mount" reason="Never" />
-        <disable_collisions link1="${prefix}grav_base_link" link2="${prefix}right_finger_tip" reason="Never" />
-        <disable_collisions link1="${prefix}left_outer_bar" link2="${prefix}left_finger_mount" reason="Adjacent" />
-        <disable_collisions link1="${prefix}left_inner_bar" link2="${prefix}left_finger_mount" reason="Adjacent" />
-        <disable_collisions link1="${prefix}left_outer_bar" link2="${prefix}left_finger_tip" reason="Never" />
-        <disable_collisions link1="${prefix}left_inner_bar" link2="${prefix}left_finger_tip" reason="Never" />
-        <disable_collisions link1="${prefix}left_finger_mount" link2="${prefix}left_finger_tip" reason="Adjacent" />
-        <disable_collisions link1="${prefix}right_outer_bar" link2="${prefix}right_finger_mount" reason="Adjacent" />
-        <disable_collisions link1="${prefix}right_inner_bar" link2="${prefix}right_finger_mount" reason="Adjacent" />
-        <disable_collisions link1="${prefix}right_outer_bar" link2="${prefix}right_finger_tip" reason="Never" />
-        <disable_collisions link1="${prefix}right_inner_bar" link2="${prefix}right_finger_tip" reason="Never" />
-        <disable_collisions link1="${prefix}right_finger_mount" link2="${prefix}right_finger_tip" reason="Adjacent" />
-        <disable_collisions link1="${prefix}left_finger_tip" link2="${prefix}closed_fingers_tcp" reason="Adjacent" />
-        <disable_collisions link1="${prefix}right_finger_tip" link2="${prefix}closed_fingers_tcp" reason="Adjacent" />
+        <disable_collisions link1="${prefix}grav_base_link" link2="${prefix}closed_fingers_tcp"
+            reason="Never" />
+        <disable_collisions link1="${prefix}grav_base_link" link2="${prefix}right_finger_tcp"
+            reason="Never" />
+        <disable_collisions link1="${prefix}grav_base_link" link2="${prefix}left_finger_tcp"
+            reason="Never" />
+        <disable_collisions link1="${prefix}grav_base_link" link2="${prefix}left_outer_bar"
+            reason="Adjacent" />
+        <disable_collisions link1="${prefix}grav_base_link" link2="${prefix}left_inner_bar"
+            reason="Adjacent" />
+        <disable_collisions link1="${prefix}grav_base_link" link2="${prefix}right_outer_bar"
+            reason="Adjacent" />
+        <disable_collisions link1="${prefix}grav_base_link" link2="${prefix}right_inner_bar"
+            reason="Adjacent" />
+        <disable_collisions link1="${prefix}grav_base_link" link2="${prefix}left_finger_mount"
+            reason="Never" />
+        <disable_collisions link1="${prefix}grav_base_link" link2="${prefix}left_finger_tip"
+            reason="Never" />
+        <disable_collisions link1="${prefix}grav_base_link" link2="${prefix}right_finger_mount"
+            reason="Never" />
+        <disable_collisions link1="${prefix}grav_base_link" link2="${prefix}right_finger_tip"
+            reason="Never" />
+        <disable_collisions link1="${prefix}left_outer_bar" link2="${prefix}left_finger_mount"
+            reason="Adjacent" />
+        <disable_collisions link1="${prefix}left_inner_bar" link2="${prefix}left_finger_mount"
+            reason="Adjacent" />
+        <disable_collisions link1="${prefix}left_outer_bar" link2="${prefix}left_finger_tip"
+            reason="Never" />
+        <disable_collisions link1="${prefix}left_inner_bar" link2="${prefix}left_finger_tip"
+            reason="Never" />
+        <disable_collisions link1="${prefix}left_finger_mount" link2="${prefix}left_finger_tip"
+            reason="Adjacent" />
+        <disable_collisions link1="${prefix}right_outer_bar" link2="${prefix}right_finger_mount"
+            reason="Adjacent" />
+        <disable_collisions link1="${prefix}right_inner_bar" link2="${prefix}right_finger_mount"
+            reason="Adjacent" />
+        <disable_collisions link1="${prefix}right_outer_bar" link2="${prefix}right_finger_tip"
+            reason="Never" />
+        <disable_collisions link1="${prefix}right_inner_bar" link2="${prefix}right_finger_tip"
+            reason="Never" />
+        <disable_collisions link1="${prefix}right_finger_mount" link2="${prefix}right_finger_tip"
+            reason="Adjacent" />
+        <disable_collisions link1="${prefix}left_finger_tip" link2="${prefix}closed_fingers_tcp"
+            reason="Adjacent" />
+        <disable_collisions link1="${prefix}right_finger_tip" link2="${prefix}closed_fingers_tcp"
+            reason="Adjacent" />
         <disable_collisions link1="${prefix}grav_base_link" link2="${prefix}link7" reason="Adjacent" />
-        <disable_collisions link1="${prefix}grav_base_link" link2="${prefix}flange" reason="Adjacent" />
-        <disable_collisions link1="${prefix}closed_fingers_tcp" link2="${prefix}link7" reason="Adjacent" />
-        <disable_collisions link1="${prefix}closed_fingers_tcp" link2="${prefix}flange" reason="Adjacent" />
+        <disable_collisions link1="${prefix}grav_base_link" link2="${prefix}flange"
+            reason="Adjacent" />
+        <disable_collisions link1="${prefix}closed_fingers_tcp" link2="${prefix}link7"
+            reason="Adjacent" />
+        <disable_collisions link1="${prefix}closed_fingers_tcp" link2="${prefix}flange"
+            reason="Adjacent" />
+        <xacro:if value="${load_mounted_ft_sensor}">
+            <disable_collisions link1="${prefix}grav_base_link"
+                link2="${prefix}wrist-sensor.base_link"
+                reason="Adjacent" />
+            <disable_collisions link1="${prefix}grav_base_link"
+                link2="${prefix}wrist-sensor.proximal_link" reason="Adjacent" />
+            <disable_collisions link1="${prefix}grav_base_link"
+                link2="${prefix}wrist-sensor.distal_link" reason="Adjacent" />
+            <disable_collisions link1="${prefix}closed_fingers_tcp" link2="${prefix}link7"
+                reason="Adjacent" />
+            <disable_collisions link1="${prefix}closed_fingers_tcp" link2="${prefix}flange"
+                reason="Adjacent" />
+            <disable_collisions link1="${prefix}closed_fingers_tcp"
+                link2="${prefix}wrist-sensor.base_link" reason="Adjacent" />
+            <disable_collisions link1="${prefix}closed_fingers_tcp"
+                link2="${prefix}wrist-sensor.proximal_link" reason="Adjacent" />
+            <disable_collisions link1="${prefix}closed_fingers_tcp"
+                link2="${prefix}wrist-sensor.distal_link" reason="Adjacent" />
+        </xacro:if>
     </xacro:macro>
 </robot>

File: flexiv_moveit_config/srdf/rizon.srdf.xacro (robot description, xacro)
@@ -5,10 +5,13 @@
     <xacro:arg name="robot_sn" default="" />
     <xacro:arg name="load_gripper" default="false" />
+    <xacro:arg name="load_mounted_ft_sensor" default="false" />
     <xacro:include filename="$(find flexiv_moveit_config)/srdf/rizon_macro.srdf.xacro" />
-    <xacro:rizon_srdf arm_prefix="$(arg arm_prefix)" robot_sn="$(arg robot_sn)" />
+    <xacro:rizon_srdf arm_prefix="$(arg arm_prefix)" robot_sn="$(arg robot_sn)"
+        load_mounted_ft_sensor="$(arg load_mounted_ft_sensor)" />
     <!-- Load gripper -->
     <xacro:if value="$(arg load_gripper)">
         <xacro:include filename="$(find flexiv_moveit_config)/srdf/grav.srdf.xacro" />
-        <xacro:grav_srdf arm_prefix="$(arg arm_prefix)" robot_sn="$(arg robot_sn)" />
+        <xacro:grav_srdf arm_prefix="$(arg arm_prefix)" robot_sn="$(arg robot_sn)"
+            load_mounted_ft_sensor="$(arg load_mounted_ft_sensor)" />
     </xacro:if>
 </robot>

File: flexiv_moveit_config/srdf/rizon_macro.srdf.xacro (robot description, xacro)
@@ -1,5 +1,5 @@
 <?xml version="1.0" encoding="UTF-8"?>
 <robot xmlns:xacro="http://www.ros.org/wiki/xacro">
-    <xacro:macro name="rizon_srdf" params="arm_prefix robot_sn">
+    <xacro:macro name="rizon_srdf" params="arm_prefix robot_sn load_mounted_ft_sensor">
         <!-- Prefix defaults to 'arm_prefix_robot_sn' -->
         <xacro:property name="prefix" value="${arm_prefix + robot_sn + '_'}" />
@@ -38,4 +38,19 @@
         <disable_collisions link1="${prefix}link6" link2="${prefix}link7" reason="Adjacent" />
         <disable_collisions link1="${prefix}link7" link2="${prefix}flange" reason="Adjacent" />
+        <xacro:if value="${load_mounted_ft_sensor}">
+            <!-- Disable collisions for FT sensor fixed-link chain -->
+            <disable_collisions link1="${prefix}link7" link2="${prefix}wrist-sensor.base_link"
+                reason="Adjacent" />
+            <disable_collisions link1="${prefix}wrist-sensor.base_link"
+                link2="${prefix}wrist-sensor.proximal_link" reason="Adjacent" />
+            <disable_collisions link1="${prefix}wrist-sensor.proximal_link"
+                link2="${prefix}wrist-sensor.distal_link" reason="Adjacent" />
+            <disable_collisions link1="${prefix}wrist-sensor.distal_link" link2="${prefix}flange"
+                reason="Adjacent" />
+            <disable_collisions link1="${prefix}link7" link2="${prefix}wrist-sensor.proximal_link"
+                reason="Adjacent" />
+            <disable_collisions link1="${prefix}link7" link2="${prefix}wrist-sensor.distal_link"
+                reason="Adjacent" />
+        </xacro:if>
     </xacro:macro>
 </robot>
