Commit message: Refactor robot serial number parameters to unify naming across configurations

File: flexiv_moveit_config/srdf/aico2.srdf.xacro (robot description, xacro)
@@ -4,6 +4,5 @@
     <xacro:arg name="external_axis_type" default="aico2_4_v1" />
     <xacro:arg name="external_axis_prefix" default="" />
-    <xacro:arg name="robot_sn_left" default="" />
-    <xacro:arg name="robot_sn_right" default="" />
+    <xacro:arg name="robot_sn" default="" />
     <xacro:arg name="load_gripper_left" default="false" />
     <xacro:arg name="load_gripper_right" default="false" />
@@ -14,12 +13,12 @@
     <xacro:include filename="$(find flexiv_moveit_config)/srdf/rizon_macro.srdf.xacro" />
     <!-- Left Arm -->
-    <xacro:rizon_srdf arm_prefix="$(arg arm_prefix_left)" robot_sn="$(arg robot_sn_left)"
+    <xacro:rizon_srdf arm_prefix="$(arg arm_prefix_left)" robot_sn="$(arg robot_sn)"
         load_mounted_ft_sensor="$(arg load_mounted_ft_sensor_left)" use_virtual_joint="false" />
     <!-- Right Arm -->
-    <xacro:rizon_srdf arm_prefix="$(arg arm_prefix_right)" robot_sn="$(arg robot_sn_right)"
+    <xacro:rizon_srdf arm_prefix="$(arg arm_prefix_right)" robot_sn="$(arg robot_sn)"
         load_mounted_ft_sensor="$(arg load_mounted_ft_sensor_right)" use_virtual_joint="false" />
     <!-- Prefixes -->
-    <xacro:property name="prefix_left" value="$(arg arm_prefix_left)$(arg robot_sn_left)_" />
-    <xacro:property name="prefix_right" value="$(arg arm_prefix_right)$(arg robot_sn_right)_" />
+    <xacro:property name="prefix_left" value="$(arg arm_prefix_left)$(arg robot_sn)_" />
+    <xacro:property name="prefix_right" value="$(arg arm_prefix_right)$(arg robot_sn)_" />
     <xacro:property name="external_axis_prefix" value="$(arg external_axis_prefix)" />
     <!-- Virtual Joint and External Axis Group -->
@@ -118,10 +117,10 @@
     <xacro:if value="$(arg load_gripper_left)">
         <xacro:include filename="$(find flexiv_moveit_config)/srdf/grav.srdf.xacro" />
-        <xacro:grav_srdf arm_prefix="$(arg prefix_left)" robot_sn="$(arg robot_sn_left)"
+        <xacro:grav_srdf arm_prefix="$(arg arm_prefix_left)" robot_sn="$(arg robot_sn)"
             load_mounted_ft_sensor="$(arg load_mounted_ft_sensor_left)" />
     </xacro:if>
     <xacro:if value="$(arg load_gripper_right)">
         <xacro:include filename="$(find flexiv_moveit_config)/srdf/grav.srdf.xacro" />
-        <xacro:grav_srdf arm_prefix="$(arg prefix_right)" robot_sn="$(arg robot_sn_right)"
+        <xacro:grav_srdf arm_prefix="$(arg arm_prefix_right)" robot_sn="$(arg robot_sn)"
             load_mounted_ft_sensor="$(arg load_mounted_ft_sensor_right)" />
     </xacro:if>

File: flexiv_moveit_config/srdf/rizon_dual.srdf.xacro (robot description, xacro)
@@ -2,6 +2,5 @@
 <robot xmlns:xacro="http://wiki.ros.org/xacro" name="rizon_dual">
     <!-- parameters -->
-    <xacro:arg name="robot_sn_left" default="" />
-    <xacro:arg name="robot_sn_right" default="" />
+    <xacro:arg name="robot_sn" default="" />
     <xacro:arg name="load_gripper_left" default="false" />
     <xacro:arg name="load_gripper_right" default="false" />
@@ -12,12 +11,12 @@
     <xacro:include filename="$(find flexiv_moveit_config)/srdf/rizon_macro.srdf.xacro" />
     <!-- Left Arm -->
-    <xacro:rizon_srdf arm_prefix="$(arg prefix_left)" robot_sn="$(arg robot_sn_left)"
+    <xacro:rizon_srdf arm_prefix="$(arg prefix_left)" robot_sn="$(arg robot_sn)"
         load_mounted_ft_sensor="$(arg load_mounted_ft_sensor_left)" />
     <!-- Right Arm -->
-    <xacro:rizon_srdf arm_prefix="$(arg prefix_right)" robot_sn="$(arg robot_sn_right)"
+    <xacro:rizon_srdf arm_prefix="$(arg prefix_right)" robot_sn="$(arg robot_sn)"
         load_mounted_ft_sensor="$(arg load_mounted_ft_sensor_right)" />
     <!-- Arm Prefixes -->
-    <xacro:property name="left_arm_prefix" value="$(arg prefix_left)$(arg robot_sn_left)_" />
-    <xacro:property name="right_arm_prefix" value="$(arg prefix_right)$(arg robot_sn_right)_" />
+    <xacro:property name="left_arm_prefix" value="$(arg prefix_left)$(arg robot_sn)_" />
+    <xacro:property name="right_arm_prefix" value="$(arg prefix_right)$(arg robot_sn)_" />
     <!-- Left and Right Arms Collisions -->
     <disable_collisions link1="${left_arm_prefix}base_link" link2="${right_arm_prefix}base_link" reason="Never" />
@@ -26,10 +25,10 @@
     <xacro:if value="$(arg load_gripper_left)">
         <xacro:include filename="$(find flexiv_moveit_config)/srdf/grav.srdf.xacro" />
-        <xacro:grav_srdf arm_prefix="$(arg prefix_left)" robot_sn="$(arg robot_sn_left)"
+        <xacro:grav_srdf arm_prefix="$(arg prefix_left)" robot_sn="$(arg robot_sn)"
             load_mounted_ft_sensor="$(arg load_mounted_ft_sensor_left)" />
     </xacro:if>
     <xacro:if value="$(arg load_gripper_right)">
         <xacro:include filename="$(find flexiv_moveit_config)/srdf/grav.srdf.xacro" />
-        <xacro:grav_srdf arm_prefix="$(arg prefix_right)" robot_sn="$(arg robot_sn_right)"
+        <xacro:grav_srdf arm_prefix="$(arg prefix_right)" robot_sn="$(arg robot_sn)"
             load_mounted_ft_sensor="$(arg load_mounted_ft_sensor_right)" />
     </xacro:if>
