Commit message: Update Flexiv MoveIt config

File: flexiv_moveit_config/srdf/flexiv_macro.srdf.xacro (robot description, xacro)
@@ -1,5 +1,5 @@
 <?xml version="1.0" encoding="UTF-8"?>
 <robot xmlns:xacro="http://www.ros.org/wiki/xacro">
-    <xacro:macro name="rizon_srdf" params="arm_prefix robot_sn load_mounted_ft_sensor use_virtual_joint:=true">
+    <xacro:macro name="flexiv_srdf" params="arm_prefix robot_sn load_mounted_ft_sensor use_virtual_joint:=true">
         <!-- Prefix defaults to 'arm_prefix_robot_sn' -->
         <xacro:property name="prefix" value="${arm_prefix + robot_sn + '_'}" />
@@ -42,10 +42,16 @@
         <xacro:if value="${load_mounted_ft_sensor}">
             <!-- Disable collisions for FT sensor fixed-link chain -->
-            <disable_collisions link1="${prefix}link7" link2="${prefix}wrist-sensor.base_link" reason="Adjacent" />
-            <disable_collisions link1="${prefix}wrist-sensor.base_link" link2="${prefix}wrist-sensor.proximal_link" reason="Adjacent" />
-            <disable_collisions link1="${prefix}wrist-sensor.proximal_link" link2="${prefix}wrist-sensor.distal_link" reason="Adjacent" />
-            <disable_collisions link1="${prefix}wrist-sensor.distal_link" link2="${prefix}flange" reason="Adjacent" />
-            <disable_collisions link1="${prefix}link7" link2="${prefix}wrist-sensor.proximal_link" reason="Adjacent" />
-            <disable_collisions link1="${prefix}link7" link2="${prefix}wrist-sensor.distal_link" reason="Adjacent" />
+            <disable_collisions link1="${prefix}link7" link2="${prefix}wrist-sensor.base_link"
+                reason="Adjacent" />
+            <disable_collisions link1="${prefix}wrist-sensor.base_link"
+                link2="${prefix}wrist-sensor.proximal_link" reason="Adjacent" />
+            <disable_collisions link1="${prefix}wrist-sensor.proximal_link"
+                link2="${prefix}wrist-sensor.distal_link" reason="Adjacent" />
+            <disable_collisions link1="${prefix}wrist-sensor.distal_link" link2="${prefix}flange"
+                reason="Adjacent" />
+            <disable_collisions link1="${prefix}link7" link2="${prefix}wrist-sensor.proximal_link"
+                reason="Adjacent" />
+            <disable_collisions link1="${prefix}link7" link2="${prefix}wrist-sensor.distal_link"
+                reason="Adjacent" />
         </xacro:if>
     </xacro:macro>

Commit message: Update Enlight joint config for Home position

File: flexiv_moveit_config/srdf/flexiv_macro.srdf.xacro (robot description, xacro)
@@ -13,5 +13,5 @@
             <joint name="${prefix}joint4" value="${pi/2}" />
             <joint name="${prefix}joint5" value="0" />
-            <joint name="${prefix}joint6" value="${2*pi/9}" />
+            <joint name="${prefix}joint6" value="${-5*pi/18}" />
             <joint name="${prefix}joint7" value="0" />
         </group_state>
