Commit message: Consolidate MoveIt configs and fix MoveIt Servo for Jazzy

File: flexiv_moveit_config/srdf/flexiv.srdf.xacro (robot description, xacro)
@@ -26,11 +26,9 @@
              The macro computes prefix = arm_prefix + robot_sn + '_', so
              arm_prefix="left_" yields prefix "left_<sn>_" as required.
-             Virtual joints are disabled because both arms parent to 'world' via the URDF. -->
+             No virtual joint is declared: the URDF already roots every arm at 'world'. -->
         <xacro:flexiv_srdf arm_prefix="left_" robot_sn="$(arg robot_sn)"
-            load_mounted_ft_sensor="$(arg load_mounted_ft_sensor)"
-            use_virtual_joint="false" />
+            load_mounted_ft_sensor="$(arg load_mounted_ft_sensor)" />
         <xacro:flexiv_srdf arm_prefix="right_" robot_sn="$(arg robot_sn)"
-            load_mounted_ft_sensor="$(arg load_mounted_ft_sensor)"
-            use_virtual_joint="false" />
+            load_mounted_ft_sensor="$(arg load_mounted_ft_sensor)" />
         <!-- Combined group that references both arm sub-groups -->
         <xacro:property name="left_prefix" value="${'left_' + '$(arg robot_sn)' + '_'}" />

File: flexiv_moveit_config/srdf/flexiv_macro.srdf.xacro (robot description, xacro)
@@ -1,5 +1,5 @@
 <?xml version="1.0" encoding="UTF-8"?>
 <robot xmlns:xacro="http://www.ros.org/wiki/xacro">
-    <xacro:macro name="flexiv_srdf" params="arm_prefix robot_sn load_mounted_ft_sensor use_virtual_joint:=true">
+    <xacro:macro name="flexiv_srdf" params="arm_prefix robot_sn load_mounted_ft_sensor">
         <!-- Prefix defaults to 'arm_prefix_robot_sn' -->
         <xacro:property name="prefix" value="${arm_prefix + robot_sn + '_'}" />
@@ -16,8 +16,4 @@
             <joint name="${prefix}joint7" value="0" />
         </group_state>
-        <xacro:if value="${use_virtual_joint}">
-            <virtual_joint name="virtual_joint" type="fixed" parent_frame="world"
-                child_link="${prefix}base_link" />
-        </xacro:if>
         <disable_collisions link1="${prefix}base_link" link2="${prefix}link1" reason="Adjacent" />
         <disable_collisions link1="${prefix}base_link" link2="${prefix}link2" reason="Never" />

Commit message: Disable collision checks between the MICO neck, head and their rigidly attached links in the SRDF

File: flexiv_moveit_config/srdf/flexiv.srdf.xacro (robot description, xacro)
@@ -56,4 +56,19 @@
         value="${'$(arg robot_type)' in ['MICO-Plus', 'MICO-Ultra']}" />
     <xacro:property name="torso_prefix" value="${'$(arg robot_sn)' + '_torso_'}" />
+    <!-- The neck and head (flexiv_description jazzy-v3.1) are fixed to the torso link the arms
+         mount on, so their poses relative to that link and to both arm bases never change. Their
+         collision checks are disabled against all of these; the arm links keep theirs. -->
+    <xacro:macro name="mico_neck_head_collisions" params="mount">
+        <disable_collisions link1="${mount}" link2="${torso_prefix}neck_link" reason="Adjacent" />
+        <disable_collisions link1="${torso_prefix}neck_link" link2="${torso_prefix}head_link"
+            reason="Adjacent" />
+        <disable_collisions link1="${mount}" link2="${torso_prefix}head_link" reason="Never" />
+        <xacro:macro name="mico_rigid_to_arm_bases" params="link">
+            <disable_collisions link1="${link}" link2="${left_prefix}base_link" reason="Never" />
+            <disable_collisions link1="${link}" link2="${right_prefix}base_link" reason="Never" />
+        </xacro:macro>
+        <xacro:mico_rigid_to_arm_bases link="${torso_prefix}neck_link" />
+        <xacro:mico_rigid_to_arm_bases link="${torso_prefix}head_link" />
+    </xacro:macro>
     <!-- MICO-Core: fixed torso; both arm bases mount directly on the torso base_link. -->
     <xacro:if value="${is_mico_core}">
@@ -64,4 +79,5 @@
         <disable_collisions link1="${left_prefix}base_link" link2="${right_prefix}base_link"
             reason="Never" />
+        <xacro:mico_neck_head_collisions mount="${torso_prefix}base_link" />
     </xacro:if>
     <!-- MICO-Plus / MICO-Ultra: 2-DoF torso (base_link -> link1 -> link2); arms mount on link2. -->
@@ -93,4 +109,5 @@
         <disable_collisions link1="${left_prefix}base_link" link2="${right_prefix}base_link"
             reason="Never" />
+        <xacro:mico_neck_head_collisions mount="${torso_prefix}link2" />
     </xacro:if>
 </robot>

Commit message: Load the MoveIt SRDF home poses from the flexiv_description initial positions

File: flexiv_moveit_config/srdf/flexiv.srdf.xacro (robot description, xacro)
@@ -29,6 +29,9 @@
         <xacro:flexiv_srdf arm_prefix="left_" robot_sn="$(arg robot_sn)"
             load_mounted_ft_sensor="$(arg load_mounted_ft_sensor)" />
+        <!-- The MICO arms face each other, so the right arm starts mirrored, as in the URDF -->
+        <xacro:property name="init_dir" value="$(find flexiv_description)/config/Enlight-L" />
         <xacro:flexiv_srdf arm_prefix="right_" robot_sn="$(arg robot_sn)"
-            load_mounted_ft_sensor="$(arg load_mounted_ft_sensor)" />
+            load_mounted_ft_sensor="$(arg load_mounted_ft_sensor)"
+            initial_positions_file="${init_dir + ('/initial_positions.yaml' if '$(arg robot_type)' == 'Enlight-LL' else '/initial_positions_mirrored.yaml')}" />
         <!-- Combined group that references both arm sub-groups -->
         <xacro:property name="left_prefix" value="${'left_' + '$(arg robot_sn)' + '_'}" />

File: flexiv_moveit_config/srdf/flexiv_macro.srdf.xacro (robot description, xacro)
@@ -1,18 +1,22 @@
 <?xml version="1.0" encoding="UTF-8"?>
 <robot xmlns:xacro="http://www.ros.org/wiki/xacro">
-    <xacro:macro name="flexiv_srdf" params="arm_prefix robot_sn load_mounted_ft_sensor">
+    <xacro:macro name="flexiv_srdf"
+        params="arm_prefix robot_sn load_mounted_ft_sensor
+                initial_positions_file:='$(find flexiv_description)/config/Enlight-L/initial_positions.yaml'">
         <!-- Prefix defaults to 'arm_prefix_robot_sn' -->
         <xacro:property name="prefix" value="${arm_prefix + robot_sn + '_'}" />
+        <!-- Home is the arm's initial pose in flexiv_description, the same one the URDF starts from -->
+        <xacro:property name="home" value="${xacro.load_yaml(initial_positions_file)['initial_positions']}" />
         <group name="${prefix}arm">
             <chain base_link="${prefix}base_link" tip_link="${prefix}flange" />
         </group>
         <group_state name="${prefix}home" group="${prefix}arm">
-            <joint name="${prefix}joint1" value="0" />
-            <joint name="${prefix}joint2" value="${-2*pi/9}" />
-            <joint name="${prefix}joint3" value="0" />
-            <joint name="${prefix}joint4" value="${pi/2}" />
-            <joint name="${prefix}joint5" value="0" />
-            <joint name="${prefix}joint6" value="${2*pi/9}" />
-            <joint name="${prefix}joint7" value="0" />
+            <joint name="${prefix}joint1" value="${home['joint1']}" />
+            <joint name="${prefix}joint2" value="${home['joint2']}" />
+            <joint name="${prefix}joint3" value="${home['joint3']}" />
+            <joint name="${prefix}joint4" value="${home['joint4']}" />
+            <joint name="${prefix}joint5" value="${home['joint5']}" />
+            <joint name="${prefix}joint6" value="${home['joint6']}" />
+            <joint name="${prefix}joint7" value="${home['joint7']}" />
         </group_state>
         <disable_collisions link1="${prefix}base_link" link2="${prefix}link1" reason="Adjacent" />
