Commit message: Support the six new AICO2 platform types

File: flexiv_hardware/ros2_control/rizon_dual.ros2_control.xacro (robot description, xacro)
@@ -65,7 +65,8 @@
       <xacro:configure_joint joint_name="${prefix_left}joint6" initial_pos="${initial_positions_left['joint6']}" />
       <xacro:configure_joint joint_name="${prefix_left}joint7" initial_pos="${initial_positions_left['joint7']}" />
-      <!-- External axis joints -->
-      <xacro:if value="${external_axis_type == 'aico2_4_v1'}">
-        <joint name="${external_axis_prefix}aico2_4_v1_joint1">
+      <!-- External axis joints. Every AICO2 axis exposes joint1 and joint2, named
+           after the robot type lowercased with dashes as underscores. -->
+      <xacro:if value="${external_axis_type.startswith('aico2')}">
+        <joint name="${external_axis_prefix}${external_axis_type}_joint1">
           <command_interface name="position" />
           <command_interface name="velocity" />
@@ -77,49 +78,5 @@
           <state_interface name="effort" />
         </joint>
-        <joint name="${external_axis_prefix}aico2_4_v1_joint2">
-          <command_interface name="position" />
-          <command_interface name="velocity" />
-          <command_interface name="effort" />
-          <state_interface name="position">
-            <param name="initial_value">0.0</param>
-          </state_interface>
-          <state_interface name="velocity" />
-          <state_interface name="effort" />
-        </joint>
-      </xacro:if>
-      <xacro:if value="${external_axis_type == 'aico2_4_v2'}">
-        <joint name="${external_axis_prefix}aico2_4_v2_joint1">
-          <command_interface name="position" />
-          <command_interface name="velocity" />
-          <command_interface name="effort" />
-          <state_interface name="position">
-            <param name="initial_value">0.0</param>
-          </state_interface>
-          <state_interface name="velocity" />
-          <state_interface name="effort" />
-        </joint>
-        <joint name="${external_axis_prefix}aico2_4_v2_joint2">
-          <command_interface name="position" />
-          <command_interface name="velocity" />
-          <command_interface name="effort" />
-          <state_interface name="position">
-            <param name="initial_value">0.0</param>
-          </state_interface>
-          <state_interface name="velocity" />
-          <state_interface name="effort" />
-        </joint>
-      </xacro:if>
-      <xacro:if value="${external_axis_type == 'aico2_10_v1'}">
-        <joint name="${external_axis_prefix}aico2_10_v1_joint1">
-          <command_interface name="position" />
-          <command_interface name="velocity" />
-          <command_interface name="effort" />
-          <state_interface name="position">
-            <param name="initial_value">0.0</param>
-          </state_interface>
-          <state_interface name="velocity" />
-          <state_interface name="effort" />
-        </joint>
-        <joint name="${external_axis_prefix}aico2_10_v1_joint2">
+        <joint name="${external_axis_prefix}${external_axis_type}_joint2">
           <command_interface name="position" />
           <command_interface name="velocity" />

File: flexiv_hardware/urdf/flexiv.urdf.xacro (robot description, xacro)
@@ -27,8 +27,11 @@
     <xacro:property name="single_arms"
       value="${['Rizon4', 'Rizon4s', 'Rizon4M', 'Rizon4R', 'Rizon10', 'Rizon10s', 'Rizon10R']}" />
+    <xacro:property name="aico1_types" value="${['AICO1-4-V1', 'AICO1-4-V2']}" />
+    <xacro:property name="aico2_types"
+      value="${['AICO2-4-V1', 'AICO2-4-V2', 'AICO2-4-D3', 'AICO2-4E-D1', 'AICO2-4U-D1',
+                'AICO2-10-V1', 'AICO2-10-D2', 'AICO2-10E-D1', 'AICO2-10U-D1']}" />
     <xacro:property name="is_single" value="${rtype in single_arms}" />
-    <xacro:property name="is_aico1" value="${rtype in ['AICO1-4-V1', 'AICO1-4-V2']}" />
-    <xacro:property name="is_aico2"
-      value="${rtype in ['AICO2-4-V1', 'AICO2-4-V2', 'AICO2-10-V1']}" />
+    <xacro:property name="is_aico1" value="${rtype in aico1_types}" />
+    <xacro:property name="is_aico2" value="${rtype in aico2_types}" />
     <xacro:property name="is_rizon_dual" value="${rtype == 'Rizon-Dual'}" />
     <!-- Two robots with two serial numbers, as opposed to one robot with two arms. -->
@@ -36,5 +39,5 @@
     <xacro:unless value="${is_single or is_aico1 or is_paired}">
       ${xacro.error('robot_type ' + rtype + ' is not supported by this release. Supported: '
-        + ', '.join(single_arms + ['AICO1-4-V1', 'AICO1-4-V2', 'Rizon-Dual', 'AICO2-4-V1', 'AICO2-4-V2', 'AICO2-10-V1']))}
+        + ', '.join(single_arms + aico1_types + ['Rizon-Dual'] + aico2_types))}
     </xacro:unless>
     <!-- The hardware interface takes the external axis as a lowercase name. -->
@@ -45,6 +48,7 @@
     <xacro:property name="aico1_arm"
       value="${'$(arg arm_type)' if '$(arg arm_type)' != '' else 'Rizon4'}" />
-    <xacro:property name="paired_default_left" value="${'Rizon10' if rtype == 'AICO2-10-V1' else 'Rizon4'}" />
-    <xacro:property name="paired_default_right" value="${'Rizon10R' if rtype == 'AICO2-10-V1' else 'Rizon4R'}" />
+    <xacro:property name="is_aico2_10" value="${rtype.startswith('AICO2-10')}" />
+    <xacro:property name="paired_default_left" value="${'Rizon10' if is_aico2_10 else 'Rizon4'}" />
+    <xacro:property name="paired_default_right" value="${'Rizon10R' if is_aico2_10 else 'Rizon4R'}" />
     <xacro:property name="arm_left"
       value="${'$(arg arm_type_left)' if '$(arg arm_type_left)' != '' else paired_default_left}" />

File: flexiv_moveit_config/srdf/aico2.srdf.xacro (robot description, xacro)
@@ -29,96 +29,34 @@
     <xacro:rizon_srdf prefix="${prefix_right}"
         load_mounted_ft_sensor="$(arg load_mounted_ft_sensor_right)" use_virtual_joint="false" />
-    <!-- Virtual Joint and External Axis Group -->
-    <xacro:if value="${axis_name == 'aico2_4_v1'}">
-        <virtual_joint name="virtual_joint" type="fixed" parent_frame="world"
-            child_link="${external_axis_prefix}aico2_4_v1_base_link" />
-        <group name="${external_axis_prefix}aico2_4_v1_platform_${prefix_left}arm">
-            <chain base_link="${external_axis_prefix}aico2_4_v1_base_link" tip_link="${prefix_left}flange" />
-        </group>
-    </xacro:if>
-    <xacro:if value="${axis_name == 'aico2_4_v2'}">
-        <virtual_joint name="virtual_joint" type="fixed" parent_frame="world"
-            child_link="${external_axis_prefix}aico2_4_v2_base_link" />
-        <group name="${external_axis_prefix}aico2_4_v2_platform_${prefix_left}arm">
-            <chain base_link="${external_axis_prefix}aico2_4_v2_base_link" tip_link="${prefix_left}flange" />
-        </group>
-    </xacro:if>
-    <xacro:if value="${axis_name == 'aico2_10_v1'}">
-        <virtual_joint name="virtual_joint" type="fixed" parent_frame="world"
-            child_link="${external_axis_prefix}aico2_10_v1_base_link" />
-        <group name="${external_axis_prefix}aico2_10_v1_platform_${prefix_left}arm">
-            <chain base_link="${external_axis_prefix}aico2_10_v1_base_link" tip_link="${prefix_left}flange" />
-        </group>
-    </xacro:if>
+    <!-- Virtual Joint and External Axis Group. Every AICO2 axis has the same
+         base_link/link1/link2 topology, so one block covers all of them. -->
+    <xacro:property name="axis" value="${external_axis_prefix}${axis_name}" />
+    <virtual_joint name="virtual_joint" type="fixed" parent_frame="world"
+        child_link="${axis}_base_link" />
+    <group name="${axis}_platform_${prefix_left}arm">
+        <chain base_link="${axis}_base_link" tip_link="${prefix_left}flange" />
+    </group>
     <!-- External Axis Collisions -->
-    <xacro:if value="${axis_name == 'aico2_4_v1'}">
-        <!-- Left Arm -->
-        <disable_collisions link1="${prefix_left}base_link" link2="${external_axis_prefix}aico2_4_v1_link2" reason="Adjacent" />
-        <disable_collisions link1="${prefix_left}base_link" link2="${external_axis_prefix}aico2_4_v1_link1" reason="Never" />
-        <disable_collisions link1="${prefix_left}base_link" link2="${external_axis_prefix}aico2_4_v1_base_link" reason="Never" />
-        <disable_collisions link1="${prefix_left}link1" link2="${external_axis_prefix}aico2_4_v1_link2" reason="Never" />
-        <disable_collisions link1="${prefix_left}link1" link2="${external_axis_prefix}aico2_4_v1_link1" reason="Never" />
-        <disable_collisions link1="${prefix_left}link1" link2="${external_axis_prefix}aico2_4_v1_base_link" reason="Never" />
-        <!-- Right Arm -->
-        <disable_collisions link1="${prefix_right}base_link" link2="${external_axis_prefix}aico2_4_v1_link2" reason="Adjacent" />
-        <disable_collisions link1="${prefix_right}base_link" link2="${external_axis_prefix}aico2_4_v1_link1" reason="Never" />
-        <disable_collisions link1="${prefix_right}base_link" link2="${external_axis_prefix}aico2_4_v1_base_link" reason="Never" />
-        <disable_collisions link1="${prefix_right}link1" link2="${external_axis_prefix}aico2_4_v1_link2" reason="Never" />
-        <disable_collisions link1="${prefix_right}link1" link2="${external_axis_prefix}aico2_4_v1_link1" reason="Never" />
-        <disable_collisions link1="${prefix_right}link1" link2="${external_axis_prefix}aico2_4_v1_base_link" reason="Never" />
-        <!-- Left and Right Arms -->
-        <disable_collisions link1="${prefix_left}base_link" link2="${prefix_right}base_link" reason="Never" />
-        <disable_collisions link1="${prefix_left}link1" link2="${prefix_right}link1" reason="Never" />
-        <!-- External Axis internal -->
-        <disable_collisions link1="${external_axis_prefix}aico2_4_v1_base_link" link2="${external_axis_prefix}aico2_4_v1_link1" reason="Adjacent" />
-        <disable_collisions link1="${external_axis_prefix}aico2_4_v1_base_link" link2="${external_axis_prefix}aico2_4_v1_link2" reason="Never" />
-        <disable_collisions link1="${external_axis_prefix}aico2_4_v1_link1" link2="${external_axis_prefix}aico2_4_v1_link2" reason="Adjacent" />
-    </xacro:if>
-    <xacro:if value="${axis_name == 'aico2_4_v2'}">
-        <!-- Left Arm -->
-        <disable_collisions link1="${prefix_left}base_link" link2="${external_axis_prefix}aico2_4_v2_link2" reason="Adjacent" />
-        <disable_collisions link1="${prefix_left}base_link" link2="${external_axis_prefix}aico2_4_v2_link1" reason="Never" />
-        <disable_collisions link1="${prefix_left}base_link" link2="${external_axis_prefix}aico2_4_v2_base_link" reason="Never" />
-        <disable_collisions link1="${prefix_left}link1" link2="${external_axis_prefix}aico2_4_v2_link2" reason="Never" />
-        <disable_collisions link1="${prefix_left}link1" link2="${external_axis_prefix}aico2_4_v2_link1" reason="Never" />
-        <disable_collisions link1="${prefix_left}link1" link2="${external_axis_prefix}aico2_4_v2_base_link" reason="Never" />
-        <!-- Right Arm -->
-        <disable_collisions link1="${prefix_right}base_link" link2="${external_axis_prefix}aico2_4_v2_link2" reason="Adjacent" />
-        <disable_collisions link1="${prefix_right}base_link" link2="${external_axis_prefix}aico2_4_v2_link1" reason="Never" />
-        <disable_collisions link1="${prefix_right}base_link" link2="${external_axis_prefix}aico2_4_v2_base_link" reason="Never" />
-        <disable_collisions link1="${prefix_right}link1" link2="${external_axis_prefix}aico2_4_v2_link2" reason="Never" />
-        <disable_collisions link1="${prefix_right}link1" link2="${external_axis_prefix}aico2_4_v2_link1" reason="Never" />
-        <disable_collisions link1="${prefix_right}link1" link2="${external_axis_prefix}aico2_4_v2_base_link" reason="Never" />
-        <!-- Left and Right Arms -->
-        <disable_collisions link1="${prefix_left}base_link" link2="${prefix_right}base_link" reason="Never" />
-        <disable_collisions link1="${prefix_left}link1" link2="${prefix_right}link1" reason="Never" />
-        <!-- External Axis internal -->
-        <disable_collisions link1="${external_axis_prefix}aico2_4_v2_base_link" link2="${external_axis_prefix}aico2_4_v2_link1" reason="Adjacent" />
-        <disable_collisions link1="${external_axis_prefix}aico2_4_v2_base_link" link2="${external_axis_prefix}aico2_4_v2_link2" reason="Never" />
-        <disable_collisions link1="${external_axis_prefix}aico2_4_v2_link1" link2="${external_axis_prefix}aico2_4_v2_link2" reason="Adjacent" />
-    </xacro:if>
-    <xacro:if value="${axis_name == 'aico2_10_v1'}">
-        <!-- Left Arm -->
-        <disable_collisions link1="${prefix_left}base_link" link2="${external_axis_prefix}aico2_10_v1_link2" reason="Adjacent" />
-        <disable_collisions link1="${prefix_left}base_link" link2="${external_axis_prefix}aico2_10_v1_link1" reason="Never" />
-        <disable_collisions link1="${prefix_left}base_link" link2="${external_axis_prefix}aico2_10_v1_base_link" reason="Never" />
-        <disable_collisions link1="${prefix_left}link1" link2="${external_axis_prefix}aico2_10_v1_link2" reason="Never" />
-        <disable_collisions link1="${prefix_left}link1" link2="${external_axis_prefix}aico2_10_v1_link1" reason="Never" />
-        <disable_collisions link1="${prefix_left}link1" link2="${external_axis_prefix}aico2_10_v1_base_link" reason="Never" />
-        <!-- Right Arm -->
-        <disable_collisions link1="${prefix_right}base_link" link2="${external_axis_prefix}aico2_10_v1_link2" reason="Adjacent" />
-        <disable_collisions link1="${prefix_right}base_link" link2="${external_axis_prefix}aico2_10_v1_link1" reason="Never" />
-        <disable_collisions link1="${prefix_right}base_link" link2="${external_axis_prefix}aico2_10_v1_base_link" reason="Never" />
-        <disable_collisions link1="${prefix_right}link1" link2="${external_axis_prefix}aico2_10_v1_link2" reason="Never" />
-        <disable_collisions link1="${prefix_right}link1" link2="${external_axis_prefix}aico2_10_v1_link1" reason="Never" />
-        <disable_collisions link1="${prefix_right}link1" link2="${external_axis_prefix}aico2_10_v1_base_link" reason="Never" />
-        <!-- Left and Right Arms -->
-        <disable_collisions link1="${prefix_left}base_link" link2="${prefix_right}base_link" reason="Never" />
-        <disable_collisions link1="${prefix_left}link1" link2="${prefix_right}link1" reason="Never" />
-        <!-- External Axis internal -->
-        <disable_collisions link1="${external_axis_prefix}aico2_10_v1_base_link" link2="${external_axis_prefix}aico2_10_v1_link1" reason="Adjacent" />
-        <disable_collisions link1="${external_axis_prefix}aico2_10_v1_base_link" link2="${external_axis_prefix}aico2_10_v1_link2" reason="Never" />
-        <disable_collisions link1="${external_axis_prefix}aico2_10_v1_link1" link2="${external_axis_prefix}aico2_10_v1_link2" reason="Adjacent" />
-    </xacro:if>
+    <!-- Left Arm -->
+    <disable_collisions link1="${prefix_left}base_link" link2="${axis}_link2" reason="Adjacent" />
+    <disable_collisions link1="${prefix_left}base_link" link2="${axis}_link1" reason="Never" />
+    <disable_collisions link1="${prefix_left}base_link" link2="${axis}_base_link" reason="Never" />
+    <disable_collisions link1="${prefix_left}link1" link2="${axis}_link2" reason="Never" />
+    <disable_collisions link1="${prefix_left}link1" link2="${axis}_link1" reason="Never" />
+    <disable_collisions link1="${prefix_left}link1" link2="${axis}_base_link" reason="Never" />
+    <!-- Right Arm -->
+    <disable_collisions link1="${prefix_right}base_link" link2="${axis}_link2" reason="Adjacent" />
+    <disable_collisions link1="${prefix_right}base_link" link2="${axis}_link1" reason="Never" />
+    <disable_collisions link1="${prefix_right}base_link" link2="${axis}_base_link" reason="Never" />
+    <disable_collisions link1="${prefix_right}link1" link2="${axis}_link2" reason="Never" />
+    <disable_collisions link1="${prefix_right}link1" link2="${axis}_link1" reason="Never" />
+    <disable_collisions link1="${prefix_right}link1" link2="${axis}_base_link" reason="Never" />
+    <!-- Left and Right Arms -->
+    <disable_collisions link1="${prefix_left}base_link" link2="${prefix_right}base_link" reason="Never" />
+    <disable_collisions link1="${prefix_left}link1" link2="${prefix_right}link1" reason="Never" />
+    <!-- External Axis internal -->
+    <disable_collisions link1="${axis}_base_link" link2="${axis}_link1" reason="Adjacent" />
+    <disable_collisions link1="${axis}_base_link" link2="${axis}_link2" reason="Never" />
+    <disable_collisions link1="${axis}_link1" link2="${axis}_link2" reason="Adjacent" />
     <!-- Load grippers -->
     <xacro:if value="$(arg load_gripper_left)">

Commit message: Support the six new AICO2 platform types

File: flexiv_hardware/ros2_control/rizon_dual.ros2_control.xacro (robot description, xacro)
@@ -65,7 +65,8 @@
       <xacro:configure_joint joint_name="${prefix_left}joint6" initial_pos="${initial_positions_left['joint6']}" />
       <xacro:configure_joint joint_name="${prefix_left}joint7" initial_pos="${initial_positions_left['joint7']}" />
-      <!-- External axis joints -->
-      <xacro:if value="${external_axis_type == 'aico2_4_v1'}">
-        <joint name="${external_axis_prefix}aico2_4_v1_joint1">
+      <!-- External axis joints. Every AICO2 axis exposes joint1 and joint2, named
+           after the robot type lowercased with dashes as underscores. -->
+      <xacro:if value="${external_axis_type.startswith('aico2')}">
+        <joint name="${external_axis_prefix}${external_axis_type}_joint1">
           <command_interface name="position" />
           <command_interface name="velocity" />
@@ -77,49 +78,5 @@
           <state_interface name="effort" />
         </joint>
-        <joint name="${external_axis_prefix}aico2_4_v1_joint2">
-          <command_interface name="position" />
-          <command_interface name="velocity" />
-          <command_interface name="effort" />
-          <state_interface name="position">
-            <param name="initial_value">0.0</param>
-          </state_interface>
-          <state_interface name="velocity" />
-          <state_interface name="effort" />
-        </joint>
-      </xacro:if>
-      <xacro:if value="${external_axis_type == 'aico2_4_v2'}">
-        <joint name="${external_axis_prefix}aico2_4_v2_joint1">
-          <command_interface name="position" />
-          <command_interface name="velocity" />
-          <command_interface name="effort" />
-          <state_interface name="position">
-            <param name="initial_value">0.0</param>
-          </state_interface>
-          <state_interface name="velocity" />
-          <state_interface name="effort" />
-        </joint>
-        <joint name="${external_axis_prefix}aico2_4_v2_joint2">
-          <command_interface name="position" />
-          <command_interface name="velocity" />
-          <command_interface name="effort" />
-          <state_interface name="position">
-            <param name="initial_value">0.0</param>
-          </state_interface>
-          <state_interface name="velocity" />
-          <state_interface name="effort" />
-        </joint>
-      </xacro:if>
-      <xacro:if value="${external_axis_type == 'aico2_10_v1'}">
-        <joint name="${external_axis_prefix}aico2_10_v1_joint1">
-          <command_interface name="position" />
-          <command_interface name="velocity" />
-          <command_interface name="effort" />
-          <state_interface name="position">
-            <param name="initial_value">0.0</param>
-          </state_interface>
-          <state_interface name="velocity" />
-          <state_interface name="effort" />
-        </joint>
-        <joint name="${external_axis_prefix}aico2_10_v1_joint2">
+        <joint name="${external_axis_prefix}${external_axis_type}_joint2">
           <command_interface name="position" />
           <command_interface name="velocity" />
