Commit message: Update digital IO port count to match RDK v2.2

File: flexiv_hardware/ros2_control/flexiv.ros2_control.xacro (robot description, xacro)
@@ -10,5 +10,5 @@
     fake_sensor_commands:=false
     initial_positions_file
-    num_gpio_ports:=20
+    num_gpio_ports:=24
     ">
     <xacro:property name="initial_positions" value="${xacro.load_yaml(initial_positions_file)['initial_positions']}"/>
@@ -103,6 +103,7 @@
         <state_interface name="effort" />
       </joint>
-      <!-- Digital IO ports: 16 on the control box plus 2 in each wrist connector.
-           Enlight-L and MICO have two wrist connectors (20); Rizon has one (18). -->
+      <!-- Digital IO ports, matching flexiv::rdk::kIOPorts: 16 on the control box, then the
+           M8 connector of each wrist (2 ports per wrist), then the pogo pin connector of each
+           wrist (2 ports per wrist). -->
       <xacro:macro name="loop_gpio" params="idx">
         <command_interface name="digital_output_${idx}" />

File: flexiv_hardware/ros2_control/flexiv_dual.ros2_control.xacro (robot description, xacro)
@@ -18,4 +18,5 @@
     initial_positions_file_left
     initial_positions_file_right
+    num_gpio_ports:=24
     ">
     <xacro:include filename="$(find flexiv_description)/urdf/common/flexiv_common.xacro" />
@@ -65,8 +66,11 @@
            interfaces "<robot_sn>_gpio" (or "gpio" when robot_sn is empty) regardless of
            arm count. -->
+      <!-- Digital IO ports, matching flexiv::rdk::kIOPorts: 16 on the control box, then the
+           M8 connector of each wrist (2 ports per wrist), then the pogo pin connector of each
+           wrist (2 ports per wrist). -->
       <xacro:macro name="loop_gpio" params="idx">
         <command_interface name="digital_output_${idx}" />
         <state_interface name="digital_input_${idx}" />
-        <xacro:if value="${idx &lt; 19}">
+        <xacro:if value="${idx &lt; num_gpio_ports - 1}">
           <xacro:loop_gpio idx="${idx+1}" />
         </xacro:if>

File: flexiv_hardware/ros2_control/flexiv_mico.ros2_control.xacro (robot description, xacro)
@@ -18,4 +18,5 @@
     initial_positions_file_right
     torso_initial_positions_file
+    num_gpio_ports:=24
     ">
     <xacro:include filename="$(find flexiv_description)/urdf/common/flexiv_common.xacro" />
@@ -85,9 +86,12 @@
         <state_interface name="effort" />
       </joint>
-      <!-- Single GPIO block for the whole robot. 20 ports -->
+      <!-- Single GPIO block for the whole robot. -->
+      <!-- Digital IO ports, matching flexiv::rdk::kIOPorts: 16 on the control box, then the
+           M8 connector of each wrist (2 ports per wrist), then the pogo pin connector of each
+           wrist (2 ports per wrist). -->
       <xacro:macro name="mico_loop_gpio" params="idx">
         <command_interface name="digital_output_${idx}" />
         <state_interface name="digital_input_${idx}" />
-        <xacro:if value="${idx &lt; 19}">
+        <xacro:if value="${idx &lt; num_gpio_ports - 1}">
           <xacro:mico_loop_gpio idx="${idx+1}" />
         </xacro:if>

File: flexiv_hardware/urdf/flexiv.urdf.xacro (robot description, xacro)
@@ -34,7 +34,8 @@
         + 'Enlight-L, Enlight-LL, MICO-Core, MICO-Plus, MICO-Ultra')}
     </xacro:unless>
-    <!-- Enlight-L has 20 digital IO ports: 16 on the control box plus 2 in each of
-         its two wrist connectors. -->
-    <xacro:property name="num_gpio_ports" value="20" />
+    <!-- Digital IO ports, matching flexiv::rdk::kIOPorts: 16 on the control box, then the M8
+         connector of each wrist (2 ports per wrist), then the pogo pin connector of each wrist
+         (2 ports per wrist). -->
+    <xacro:property name="num_gpio_ports" value="24" />
     <xacro:property name="arm_init" value="${cfg}/Enlight-L/initial_positions.yaml" />
     <xacro:property name="arm_init_mirrored"
@@ -73,5 +74,6 @@
           fake_sensor_commands="$(arg fake_sensor_commands)"
           initial_positions_file_left="${arm_init}"
-          initial_positions_file_right="${init_right}" />
+          initial_positions_file_right="${init_right}"
+          num_gpio_ports="${num_gpio_ports}" />
       </xacro:unless>
       <xacro:if value="${is_mico_torso}">
@@ -85,5 +87,6 @@
           initial_positions_file_left="${arm_init}"
           initial_positions_file_right="${init_right}"
-          torso_initial_positions_file="${cfg}/${rtype}/torso_initial_positions.yaml" />
+          torso_initial_positions_file="${cfg}/${rtype}/torso_initial_positions.yaml"
+          num_gpio_ports="${num_gpio_ports}" />
       </xacro:if>
     </xacro:if>

Commit message: Sync launch files and configs, fix AICO1-4-V2 actuated joints and SRDF collisions, and update dependencies, CI and docs

File: flexiv_hardware/ros2_control/flexiv.ros2_control.xacro (robot description, xacro)
@@ -18,5 +18,6 @@
     <xacro:property name="initial_positions" value="${xacro.load_yaml(initial_positions_file)['initial_positions']}"/>
     <xacro:include filename="$(find flexiv_description)/urdf/common/flexiv_common.xacro" />
-    <!-- GPIO is named from robot_sn alone, matching the hardware interface. -->
+    <!-- GPIO is named from robot_sn alone, as gpio_controller expects. The hardware interface
+         names it from its prefix parameter, which is the same while arm_prefix is empty. -->
     <xacro:compute_arm_prefix robot_sn="${robot_sn}" />
     <xacro:property name="sn_prefix" value="${computed_arm_prefix}" lazy_eval="false" />
@@ -127,7 +128,6 @@
       </xacro:if>
       <xacro:if value="${external_axis_type == 'aico1_4_v2'}">
+        <!-- joint2 and joint_head are not actuated on this variant. -->
         <xacro:ext_axis_joint name="aico1_4_v2_joint1" />
-        <xacro:ext_axis_joint name="aico1_4_v2_joint2" />
-        <xacro:ext_axis_joint name="aico1_4_v2_joint_head" />
       </xacro:if>
       <!-- Digital IO ports: 16 on the control box plus 2 in each wrist connector.

File: flexiv_moveit_config/srdf/aico1.srdf.xacro (robot description, xacro)
@@ -1,4 +1,4 @@
 <?xml version="1.0" encoding="UTF-8"?>
-<robot xmlns:xacro="http://wiki.ros.org/xacro" name="aico1">
+<robot xmlns:xacro="http://wiki.ros.org/xacro" name="$(arg robot_type)">
     <!-- parameters -->
     <xacro:arg name="robot_type" default="AICO1-4-V1" />
@@ -17,10 +17,8 @@
     <!-- Arm -->
     <xacro:rizon_srdf prefix="${prefix}"
-        load_mounted_ft_sensor="$(arg load_mounted_ft_sensor)" use_virtual_joint="false" />
+        load_mounted_ft_sensor="$(arg load_mounted_ft_sensor)" />
     <xacro:property name="external_axis_prefix" value="$(arg external_axis_prefix)" />
-    <!-- Virtual Joint and Platform Group -->
+    <!-- Platform Group -->
     <xacro:if value="${axis_name == 'aico1_4_v1'}">
-        <virtual_joint name="virtual_joint" type="fixed" parent_frame="world"
-            child_link="${external_axis_prefix}aico1_4_v1_base_link" />
         <group name="${external_axis_prefix}aico1_4_v1_platform_${prefix}arm">
             <chain base_link="${external_axis_prefix}aico1_4_v1_base_link" tip_link="${prefix}flange" />
@@ -28,6 +26,4 @@
     </xacro:if>
     <xacro:if value="${axis_name == 'aico1_4_v2'}">
-        <virtual_joint name="virtual_joint" type="fixed" parent_frame="world"
-            child_link="${external_axis_prefix}aico1_4_v2_base_link" />
         <group name="${external_axis_prefix}aico1_4_v2_platform_${prefix}arm">
             <chain base_link="${external_axis_prefix}aico1_4_v2_base_link" tip_link="${prefix}flange" />
@@ -55,4 +51,6 @@
         <disable_collisions link1="${prefix}link1" link2="${external_axis_prefix}aico1_4_v2_neck_link" reason="Never" />
         <disable_collisions link1="${prefix}link1" link2="${external_axis_prefix}aico1_4_v2_head_link" reason="Never" />
+        <disable_collisions link1="${external_axis_prefix}aico1_4_v2_base_link" link2="${external_axis_prefix}aico1_4_v2_torso_mount" reason="Adjacent" />
+        <disable_collisions link1="${external_axis_prefix}aico1_4_v2_torso_mount" link2="${external_axis_prefix}aico1_4_v2_link1" reason="Adjacent" />
         <disable_collisions link1="${external_axis_prefix}aico1_4_v2_base_link" link2="${external_axis_prefix}aico1_4_v2_link1" reason="Adjacent" />
         <disable_collisions link1="${external_axis_prefix}aico1_4_v2_base_link" link2="${external_axis_prefix}aico1_4_v2_neck_link" reason="Never" />

File: flexiv_moveit_config/srdf/aico2.srdf.xacro (robot description, xacro)
@@ -1,4 +1,4 @@
 <?xml version="1.0" encoding="UTF-8"?>
-<robot xmlns:xacro="http://wiki.ros.org/xacro" name="aico2">
+<robot xmlns:xacro="http://wiki.ros.org/xacro" name="$(arg robot_type)">
     <!-- parameters -->
     <xacro:arg name="robot_type" default="AICO2-4-V1" />
@@ -14,24 +14,20 @@
     <xacro:arg name="load_mounted_ft_sensor_left" default="false" />
     <xacro:arg name="load_mounted_ft_sensor_right" default="false" />
-    <xacro:arg name="arm_prefix_left" default="left" />
-    <xacro:arg name="arm_prefix_right" default="right" />
     <xacro:include filename="$(find flexiv_moveit_config)/srdf/rizon_macro.srdf.xacro" />
     <!-- Prefixes. lazy_eval is off so each capture resolves before the next call. -->
-    <xacro:compute_prefix side="$(arg arm_prefix_left)" robot_sn="$(arg robot_sn_left)" />
+    <xacro:compute_prefix side="left" robot_sn="$(arg robot_sn_left)" />
     <xacro:property name="prefix_left" value="${computed_prefix}" lazy_eval="false" />
-    <xacro:compute_prefix side="$(arg arm_prefix_right)" robot_sn="$(arg robot_sn_right)" />
+    <xacro:compute_prefix side="right" robot_sn="$(arg robot_sn_right)" />
     <xacro:property name="prefix_right" value="${computed_prefix}" lazy_eval="false" />
     <xacro:property name="external_axis_prefix" value="$(arg external_axis_prefix)" />
     <!-- Left Arm -->
     <xacro:rizon_srdf prefix="${prefix_left}"
-        load_mounted_ft_sensor="$(arg load_mounted_ft_sensor_left)" use_virtual_joint="false" />
+        load_mounted_ft_sensor="$(arg load_mounted_ft_sensor_left)" />
     <!-- Right Arm -->
     <xacro:rizon_srdf prefix="${prefix_right}"
-        load_mounted_ft_sensor="$(arg load_mounted_ft_sensor_right)" use_virtual_joint="false" />
-    <!-- Virtual Joint and External Axis Group. Every AICO2 axis has the same
+        load_mounted_ft_sensor="$(arg load_mounted_ft_sensor_right)" />
+    <!-- External Axis Group. Every AICO2 axis has the same
          base_link/link1/link2 topology, so one block covers all of them. -->
     <xacro:property name="axis" value="${external_axis_prefix}${axis_name}" />
-    <virtual_joint name="virtual_joint" type="fixed" parent_frame="world"
-        child_link="${axis}_base_link" />
     <group name="${axis}_platform_${prefix_left}arm">
         <chain base_link="${axis}_base_link" tip_link="${prefix_left}flange" />

File: flexiv_moveit_config/srdf/rizon_dual.srdf.xacro (robot description, xacro)
@@ -1,4 +1,4 @@
 <?xml version="1.0" encoding="UTF-8"?>
-<robot xmlns:xacro="http://wiki.ros.org/xacro" name="rizon_dual">
+<robot xmlns:xacro="http://wiki.ros.org/xacro" name="Rizon-Dual">
     <!-- parameters -->
     <xacro:arg name="robot_sn_left" default="" />
@@ -8,12 +8,9 @@
     <xacro:arg name="load_mounted_ft_sensor_left" default="false" />
     <xacro:arg name="load_mounted_ft_sensor_right" default="false" />
-    <!-- Side names carry no trailing underscore; compute_prefix inserts the separator. -->
-    <xacro:arg name="prefix_left" default="left" />
-    <xacro:arg name="prefix_right" default="right" />
     <xacro:include filename="$(find flexiv_moveit_config)/srdf/rizon_macro.srdf.xacro" />
     <!-- Arm Prefixes. lazy_eval is off so each capture resolves before the next call. -->
-    <xacro:compute_prefix side="$(arg prefix_left)" robot_sn="$(arg robot_sn_left)" />
+    <xacro:compute_prefix side="left" robot_sn="$(arg robot_sn_left)" />
     <xacro:property name="left_arm_prefix" value="${computed_prefix}" lazy_eval="false" />
-    <xacro:compute_prefix side="$(arg prefix_right)" robot_sn="$(arg robot_sn_right)" />
+    <xacro:compute_prefix side="right" robot_sn="$(arg robot_sn_right)" />
     <xacro:property name="right_arm_prefix" value="${computed_prefix}" lazy_eval="false" />
     <!-- Left Arm -->

File: flexiv_moveit_config/srdf/rizon_macro.srdf.xacro (robot description, xacro)
@@ -17,5 +17,5 @@
     </xacro:macro>
     <!-- 'prefix' is the fully-formed prefix, normally from compute_prefix above. -->
-    <xacro:macro name="rizon_srdf" params="prefix load_mounted_ft_sensor use_virtual_joint:=true">
+    <xacro:macro name="rizon_srdf" params="prefix load_mounted_ft_sensor">
         <group name="${prefix}arm">
             <chain base_link="${prefix}base_link" tip_link="${prefix}flange" />
@@ -30,8 +30,4 @@
             <joint name="${prefix}joint7" value="0" />
         </group_state>
-        <xacro:if value="${use_virtual_joint}">
-            <virtual_joint name="virtual_joint" type="fixed" parent_frame="world"
-                child_link="${prefix}base_link" />
-        </xacro:if>
         <disable_collisions link1="${prefix}base_link" link2="${prefix}link1" reason="Adjacent" />
         <disable_collisions link1="${prefix}base_link" link2="${prefix}link2" reason="Never" />
