Commit message: Release/Flexiv ROS 2 Lyrical 1.9.4 (#141)

File: flexiv_hardware/ros2_control/flexiv.ros2_control.xacro (robot description, xacro)
@@ -9,4 +9,6 @@
     robot_sn
     rdk_control_mode:='joint_position'
+    rdk_realtime_mode:=false
+    withhold_on_timeliness_failure:=true
     use_fake_hardware:=false
     fake_sensor_commands:=false
@@ -18,5 +20,6 @@
     <xacro:property name="initial_positions" value="${xacro.load_yaml(initial_positions_file)['initial_positions']}"/>
     <xacro:include filename="$(find flexiv_description)/urdf/common/flexiv_common.xacro" />
-    <!-- GPIO is named from robot_sn alone, matching the hardware interface. -->
+    <!-- GPIO is named from robot_sn alone, as gpio_controller expects. The hardware interface
+         names it from its prefix parameter, which is the same while arm_prefix is empty. -->
     <xacro:compute_arm_prefix robot_sn="${robot_sn}" />
     <xacro:property name="sn_prefix" value="${computed_arm_prefix}" lazy_eval="false" />
@@ -26,5 +29,5 @@
           <plugin>mock_components/GenericSystem</plugin>
           <param name="mock_sensor_commands">${fake_sensor_commands}</param>
-          <param name="state_following_offset">0.0</param>
+          <param name="position_state_following_offset">0.0</param>
         </xacro:if>
         <xacro:unless value="${use_fake_hardware}">
@@ -33,4 +36,6 @@
           <param name="prefix">${prefix}</param>
           <param name="rdk_control_mode">${rdk_control_mode}</param>
+          <param name="rdk_realtime_mode">${rdk_realtime_mode}</param>
+          <param name="withhold_on_timeliness_failure">${withhold_on_timeliness_failure}</param>
           <xacro:unless value="${external_axis_type == ''}">
             <param name="external_axis_type">${external_axis_type}</param>
@@ -127,7 +132,6 @@
       </xacro:if>
       <xacro:if value="${external_axis_type == 'aico1_4_v2'}">
+        <!-- joint2 and joint_head are not actuated on this variant. -->
         <xacro:ext_axis_joint name="aico1_4_v2_joint1" />
-        <xacro:ext_axis_joint name="aico1_4_v2_joint2" />
-        <xacro:ext_axis_joint name="aico1_4_v2_joint_head" />
       </xacro:if>
       <!-- Digital IO ports: 16 on the control box plus 2 in each wrist connector.
@@ -143,4 +147,6 @@
         <xacro:loop_gpio idx="0" />
       </gpio>
+      <!-- The TCP belongs to the arm, so it is named like the joints. -->
+      <xacro:flexiv_cartesian_gpio name="${prefix}tcp" />
     </ros2_control>
   </xacro:macro>

File: flexiv_hardware/ros2_control/rizon_dual.ros2_control.xacro (robot description, xacro)
@@ -8,4 +8,6 @@
     robot_sn_right
     rdk_control_mode:='joint_position'
+    rdk_realtime_mode:=false
+    withhold_on_timeliness_failure:=true
     use_fake_hardware:=false
     fake_sensor_commands:=false
@@ -28,5 +30,5 @@
           <plugin>mock_components/GenericSystem</plugin>
           <param name="mock_sensor_commands">${fake_sensor_commands}</param>
-          <param name="state_following_offset">0.0</param>
+          <param name="position_state_following_offset">0.0</param>
         </xacro:if>
         <xacro:unless value="${use_fake_hardware}">
@@ -37,4 +39,6 @@
           <param name="prefix_right">${prefix_right}</param>
           <param name="rdk_control_mode">${rdk_control_mode}</param>
+          <param name="rdk_realtime_mode">${rdk_realtime_mode}</param>
+          <param name="withhold_on_timeliness_failure">${withhold_on_timeliness_failure}</param>
           <param name="external_axis_type">${external_axis_type}</param>
           <param name="translation_left_x">${translation_left_x}</param>
@@ -65,7 +69,8 @@
       <xacro:configure_joint joint_name="${prefix_left}joint6" initial_pos="${initial_positions_left['joint6']}" />
       <xacro:configure_joint joint_name="${prefix_left}joint7" initial_pos="${initial_positions_left['joint7']}" />
-      <!-- External axis joints -->
-      <xacro:if value="${external_axis_type == 'aico2_4_v1'}">
-        <joint name="${external_axis_prefix}aico2_4_v1_joint1">
+      <!-- External axis joints. Every AICO2 axis exposes joint1 and joint2, named
+           after the robot type lowercased with dashes as underscores. -->
+      <xacro:if value="${external_axis_type.startswith('aico2')}">
+        <joint name="${external_axis_prefix}${external_axis_type}_joint1">
           <command_interface name="position" />
           <command_interface name="velocity" />
@@ -77,49 +82,5 @@
           <state_interface name="effort" />
         </joint>
-        <joint name="${external_axis_prefix}aico2_4_v1_joint2">
-          <command_interface name="position" />
-          <command_interface name="velocity" />
-          <command_interface name="effort" />
-          <state_interface name="position">
-            <param name="initial_value">0.0</param>
-          </state_interface>
-          <state_interface name="velocity" />
-          <state_interface name="effort" />
-        </joint>
-      </xacro:if>
-      <xacro:if value="${external_axis_type == 'aico2_4_v2'}">
-        <joint name="${external_axis_prefix}aico2_4_v2_joint1">
-          <command_interface name="position" />
-          <command_interface name="velocity" />
-          <command_interface name="effort" />
-          <state_interface name="position">
-            <param name="initial_value">0.0</param>
-          </state_interface>
-          <state_interface name="velocity" />
-          <state_interface name="effort" />
-        </joint>
-        <joint name="${external_axis_prefix}aico2_4_v2_joint2">
-          <command_interface name="position" />
-          <command_interface name="velocity" />
-          <command_interface name="effort" />
-          <state_interface name="position">
-            <param name="initial_value">0.0</param>
-          </state_interface>
-          <state_interface name="velocity" />
-          <state_interface name="effort" />
-        </joint>
-      </xacro:if>
-      <xacro:if value="${external_axis_type == 'aico2_10_v1'}">
-        <joint name="${external_axis_prefix}aico2_10_v1_joint1">
-          <command_interface name="position" />
-          <command_interface name="velocity" />
-          <command_interface name="effort" />
-          <state_interface name="position">
-            <param name="initial_value">0.0</param>
-          </state_interface>
-          <state_interface name="velocity" />
-          <state_interface name="effort" />
-        </joint>
-        <joint name="${external_axis_prefix}aico2_10_v1_joint2">
+        <joint name="${external_axis_prefix}${external_axis_type}_joint2">
           <command_interface name="position" />
           <command_interface name="velocity" />
@@ -153,4 +114,6 @@
         <xacro:loop_gpio idx="0" />
       </gpio>
+      <xacro:flexiv_cartesian_gpio name="${prefix_left}tcp" />
+      <xacro:flexiv_cartesian_gpio name="${prefix_right}tcp" />
     </ros2_control>
   </xacro:macro>

File: flexiv_hardware/urdf/flexiv.urdf.xacro (robot description, xacro)
@@ -8,9 +8,13 @@
   which xacro resolves before <xacro:arg> defaults are read.
 -->
-<robot xmlns:xacro="http://www.ros.org/wiki/xacro" name="$(arg robot_type)">
+<robot xmlns:xacro="http://www.ros.org/wiki/xacro" name="$(arg robot_type)" version="1.2">
   <xacro:arg name="robot_type" default="Rizon4" />
   <!-- Other args come from the description entry point included below. -->
   <xacro:arg name="ros2_control" default="true" />
   <xacro:arg name="rdk_control_mode" default="joint_position" />
+  <!-- Real-time RDK modes for the joint and Cartesian interfaces, streamed at the control rate -->
+  <xacro:arg name="rdk_realtime_mode" default="false" />
+  <!-- Withhold motion when real-time commands arrive late too often, or only warn as the RDK does -->
+  <xacro:arg name="withhold_on_timeliness_failure" default="true" />
   <xacro:arg name="use_fake_hardware" default="false" />
   <xacro:arg name="fake_sensor_commands" default="false" />
@@ -23,12 +27,16 @@
     <xacro:include filename="$(find flexiv_hardware)/ros2_control/flexiv.ros2_control.xacro" />
     <xacro:include filename="$(find flexiv_hardware)/ros2_control/rizon_dual.ros2_control.xacro" />
+    <xacro:include filename="$(find flexiv_hardware)/ros2_control/cartesian.ros2_control.xacro" />
     <xacro:property name="cfg" value="$(find flexiv_description)/config" />
     <xacro:property name="rtype" value="$(arg robot_type)" />
     <xacro:property name="single_arms"
       value="${['Rizon4', 'Rizon4s', 'Rizon4M', 'Rizon4R', 'Rizon10', 'Rizon10s', 'Rizon10R']}" />
+    <xacro:property name="aico1_types" value="${['AICO1-4-V1', 'AICO1-4-V2']}" />
+    <xacro:property name="aico2_types"
+      value="${['AICO2-4-V1', 'AICO2-4-V2', 'AICO2-4-D3', 'AICO2-4E-D1', 'AICO2-4U-D1',
+                'AICO2-10-V1', 'AICO2-10-D2', 'AICO2-10E-D1', 'AICO2-10U-D1']}" />
     <xacro:property name="is_single" value="${rtype in single_arms}" />
-    <xacro:property name="is_aico1" value="${rtype in ['AICO1-4-V1', 'AICO1-4-V2']}" />
-    <xacro:property name="is_aico2"
-      value="${rtype in ['AICO2-4-V1', 'AICO2-4-V2', 'AICO2-10-V1']}" />
+    <xacro:property name="is_aico1" value="${rtype in aico1_types}" />
+    <xacro:property name="is_aico2" value="${rtype in aico2_types}" />
     <xacro:property name="is_rizon_dual" value="${rtype == 'Rizon-Dual'}" />
     <!-- Two robots with two serial numbers, as opposed to one robot with two arms. -->
@@ -36,5 +44,5 @@
     <xacro:unless value="${is_single or is_aico1 or is_paired}">
       ${xacro.error('robot_type ' + rtype + ' is not supported by this release. Supported: '
-        + ', '.join(single_arms + ['AICO1-4-V1', 'AICO1-4-V2', 'Rizon-Dual', 'AICO2-4-V1', 'AICO2-4-V2', 'AICO2-10-V1']))}
+        + ', '.join(single_arms + aico1_types + ['Rizon-Dual'] + aico2_types))}
     </xacro:unless>
     <!-- The hardware interface takes the external axis as a lowercase name. -->
@@ -45,6 +53,7 @@
     <xacro:property name="aico1_arm"
       value="${'$(arg arm_type)' if '$(arg arm_type)' != '' else 'Rizon4'}" />
-    <xacro:property name="paired_default_left" value="${'Rizon10' if rtype == 'AICO2-10-V1' else 'Rizon4'}" />
-    <xacro:property name="paired_default_right" value="${'Rizon10R' if rtype == 'AICO2-10-V1' else 'Rizon4R'}" />
+    <xacro:property name="is_aico2_10" value="${rtype.startswith('AICO2-10')}" />
+    <xacro:property name="paired_default_left" value="${'Rizon10' if is_aico2_10 else 'Rizon4'}" />
+    <xacro:property name="paired_default_right" value="${'Rizon10R' if is_aico2_10 else 'Rizon4R'}" />
     <xacro:property name="arm_left"
       value="${'$(arg arm_type_left)' if '$(arg arm_type_left)' != '' else paired_default_left}" />
@@ -63,4 +72,6 @@
         robot_sn="$(arg robot_sn)"
         rdk_control_mode="$(arg rdk_control_mode)"
+        rdk_realtime_mode="$(arg rdk_realtime_mode)"
+        withhold_on_timeliness_failure="$(arg withhold_on_timeliness_failure)"
         use_fake_hardware="$(arg use_fake_hardware)"
         fake_sensor_commands="$(arg fake_sensor_commands)"
@@ -76,4 +87,6 @@
         robot_sn="$(arg robot_sn)"
         rdk_control_mode="$(arg rdk_control_mode)"
+        rdk_realtime_mode="$(arg rdk_realtime_mode)"
+        withhold_on_timeliness_failure="$(arg withhold_on_timeliness_failure)"
         use_fake_hardware="$(arg use_fake_hardware)"
         fake_sensor_commands="$(arg fake_sensor_commands)"
@@ -95,4 +108,6 @@
         robot_sn_right="$(arg robot_sn_right)"
         rdk_control_mode="$(arg rdk_control_mode)"
+        rdk_realtime_mode="$(arg rdk_realtime_mode)"
+        withhold_on_timeliness_failure="$(arg withhold_on_timeliness_failure)"
         use_fake_hardware="$(arg use_fake_hardware)"
         fake_sensor_commands="$(arg fake_sensor_commands)"
