Commit message: Forwardport/Jazzy v1.9.4 features to v2.2 (#142)

File: flexiv_hardware/ros2_control/flexiv.ros2_control.xacro (robot description, xacro)
@@ -7,4 +7,7 @@
     robot_sn
     rdk_control_mode:='joint_position'
+    rdk_realtime_mode:=true
+    withhold_on_timeliness_failure:=false
+    max_joint_acceleration:=5.0
     use_fake_hardware:=false
     fake_sensor_commands:=false
@@ -31,4 +34,7 @@
           <param name="prefix">${prefix}</param>
           <param name="rdk_control_mode">${rdk_control_mode}</param>
+          <param name="rdk_realtime_mode">${rdk_realtime_mode}</param>
+          <param name="withhold_on_timeliness_failure">${withhold_on_timeliness_failure}</param>
+          <param name="max_joint_acceleration">${max_joint_acceleration}</param>
         </xacro:unless>
       </hardware>
@@ -116,4 +122,6 @@
         <xacro:loop_gpio idx="0" />
       </gpio>
+      <!-- The TCP belongs to the arm, so it is named like the joints. -->
+      <xacro:flexiv_cartesian_gpio name="${prefix}tcp" />
     </ros2_control>
   </xacro:macro>

File: flexiv_hardware/ros2_control/flexiv_dual.ros2_control.xacro (robot description, xacro)
@@ -14,4 +14,7 @@
     robot_sn
     rdk_control_mode:='joint_position'
+    rdk_realtime_mode:=true
+    withhold_on_timeliness_failure:=false
+    max_joint_acceleration:=5.0
     use_fake_hardware:=false
     fake_sensor_commands:=false
@@ -42,4 +45,7 @@
           <param name="prefix_right">${prefix_right}</param>
           <param name="rdk_control_mode">${rdk_control_mode}</param>
+          <param name="rdk_realtime_mode">${rdk_realtime_mode}</param>
+          <param name="withhold_on_timeliness_failure">${withhold_on_timeliness_failure}</param>
+          <param name="max_joint_acceleration">${max_joint_acceleration}</param>
         </xacro:unless>
       </hardware>
@@ -79,4 +85,7 @@
         <xacro:loop_gpio idx="0" />
       </gpio>
+      <!-- The TCP belongs to the arm, so it is named like the joints. -->
+      <xacro:flexiv_cartesian_gpio name="${prefix_left}tcp" />
+      <xacro:flexiv_cartesian_gpio name="${prefix_right}tcp" />
     </ros2_control>
   </xacro:macro>

File: flexiv_hardware/ros2_control/flexiv_mico.ros2_control.xacro (robot description, xacro)
@@ -13,4 +13,7 @@
     robot_sn
     rdk_control_mode:='joint_position'
+    rdk_realtime_mode:=true
+    withhold_on_timeliness_failure:=false
+    max_joint_acceleration:=5.0
     use_fake_hardware:=false
     fake_sensor_commands:=false
@@ -44,4 +47,7 @@
           <param name="prefix_right">${prefix_right}</param>
           <param name="rdk_control_mode">${rdk_control_mode}</param>
+          <param name="rdk_realtime_mode">${rdk_realtime_mode}</param>
+          <param name="withhold_on_timeliness_failure">${withhold_on_timeliness_failure}</param>
+          <param name="max_joint_acceleration">${max_joint_acceleration}</param>
         </xacro:unless>
       </hardware>
@@ -100,4 +106,7 @@
         <xacro:mico_loop_gpio idx="0" />
       </gpio>
+      <!-- The TCP belongs to the arm, so it is named like the joints. -->
+      <xacro:flexiv_cartesian_gpio name="${prefix_left}tcp" />
+      <xacro:flexiv_cartesian_gpio name="${prefix_right}tcp" />
     </ros2_control>
   </xacro:macro>

File: flexiv_hardware/urdf/flexiv.urdf.xacro (robot description, xacro)
@@ -16,4 +16,11 @@
   <xacro:arg name="fake_sensor_commands" default="false" />
   <xacro:arg name="initial_positions_file" default="" />
+  <!-- Real-time RDK modes for the joint and Cartesian interfaces, streamed at the control rate.
+       false selects the non-real-time modes, smoothed by the robot's motion generator. -->
+  <xacro:arg name="rdk_realtime_mode" default="true" />
+  <!-- Withhold motion when real-time commands arrive late too often, or only warn as the RDK does -->
+  <xacro:arg name="withhold_on_timeliness_failure" default="false" />
+  <!-- Acceleration limit of the robot's joint motion generator in the non-real-time modes [rad/s^2] -->
+  <xacro:arg name="max_joint_acceleration" default="5.0" />
   <!-- Robot model, including the arg declarations this file relies on
        (robot_sn, arm_prefix). -->
@@ -24,4 +31,5 @@
     <xacro:include filename="$(find flexiv_hardware)/ros2_control/flexiv_dual.ros2_control.xacro" />
     <xacro:include filename="$(find flexiv_hardware)/ros2_control/flexiv_mico.ros2_control.xacro" />
+    <xacro:include filename="$(find flexiv_hardware)/ros2_control/cartesian.ros2_control.xacro" />
     <xacro:property name="cfg" value="$(find flexiv_description)/config" />
     <xacro:property name="rtype" value="$(arg robot_type)" />
@@ -51,4 +59,7 @@
         robot_sn="$(arg robot_sn)"
         rdk_control_mode="$(arg rdk_control_mode)"
+        rdk_realtime_mode="$(arg rdk_realtime_mode)"
+        withhold_on_timeliness_failure="$(arg withhold_on_timeliness_failure)"
+        max_joint_acceleration="$(arg max_joint_acceleration)"
         use_fake_hardware="$(arg use_fake_hardware)"
         fake_sensor_commands="$(arg fake_sensor_commands)"
@@ -71,4 +82,7 @@
           robot_sn="$(arg robot_sn)"
           rdk_control_mode="$(arg rdk_control_mode)"
+          rdk_realtime_mode="$(arg rdk_realtime_mode)"
+          withhold_on_timeliness_failure="$(arg withhold_on_timeliness_failure)"
+          max_joint_acceleration="$(arg max_joint_acceleration)"
           use_fake_hardware="$(arg use_fake_hardware)"
           fake_sensor_commands="$(arg fake_sensor_commands)"
@@ -83,4 +97,7 @@
           robot_sn="$(arg robot_sn)"
           rdk_control_mode="$(arg rdk_control_mode)"
+          rdk_realtime_mode="$(arg rdk_realtime_mode)"
+          withhold_on_timeliness_failure="$(arg withhold_on_timeliness_failure)"
+          max_joint_acceleration="$(arg max_joint_acceleration)"
           use_fake_hardware="$(arg use_fake_hardware)"
           fake_sensor_commands="$(arg fake_sensor_commands)"

File: flexiv_moveit_config/srdf/flexiv.srdf.xacro (robot description, xacro)
@@ -26,11 +26,12 @@
              The macro computes prefix = arm_prefix + robot_sn + '_', so
              arm_prefix="left_" yields prefix "left_<sn>_" as required.
-             Virtual joints are disabled because both arms parent to 'world' via the URDF. -->
+             No virtual joint is declared: the URDF already roots every arm at 'world'. -->
         <xacro:flexiv_srdf arm_prefix="left_" robot_sn="$(arg robot_sn)"
-            load_mounted_ft_sensor="$(arg load_mounted_ft_sensor)"
-            use_virtual_joint="false" />
+            load_mounted_ft_sensor="$(arg load_mounted_ft_sensor)" />
+        <!-- The MICO arms face each other, so the right arm starts mirrored, as in the URDF -->
+        <xacro:property name="init_dir" value="$(find flexiv_description)/config/Enlight-L" />
         <xacro:flexiv_srdf arm_prefix="right_" robot_sn="$(arg robot_sn)"
             load_mounted_ft_sensor="$(arg load_mounted_ft_sensor)"
-            use_virtual_joint="false" />
+            initial_positions_file="${init_dir + ('/initial_positions.yaml' if '$(arg robot_type)' == 'Enlight-LL' else '/initial_positions_mirrored.yaml')}" />
         <!-- Combined group that references both arm sub-groups -->
         <xacro:property name="left_prefix" value="${'left_' + '$(arg robot_sn)' + '_'}" />
@@ -58,4 +59,19 @@
         value="${'$(arg robot_type)' in ['MICO-Plus', 'MICO-Ultra']}" />
     <xacro:property name="torso_prefix" value="${'$(arg robot_sn)' + '_torso_'}" />
+    <!-- The neck and head (flexiv_description jazzy-v3.1) are fixed to the torso link the arms
+         mount on, so their poses relative to that link and to both arm bases never change. Their
+         collision checks are disabled against all of these; the arm links keep theirs. -->
+    <xacro:macro name="mico_neck_head_collisions" params="mount">
+        <disable_collisions link1="${mount}" link2="${torso_prefix}neck_link" reason="Adjacent" />
+        <disable_collisions link1="${torso_prefix}neck_link" link2="${torso_prefix}head_link"
+            reason="Adjacent" />
+        <disable_collisions link1="${mount}" link2="${torso_prefix}head_link" reason="Never" />
+        <xacro:macro name="mico_rigid_to_arm_bases" params="link">
+            <disable_collisions link1="${link}" link2="${left_prefix}base_link" reason="Never" />
+            <disable_collisions link1="${link}" link2="${right_prefix}base_link" reason="Never" />
+        </xacro:macro>
+        <xacro:mico_rigid_to_arm_bases link="${torso_prefix}neck_link" />
+        <xacro:mico_rigid_to_arm_bases link="${torso_prefix}head_link" />
+    </xacro:macro>
     <!-- MICO-Core: fixed torso; both arm bases mount directly on the torso base_link. -->
     <xacro:if value="${is_mico_core}">
@@ -66,4 +82,5 @@
         <disable_collisions link1="${left_prefix}base_link" link2="${right_prefix}base_link"
             reason="Never" />
+        <xacro:mico_neck_head_collisions mount="${torso_prefix}base_link" />
     </xacro:if>
     <!-- MICO-Plus / MICO-Ultra: 2-DoF torso (base_link -> link1 -> link2); arms mount on link2. -->
@@ -95,4 +112,5 @@
         <disable_collisions link1="${left_prefix}base_link" link2="${right_prefix}base_link"
             reason="Never" />
+        <xacro:mico_neck_head_collisions mount="${torso_prefix}link2" />
     </xacro:if>
 </robot>

File: flexiv_moveit_config/srdf/flexiv_macro.srdf.xacro (robot description, xacro)
@@ -1,23 +1,23 @@
 <?xml version="1.0" encoding="UTF-8"?>
 <robot xmlns:xacro="http://www.ros.org/wiki/xacro">
-    <xacro:macro name="flexiv_srdf" params="arm_prefix robot_sn load_mounted_ft_sensor use_virtual_joint:=true">
+    <xacro:macro name="flexiv_srdf"
+        params="arm_prefix robot_sn load_mounted_ft_sensor
+                initial_positions_file:='$(find flexiv_description)/config/Enlight-L/initial_positions.yaml'">
         <!-- Prefix defaults to 'arm_prefix_robot_sn' -->
         <xacro:property name="prefix" value="${arm_prefix + robot_sn + '_'}" />
+        <!-- Home is the arm's initial pose in flexiv_description, the same one the URDF starts from -->
+        <xacro:property name="home" value="${xacro.load_yaml(initial_positions_file)['initial_positions']}" />
         <group name="${prefix}arm">
             <chain base_link="${prefix}base_link" tip_link="${prefix}flange" />
         </group>
         <group_state name="${prefix}home" group="${prefix}arm">
-            <joint name="${prefix}joint1" value="0" />
-            <joint name="${prefix}joint2" value="${-2*pi/9}" />
-            <joint name="${prefix}joint3" value="0" />
-            <joint name="${prefix}joint4" value="${pi/2}" />
-            <joint name="${prefix}joint5" value="0" />
-            <joint name="${prefix}joint6" value="${2*pi/9}" />
-            <joint name="${prefix}joint7" value="0" />
+            <joint name="${prefix}joint1" value="${home['joint1']}" />
+            <joint name="${prefix}joint2" value="${home['joint2']}" />
+            <joint name="${prefix}joint3" value="${home['joint3']}" />
+            <joint name="${prefix}joint4" value="${home['joint4']}" />
+            <joint name="${prefix}joint5" value="${home['joint5']}" />
+            <joint name="${prefix}joint6" value="${home['joint6']}" />
+            <joint name="${prefix}joint7" value="${home['joint7']}" />
         </group_state>
-        <xacro:if value="${use_virtual_joint}">
-            <virtual_joint name="virtual_joint" type="fixed" parent_frame="world"
-                child_link="${prefix}base_link" />
-        </xacro:if>
         <disable_collisions link1="${prefix}base_link" link2="${prefix}link1" reason="Adjacent" />
         <disable_collisions link1="${prefix}base_link" link2="${prefix}link2" reason="Never" />
