Commit message: Add Rizon10R support

File: flexiv_hardware/urdf/flexiv.urdf.xacro (robot description, xacro)
@@ -26,5 +26,5 @@
     <xacro:property name="rtype" value="$(arg robot_type)" />
     <xacro:property name="single_arms"
-      value="${['Rizon4', 'Rizon4s', 'Rizon4M', 'Rizon4R', 'Rizon10', 'Rizon10s']}" />
+      value="${['Rizon4', 'Rizon4s', 'Rizon4M', 'Rizon4R', 'Rizon10', 'Rizon10s', 'Rizon10R']}" />
     <xacro:property name="is_single" value="${rtype in single_arms}" />
     <xacro:property name="is_aico1" value="${rtype in ['AICO1-4-V1', 'AICO1-4-V2']}" />
@@ -46,5 +46,5 @@
       value="${'$(arg arm_type)' if '$(arg arm_type)' != '' else 'Rizon4'}" />
     <xacro:property name="paired_default_left" value="${'Rizon10' if rtype == 'AICO2-10-V1' else 'Rizon4'}" />
-    <xacro:property name="paired_default_right" value="${'Rizon10' if rtype == 'AICO2-10-V1' else 'Rizon4R'}" />
+    <xacro:property name="paired_default_right" value="${'Rizon10R' if rtype == 'AICO2-10-V1' else 'Rizon4R'}" />
     <xacro:property name="arm_left"
       value="${'$(arg arm_type_left)' if '$(arg arm_type_left)' != '' else paired_default_left}" />

Commit message: Use RDK v2.1 and its 20 digital IO ports for testing with RCA v3E.1

File: flexiv_hardware/urdf/flexiv.urdf.xacro (robot description, xacro)
@@ -42,8 +42,8 @@
         + 'Enlight-L, Enlight-LL, MICO-Core, MICO-Plus, MICO-Ultra')}
     </xacro:unless>
-    <!-- Digital IO ports, matching flexiv::rdk::kIOPorts: 16 on the control box, then the M8
-         connector of each wrist (2 ports per wrist), then the pogo pin connector of each wrist
-         (2 ports per wrist). -->
-    <xacro:property name="num_gpio_ports" value="24" />
+    <!-- Digital IO ports, matching flexiv::rdk::kIOPorts of RDK v2.1: 16 on the control box, then
+         the M8 connector of each wrist (2 ports per wrist). RDK v2.2 adds the pogo pin connector of
+         each wrist, for 24. -->
+    <xacro:property name="num_gpio_ports" value="20" />
     <xacro:property name="arm_init" value="${cfg}/Enlight-L/initial_positions.yaml" />
     <xacro:property name="arm_init_mirrored"
